File: 03-engine_dyno/engine_dyno_v1/MCU.kicad_sch (KiCad schematic)
At the start: 3 parts, among them IC1 TEENSY_4.1, P1 J1B1211CCD

Commit message: transducer and hall preliminary design
Connections:
- net A2: now reaches IC1.16 (A2)
- net A3: now reaches IC1.17 (A3)
- net A14: now reaches IC1.38 (A14)
Changed lines of the file:
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@@
+	(wire
+		(pts
+			(xy 113.03 99.06) (xy 115.57 99.06)
+		)
+		(stroke
+			(width 0)
+			(type default)
+		)
+	)
 	(wire
 		(pts
@@
 	(wire
 		(pts
+			(xy 168.91 76.2) (xy 171.45 76.2)
+		)
+		(stroke
+			(width 0)
+			(type default)
+		)
+	)
+	(wire
+		(pts
 			(xy 198.12 116.84) (xy 201.93 116.84)
 		)
@@
 	(wire
 		(pts
+			(xy 113.03 96.52) (xy 115.57 96.52)
+		)
+		(stroke
+			(width 0)
+			(type default)
+		)
+	)
+	(wire
+		(pts
 			(xy 168.91 121.92) (xy 172.72 121.92)
 		)
@@
 		)
 	)
+	(hierarchical_label "A14"
+		(shape input)
+		(at 171.45 76.2 0)
+		(effects
+			(font
+				(size 1.27 1.27)
+			)
+			(justify left)
+		)
+	)
+	(hierarchical_label "A3"
+		(shape input)
+		(at 113.03 99.06 180)
+		(effects
+			(font
+				(size 1.27 1.27)
+			)
+			(justify right)
+		)
+	)
 	(hierarchical_label "CS_2"
 		(shape output)
@@
 		)
 	)
+	(hierarchical_label "A2"
+		(shape input)
+		(at 113.03 96.52 180)
+		(effects
+			(font
+				(size 1.27 1.27)
+			)
+			(justify right)
+		)
+	)
