File: 03-engine_dyno/engine_dyno_v1/MCU.kicad_sch (KiCad schematic)
At the start: 3 parts, among them IC1 TEENSY_4.1, P1 J1B1211CCD

Commit message: clean up
Parts:
- added U6: Teensy4.1, 22XT_Main:Teensy41, symbol 22XT_Main:Teensy4.1
Connections:
- net A15: now reaches IC1.39 (A15)
Other:
- moved on the sheet: P1

Commit message: new transducer
Parts:
- removed IC1: TEENSY_4.1, engine_dyno:TEENSY41, symbol TEENSY_4.1:TEENSY_4.1
- added C37: 0.1u, symbol Device:C_Small
Connections:
- net +3V3: now also P1.10 (GRN+), U6.15 (3V3)
- net +5V: now also U6.48 (VIN)
- net +5V_USB: now also U6.49 (VUSB)
- net A14: now also U6.30 (38_CS1_IN1)
- net A15: now also U6.31 (39_MISO1_OUT1A)
- net A2: now also U6.38 (16_A2_RX4_SCL1)
- net A3: now also U6.39 (17_A3_TX4_SDA1)
- net CS_1: now also U6.12 (10_CS_MQSR)
- net CS_2: now also U6.28 (36_CS)
- net CS_3: now also U6.29 (37_CS)
- net GND: now also P1.13 (CH_GND@2), P1.14 (CH_GND@3), P1.8 (GH_GND@1), U6.1 (GND), U6.47 (GND), U6.52 (GND), U6.58 (GND), U6.59 (GND), U6.64 (GND), C37.2
- net MISO: now also U6.14 (12_MISO_MQSL)
- net MOSI: now also U6.13 (11_MOSI_CTX1)
- net SCK: now also U6.35 (13_SCK_LED)
- net at P1.1 (TD+): now also U6.63 (T+)
- net at P1.2 (TCT): now also P1.5 (RCT), C37.1
- net at P1.3 (TD-): now also U6.62 (T-)
- net at P1.4 (RD+): now also U6.60 (R+)
- net at P1.6 (RD-): now also U6.65 (R-)
- net at P1.9 (GRN-): now also U6.61 (LED)
- net A16: now reaches U6.32 (40_A16)
- no-connect marks 0 -> 45
Other:
- moved on the sheet: C9, P1, U6

Commit message: beginnings of a pcb
Parts:
- C37, C9: footprint (none) -> Capacitor_SMD:C_0402_1005Metric
- U6: footprint 22XT_Main:Teensy41 -> engine_dyno:Teensy41
Changed lines of the file:
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@@
 			)
 		)
-		(property "Footprint" ""
+		(property "Footprint" "Capacitor_SMD:C_0402_1005Metric"
 			(at 134.62 104.14 0)
 			(effects
@@
 			)
 		)
-		(property "Footprint" ""
+		(property "Footprint" "Capacitor_SMD:C_0402_1005Metric"
 			(at 135.89 41.91 0)
 			(effects
@@
 			)
 		)
-		(property "Footprint" "22XT_Main:Teensy41"
+		(property "Footprint" "engine_dyno:Teensy41"
 			(at 72.39 90.17 0)
 			(effects

Commit message: added math and changes to schematic
Changed lines of the file:
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@@
-	)
-	(junction
-		(at 128.27 45.72)
-		(diameter 0)
-		(color 0 0 0 0)
 	)
 	(junction
@@
 	(wire
 		(pts
-			(xy 110.49 45.72) (xy 128.27 45.72)
-		)
-		(stroke
-			(width 0)
-			(type default)
-		)
-	)
-	(wire
-		(pts
 			(xy 123.19 115.57) (xy 123.19 113.03)
 		)
@@
 	(wire
 		(pts
-			(xy 128.27 45.72) (xy 135.89 45.72)
+			(xy 110.49 45.72) (xy 135.89 45.72)
 		)
 		(stroke
@@
 					(unit 1)
 				)
-			)
-		)
-	)
-	(symbol
-		(lib_id "power:PWR_FLAG")
-		(at 128.27 45.72 0)
-		(unit 1)
-		(exclude_from_sim no)
-		(in_bom yes)
-		(on_board yes)
-		(dnp no)
-		(property "Reference" "#FLG04"
-			(at 128.27 43.815 0)
-			(effects
-				(font
-					(size 1.27 1.27)
-				)
-				(hide yes)
-			)
-		)
-		(property "Value" "PWR_FLAG"
-			(at 128.27 40.64 0)
-			(effects
-				(font
-					(size 1.27 1.27)
-				)
-			)
-		)
-		(property "Footprint" ""
-			(at 128.27 45.72 0)
-			(effects
-				(font
-					(size 1.27 1.27)
-				)
-				(hide yes)
-			)
-		)
-		(property "Datasheet" "~"
-			(at 128.27 45.72 0)
-			(effects
-				(font
-					(size 1.27 1.27)
-				)
-				(hide yes)
-			)
-		)
-		(property "Description" "Special symbol for telling ERC where power comes from"
-			(at 128.27 45.72 0)
-			(effects
-				(font
-					(size 1.27 1.27)
-				)
-				(hide yes)
-			)
-		)
-		(pin "1"
-		)
-		(instances
-			(project ""
-				(path "/d283b024-74fa-4d4c-9089-b2007a8f756c/98235854-983d-4e64-9110-73cbe2c5a722"
-					(reference "#FLG04")
-					(unit 1)
-				)

Commit message: general layout
Connections:
- net GND: now also U6.34 (GND)
- no-connect marks 45 -> 44
Changed lines of the file:
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@@
-	)
-	(no_connect
-		(at 110.49 81.28)
 	)
 	(no_connect
@@
 		(pts
 			(xy 123.19 113.03) (xy 137.16 113.03)
+		)
+		(stroke
+			(width 0)
+			(type default)
+		)
+	)
+	(wire
+		(pts
+			(xy 113.03 81.28) (xy 110.49 81.28)
 		)
 		(stroke
@@
 					(unit 1)
 				)
+			)
+		)
+	)
+	(symbol
+		(lib_id "power:GND")
+		(at 113.03 81.28 90)
+		(unit 1)
+		(exclude_from_sim no)
+		(in_bom yes)
+		(on_board yes)
+		(dnp no)
+		(property "Reference" "#PWR054"
+			(at 119.38 81.28 0)
+			(effects
+				(font
+					(size 1.27 1.27)
+				)
+				(hide yes)
+			)
+		)
+		(property "Value" "GND"
+			(at 116.84 81.2799 90)
+			(effects
+				(font
+					(size 1.27 1.27)
+				)
+				(justify right)
+			)
+		)
+		(property "Footprint" ""
+			(at 113.03 81.28 0)
+			(effects
+				(font
+					(size 1.27 1.27)
+				)
+				(hide yes)
+			)
+		)
+		(property "Datasheet" ""
+			(at 113.03 81.28 0)
+			(effects
+				(font
+					(size 1.27 1.27)
+				)
+				(hide yes)
+			)
+		)
+		(property "Description" "Power symbol creates a global label with name \"GND\" , ground"
+			(at 113.03 81.28 0)
+			(effects
+				(font
+					(size 1.27 1.27)
+				)
+				(hide yes)
+			)
+		)
+		(pin "1"
+		)
+		(instances
+			(project "engine_dyno_v1"
+				(path "/d283b024-74fa-4d4c-9089-b2007a8f756c/98235854-983d-4e64-9110-73cbe2c5a722"
+					(reference "#PWR054")
+					(unit 1)
+				)

Commit message: layout and 3d models
Connections:
- net A15: now also U6.45 (23_A9_CRX1_MCLK1); no longer U6.31 (39_MISO1_OUT1A)
- net A16: now also U6.20 (28_RX7); no longer U6.32 (40_A16)
- net A2: now also U6.11 (9_OUT1C); no longer U6.38 (16_A2_RX4_SCL1)
- net A3: now also U6.10 (8_TX2_IN1); no longer U6.39 (17_A3_TX4_SDA1)
- net CS_1: now also U6.37 (15_A1_RX3_SPDIF_IN); no longer U6.12 (10_CS_MQSR)
- net CS_3: now also U6.44 (22_A8_CTX1); no longer U6.29 (37_CS)
- net TD+: now reaches P1.1 (TD+), U6.63 (T+)
- net TD-: now reaches P1.3 (TD-), U6.62 (T-)
- net RD+: now reaches P1.4 (RD+), U6.60 (R+)
- net RD-: now reaches P1.6 (RD-), U6.65 (R-)
Other:
- note added: "Microcontroller + Ethernet"
Changed lines of the file:
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@@
 	(generator_version "9.0")
 	(paper "A4")
+	(rectangle
+		(start 32.512 26.162)
+		(end 172.72 162.306)
+		(stroke
+			(width 0)
+			(type default)
+		)
+		(fill
+			(type none)
+		)
+	)
+	(text "Microcontroller + Ethernet"
+		(exclude_from_sim no)
+		(at 145.288 160.274 0)
+		(effects
+			(font
+				(size 1.27 1.27)
+			)
+			(justify left)
+		)
+	)
 	(junction
 		(at 135.89 45.72)
@@
 	)
 	(no_connect
-		(at 54.61 71.12)
-	)
-	(no_connect
 		(at 54.61 120.65)
 	)
 	(no_connect
+		(at 54.61 55.88)
+	)
+	(no_connect
 		(at 110.49 104.14)
 	)
 	(no_connect
+		(at 110.49 71.12)
+	)
+	(no_connect
 		(at 54.61 50.8)
 	)
 	(no_connect
+		(at 54.61 53.34)
+	)
+	(no_connect
 		(at 54.61 58.42)
 	)
@@
 	)
 	(no_connect
-		(at 54.61 53.34)
-	)
-	(no_connect
 		(at 54.61 109.22)
 	)
@@
 	)
 	(no_connect
-		(at 110.49 55.88)
-	)
-	(no_connect
-		(at 110.49 73.66)
-	)
-	(no_connect
 		(at 54.61 66.04)
 	)
@@
 	)
 	(no_connect
-		(at 54.61 68.58)
-	)
-	(no_connect
 		(at 110.49 63.5)
 	)
 	(no_connect
-		(at 54.61 55.88)
+		(at 54.61 73.66)
+	)
+	(no_connect
+		(at 110.49 93.98)
 	)
 	(no_connect
@@
 	)
 	(no_connect
+		(at 110.49 99.06)
+	)
+	(no_connect
 		(at 110.49 50.8)
 	)
@@
 	)
 	(no_connect
-		(at 110.49 53.34)
+		(at 110.49 68.58)
 	)
 	(no_connect
@@
 	)
 	(no_connect
-		(at 54.61 93.98)
-	)
-	(no_connect
 		(at 90.17 133.35)
 	)
@@
 	)
 	(no_connect
+		(at 110.49 88.9)
+	)
+	(no_connect
 		(at 54.61 96.52)
 	)
@@
 	)
 	(no_connect
-		(at 110.49 99.06)
-	)
-	(no_connect
 		(at 54.61 60.96)
 	)
@@
 		(at 110.49 66.04)
 	)
+	(no_connect
+		(at 110.49 86.36)
+	)
 	(wire
 		(pts
@@
 	(wire
 		(pts
-			(xy 113.03 88.9) (xy 110.49 88.9)
+			(xy 113.03 53.34) (xy 110.49 53.34)
+		)
+		(stroke
+			(width 0)
+			(type default)
+		)
+	)
+	(wire
+		(pts
+			(xy 50.8 93.98) (xy 54.61 93.98)
 		)
 		(stroke
@@
 	(wire
 		(pts
-			(xy 113.03 86.36) (xy 110.49 86.36)
-		)
-		(stroke
-			(width 0)
-			(type default)
-		)
-	)
-	(wire
-		(pts
 			(xy 127 123.19) (xy 127 120.65)
 		)
@@
 	(wire
 		(pts
-			(xy 113.03 68.58) (xy 110.49 68.58)
-		)
-		(stroke
-			(width 0)
-			(type default)
-		)
-	)
-	(wire
-		(pts
 			(xy 137.16 115.57) (xy 134.62 115.57)
 		)
@@
 	(wire
 		(pts
+			(xy 113.03 73.66) (xy 110.49 73.66)
+		)
+		(stroke
+			(width 0)
+			(type default)
+		)
+	)
+	(wire
+		(pts
 			(xy 113.03 113.03) (xy 110.49 113.03)
 		)
@@
 	(wire
 		(pts
-			(xy 113.03 93.98) (xy 110.49 93.98)
-		)
-		(stroke
-			(width 0)
-			(type default)
-		)
-	)
-	(wire
-		(pts
 			(xy 135.89 45.72) (xy 139.7 45.72)
 		)
@@
 	(wire
 		(pts
+			(xy 50.8 68.58) (xy 54.61 68.58)
+		)
+		(stroke
+			(width 0)
+			(type default)
+		)
+	)
+	(wire
+		(pts
 			(xy 110.49 120.65) (xy 123.19 120.65)
 		)
@@
 	(wire
 		(pts
+			(xy 50.8 71.12) (xy 54.61 71.12)
+		)
+		(stroke
+			(width 0)
+			(type default)
+		)
+	)
+	(wire
+		(pts
 			(xy 110.49 45.72) (xy 135.89 45.72)
 		)
@@
 	(wire
 		(pts
-			(xy 113.03 71.12) (xy 110.49 71.12)
-		)
-		(stroke
-			(width 0)
-			(type default)
-		)
-	)
-	(wire
-		(pts
 			(xy 123.19 135.89) (xy 137.16 135.89)
 		)
@@
 	(wire
 		(pts
-			(xy 50.8 73.66) (xy 54.61 73.66)
-		)
-		(stroke
-			(width 0)
-			(type default)
-		)
-	)
-	(wire
-		(pts
 			(xy 113.03 78.74) (xy 110.49 78.74)
 		)
@@
 	(wire
 		(pts
+			(xy 113.03 55.88) (xy 110.49 55.88)
+		)
+		(stroke
+			(width 0)
+			(type default)
+		)
+	)
+	(wire
+		(pts
 			(xy 130.81 110.49) (xy 130.81 125.73)
 		)
@@
 			(width 0)
 			(type default)
+		)
+	)
+	(label "RD+"
+		(at 127 120.65 180)
+		(effects
+			(font
+				(size 1.27 1.27)
+			)
+			(justify right bottom)
+		)
+	)
+	(label "RD-"
+		(at 130.81 125.73 180)
+		(effects
+			(font
+				(size 1.27 1.27)
+			)
+			(justify right bottom)
+		)
+	)
+	(label "TD+"
+		(at 127 113.03 180)
+		(effects
+			(font
+				(size 1.27 1.27)
+			)
+			(justify right bottom)
+		)
+	)
+	(label "TD-"
+		(at 123.19 118.11 0)
+		(effects
+			(font
+				(size 1.27 1.27)
+			)
+			(justify left bottom)
 		)
 	)
 	(hierarchical_label "A16"
 		(shape input)
-		(at 113.03 86.36 0)
-		(effects
-			(font
-				(size 1.27 1.27)
-			)
-			(justify left)
+		(at 50.8 93.98 180)
+		(effects
+			(font
+				(size 1.27 1.27)
+			)
+			(justify right)
 		)
 	)
@@
 	(hierarchical_label "A3"
 		(shape input)
-		(at 113.03 68.58 0)
-		(effects
-			(font
-				(size 1.27 1.27)
-			)
-			(justify left)
+		(at 50.8 68.58 180)
+		(effects
+			(font
+				(size 1.27 1.27)
+			)
+			(justify right)
 		)
 	)
@@
 	(hierarchical_label "CS_1"
 		(shape output)
-		(at 50.8 73.66 180)
-		(effects
-			(font
-				(size 1.27 1.27)
-			)
-			(justify right)
+		(at 113.03 73.66 0)
+		(effects
+			(font
+				(size 1.27 1.27)
+			)
+			(justify left)
 		)
 	)
@@
 	(hierarchical_label "CS_3"
 		(shape output)
-		(at 113.03 93.98 0)
+		(at 113.03 55.88 0)
 		(effects
 			(font
@@
 	(hierarchical_label "A2"
 		(shape input)
-		(at 113.03 71.12 0)
-		(effects
-			(font
-				(size 1.27 1.27)
-			)
-			(justify left)
+		(at 50.8 71.12 180)
+		(effects
+			(font
+				(size 1.27 1.27)
+			)
+			(justify right)
 		)
 	)
 	(hierarchical_label "A15"
 		(shape input)
-		(at 113.03 88.9 0)
-		(effects
-			(font
+		(at 113.03 53.34 0)
+		(effects
+			(font

Commit message: im aboutta release
Parts:
- U6: symbol 22XT_Main:Teensy4.1 -> Teensy:Teensy4.1
Changed lines of the file:
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@@
 	)
 	(symbol
-		(lib_id "22XT_Main:Teensy4.1")
+		(lib_id "Teensy:Teensy4.1")
 		(at 82.55 100.33 0)
 		(unit 1)
