File: 03-engine_dyno/engine_dyno_v1/engine_dyno_v1.kicad_sch (KiCad schematic)
At the start: 0 parts

Commit message: transducer and hall preliminary design
Other:
- sheet Hall ports: added HALL1; removed none
- sheet MCU ports: added A14, A2, A3; removed none
- sheet Transducer ports: added BIAS_REF, CS, DIN, DOUT/~DRDY, DRDY, MID_REF, SCLK; removed none
