File: 03-engine_dyno/engine_dyno_v1/engine_dyno_v1.kicad_sch (KiCad schematic)
At the start: 0 parts

Commit message: clean up
Other:
- sheet Hall renamed Hall1
- sheet Transducer renamed Transducer1
- added sheet Hall2 (hall.kicad_sch)
- added sheet Transducer2 (transducer.kicad_sch)

Commit message: new transducer
Other:
- sheet Transducer1 renamed Model1605
- removed sheet Transducer2
- added sheet TMNR-5KM (TMNR-5KM.kicad_sch)
- sheet Hall1 ports: added HALL; removed HALL1
- sheet Hall2 ports: added HALL; removed HALL2
- sheet MCU ports: added A15, A16; removed none
- sheet Model1605: file transducer.kicad_sch -> Model1605.kicad_sch

Commit message: added math and changes to schematic
Other:
- sheet Model1605 ports: added A14, CS!, MISO, MOSI, SCK; removed CS, DIN, DOUT/~DRDY, DRDY, SCLK
- sheet References ports: added CS_1, MOSI, SCK; removed SCLK, SDIN, SYNC
- sheet TMNR-5KM ports: added A15, CS!, MISO, MOSI, SCK; removed CS, DIN, DOUT/~DRDY, DRDY, SCLK
Changed lines of the file:
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@@
 			)
 		)
-		(pin "SCLK" input
+		(pin "SCK" input
 			(at 194.31 76.2 180)
 			(effects
@@
 			)
 		)
-		(pin "SDIN" input
+		(pin "MOSI" input
 			(at 194.31 68.58 180)
 			(effects
@@
 			)
 		)
-		(pin "SYNC" input
+		(pin "CS_1" input
 			(at 194.31 44.45 180)
 			(effects
@@
 		)
 		(property "Sheetfile" "Model1605.kicad_sch"
-			(at 193.04 152.908 0)
+			(at 193.04 135.636 0)
 			(effects
 				(font
@@
 			)
 		)
-		(pin "CS" input
+		(pin "CS!" input
 			(at 214.63 99.06 90)
 			(effects
@@
 			)
 		)
-		(pin "DIN" input
+		(pin "MOSI" input
 			(at 193.04 114.3 180)
 			(effects
@@
 			)
 		)
-		(pin "DOUT{slash}~DRDY" input
+		(pin "MISO" input
 			(at 193.04 129.54 180)
 			(effects
@@
 			)
 		)
-		(pin "DRDY" input
+		(pin "A14" input
 			(at 207.01 99.06 90)
 			(effects
@@
 			)
 		)
-		(pin "SCLK" input
+		(pin "SCK" input
 			(at 193.04 121.92 180)
 			(effects
@@
 			)
 		)
-		(pin "CS" input
+		(pin "CS!" input
 			(at 144.78 99.06 90)
 			(effects
@@
 			)
 		)
-		(pin "DIN" input
+		(pin "MOSI" input
 			(at 176.53 114.3 0)
 			(effects
@@
 			)
 		)
-		(pin "DOUT{slash}~DRDY" input
+		(pin "MISO" input
 			(at 176.53 129.54 0)
 			(effects
@@
 			)
 		)
-		(pin "DRDY" input
+		(pin "A15" input
 			(at 138.43 99.06 90)
 			(effects
@@
 			)
 		)
-		(pin "SCLK" input
+		(pin "SCK" input
 			(at 176.53 121.92 0)
 			(effects

Commit message: im aboutta release
Parts:
- added H1, H2, H3, H4: MountingHole, MountingHole:MountingHole_3.2mm_M3_DIN965, symbol Mechanical:MountingHole

Commit message: fillet, plated holes, via size
Parts:
- H1, H2, H3, H4: footprint MountingHole:MountingHole_3.2mm_M3_DIN965 -> MountingHole:MountingHole_3.2mm_M3_DIN965_Pad
Changed lines of the file:
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@@
 			)
 		)
-		(property "Footprint" "MountingHole:MountingHole_3.2mm_M3_DIN965"
+		(property "Footprint" "MountingHole:MountingHole_3.2mm_M3_DIN965_Pad"
 			(at 27.94 34.29 0)
 			(effects
@@
 			)
 		)
-		(property "Footprint" "MountingHole:MountingHole_3.2mm_M3_DIN965"
+		(property "Footprint" "MountingHole:MountingHole_3.2mm_M3_DIN965_Pad"
 			(at 27.94 44.45 0)
 			(effects
@@
 			)
 		)
-		(property "Footprint" "MountingHole:MountingHole_3.2mm_M3_DIN965"
+		(property "Footprint" "MountingHole:MountingHole_3.2mm_M3_DIN965_Pad"
 			(at 27.94 39.37 0)
 			(effects
@@
 			)
 		)
-		(property "Footprint" "MountingHole:MountingHole_3.2mm_M3_DIN965"
+		(property "Footprint" "MountingHole:MountingHole_3.2mm_M3_DIN965_Pad"
 			(at 27.94 49.53 0)
 			(effects
