File: 03-engine_dyno/engine_dyno_v1/hall.kicad_sch (KiCad schematic)
At the start: 1 part, among them J3 Screw_Terminal_01x03

Commit message: transducer and hall preliminary design
Parts:
- added C19: 1n, symbol Device:C_Small
- added C20: 0.1u, symbol Device:C_Small
- added R11, R12: 4.7k, symbol Device:R_Small_US
- added U10: 74LVC1G17, symbol 74xGxx:74LVC1G17
Connections:
- net GND: now reaches J3.1 (Pin_1)
- net GND: now also C19.1, C20.2, U10.3 (GND)
- net SIG: now reaches J3.2 (Pin_2)
- net SIG: now also U10.2
- net PWR: now reaches J3.3 (Pin_3)
- new net: R11.2, R12.1, U10.4
- new net +5V: C20.1, R11.1, U10.5 (VCC)
- new net HALL1: C19.2, R12.2
