File: 03-engine_dyno/engine_dyno_v1/hall.kicad_sch (KiCad schematic)
At the start: 6 parts, among them J3 Screw_Terminal_01x03, U10 74LVC1G17

Commit message: clean up
Parts:
- renumbered C19 to C36, J3 to J7, R11 to R26, U10 to U16
Connections:
- net PWR is gone; now on net +5V: J7.3 (Pin_3)
- net +5V: no longer C20.1, U16.5 (VCC)
- net SIG: now also R26.2
- net at R12.1, U16.4: no longer R26.2
- new net +3V3: C20.1, U16.5 (VCC)
Other:
- note added: "Buffer Level Shifter"
- moved on the sheet: C20, C36, J7, R12, R26, U16

Commit message: new transducer
Connections:
- net HALL1 renamed HALL
Changed lines of the file:
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@@
 		)
 	)
-	(hierarchical_label "HALL1"
-		(shape input)
+	(hierarchical_label "HALL"
+		(shape output)
 		(at 157.48 85.09 0)
 		(effects

Commit message: beginnings of a pcb
Parts:
- C20, C36: footprint (none) -> Capacitor_SMD:C_0402_1005Metric
- J7: footprint (none) -> TerminalBlock_RND:TerminalBlock_RND_205-00233_1x03_P5.08mm_Horizontal
- R12, R26: footprint (none) -> Resistor_SMD:R_0402_1005Metric
- U16: footprint (none) -> Package_TO_SOT_SMD:SOT-23-5
Changed lines of the file:
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@@
 			)
 		)
-		(property "Footprint" ""
+		(property "Footprint" "Resistor_SMD:R_0402_1005Metric"
 			(at 109.22 80.01 0)
 			(effects
@@
 			)
 		)
-		(property "Footprint" ""
+		(property "Footprint" "Capacitor_SMD:C_0402_1005Metric"
 			(at 132.08 72.39 0)
 			(effects
@@
 			)
 		)
-		(property "Footprint" ""
+		(property "Footprint" "Capacitor_SMD:C_0402_1005Metric"
 			(at 154.94 80.01 0)
 			(effects
@@
 			)
 		)
-		(property "Footprint" ""
+		(property "Footprint" "Package_TO_SOT_SMD:SOT-23-5"
 			(at 129.54 85.09 0)
 			(effects
@@
 			)
 		)
-		(property "Footprint" ""
+		(property "Footprint" "TerminalBlock_RND:TerminalBlock_RND_205-00233_1x03_P5.08mm_Horizontal"
 			(at 96.52 99.06 0)
 			(effects
@@
 			)
 		)
-		(property "Footprint" ""
+		(property "Footprint" "Resistor_SMD:R_0402_1005Metric"
 			(at 149.86 85.09 0)
 			(effects

Commit message: added math and changes to schematic
Other:
- note added: "Pull-up: Rpu = 4.7 kΩ to +5V (open-collector high level) Noise filter: fc = 1/(2π·R·C) = 1/(2π·4.7k·1n) = 33.9 kHz Level shift: 74LVC1G17 @ VCC=3.3V → out 0/3.3V; input 5.5V-tolerant Max pulse freq = N_targets × RPM/60 (keep ≪ 33.9 kHz)"
Changed lines of the file:
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@@
 	(paper "A4")
 	(rectangle
-		(start 81.534 61.214)
+		(start 81.534 49.53)
 		(end 167.386 107.95)
 		(stroke
@@
 		)
 	)
+	(text "Pull-up: Rpu = 4.7 kΩ to +5V (open-collector high level)\nNoise filter: fc = 1/(2π·R·C) = 1/(2π·4.7k·1n) = 33.9 kHz\nLevel shift: 74LVC1G17 @ VCC=3.3V → out 0/3.3V; input 5.5V-tolerant\nMax pulse freq = N_targets × RPM/60  (keep ≪ 33.9 kHz)"
+		(exclude_from_sim no)
+		(at 124.968 55.372 0)
+		(effects
+			(font
+				(size 1.27 1.27)
+			)
+		)
+	)

Commit message: general layout
Connections:
- net HALL: now also U16.4; no longer C36.2, R12.2
- net SIG: now also R12.1; no longer U16.2
- new net: C36.2, R12.2, U16.2
Other:
- moved on the sheet: C20, C36, R12, R26, U16
