File: 03-engine_dyno/engine_dyno_v1/power.kicad_sch (KiCad schematic)
At the start: 24 parts, among them J1 Screw_Terminal_01x02, Q1 PMOS, U1 TVS1800DRV, U2 TPS2115APWR, U3 LMR51430XDDCR, U4 TPS60403DBVRG4

Commit message: transducer and hall preliminary design
Parts:
- renumbered U3 to U1, U1 to U2, U2 to U3
Changed lines of the file:
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@@
 		(on_board yes)
 		(dnp no)
-		(property "Reference" "U1"
+		(property "Reference" "U2"
 			(at 132.08 62.23 90)
 			(effects
@@
 		(pin "1"
 		)
+		(instances
+			(project "engine_dyno_v1"
+				(path "/d283b024-74fa-4d4c-9089-b2007a8f756c/3b8b6910-3a04-4ae3-b73f-448b33afb94f"
+					(reference "U2")
+					(unit 1)
+				)
+			)
+		)
 	)
 	(symbol
@@
 		(pin "1"
 		)
+		(instances
+			(project "engine_dyno_v1"
+				(path "/d283b024-74fa-4d4c-9089-b2007a8f756c/3b8b6910-3a04-4ae3-b73f-448b33afb94f"
+					(reference "C1")
+					(unit 1)
+				)
+			)
+		)
 	)
 	(symbol
@@
 		(pin "1"
 		)
+		(instances
+			(project "engine_dyno_v1"
+				(path "/d283b024-74fa-4d4c-9089-b2007a8f756c/3b8b6910-3a04-4ae3-b73f-448b33afb94f"
+					(reference "R1")
+					(unit 1)
+				)
+			)
+		)
 	)
 	(symbol
@@
 		(pin "3"
 		)
+		(instances
+			(project "engine_dyno_v1"
+				(path "/d283b024-74fa-4d4c-9089-b2007a8f756c/3b8b6910-3a04-4ae3-b73f-448b33afb94f"
+					(reference "Q1")
+					(unit 1)
+				)
+			)
+		)
 	)
 	(symbol
@@
 		(pin "1"
 		)
+		(instances
+			(project "engine_dyno_v1"
+				(path "/d283b024-74fa-4d4c-9089-b2007a8f756c/3b8b6910-3a04-4ae3-b73f-448b33afb94f"
+					(reference "J1")
+					(unit 1)
+				)
+			)
+		)
 	)
 	(symbol
@@
 		(on_board yes)
 		(dnp no)
-		(property "Reference" "U3"
+		(property "Reference" "U1"
 			(at 95.25 105.41 0)
 			(effects
@@
 		(pin "4"
 		)
+		(instances
+			(project "engine_dyno_v1"
+				(path "/d283b024-74fa-4d4c-9089-b2007a8f756c/3b8b6910-3a04-4ae3-b73f-448b33afb94f"
+					(reference "U1")
+					(unit 1)
+				)
+			)
+		)
 	)
 	(symbol
@@
 		(pin "2"
 		)
+		(instances
+			(project "engine_dyno_v1"
+				(path "/d283b024-74fa-4d4c-9089-b2007a8f756c/3b8b6910-3a04-4ae3-b73f-448b33afb94f"
+					(reference "D1")
+					(unit 1)
+				)
+			)
+		)
 	)
 	(symbol
@@
 		(pin "2"
 		)
+		(instances
+			(project "engine_dyno_v1"
+				(path "/d283b024-74fa-4d4c-9089-b2007a8f756c/3b8b6910-3a04-4ae3-b73f-448b33afb94f"
+					(reference "F1")
+					(unit 1)
+				)
+			)
+		)
 	)
 	(symbol
@@
 		(pin "1"
 		)
+		(instances
+			(project "engine_dyno_v1"
+				(path "/d283b024-74fa-4d4c-9089-b2007a8f756c/3b8b6910-3a04-4ae3-b73f-448b33afb94f"
+					(reference "L1")
+					(unit 1)
+				)
+			)
+		)
 	)
 	(symbol
@@
 		(pin "3"
 		)
+		(instances
+			(project "engine_dyno_v1"
+				(path "/d283b024-74fa-4d4c-9089-b2007a8f756c/3b8b6910-3a04-4ae3-b73f-448b33afb94f"
+					(reference "U4")
+					(unit 1)
+				)
+			)
+		)
 	)
 	(symbol
@@
 		(on_board yes)
 		(dnp no)
-		(property "Reference" "U2"
+		(property "Reference" "U3"
 			(at 209.55 58.42 0)
 			(effects
@@
 		(pin "5"
 		)
+		(instances
+			(project "engine_dyno_v1"
+				(path "/d283b024-74fa-4d4c-9089-b2007a8f756c/3b8b6910-3a04-4ae3-b73f-448b33afb94f"
+					(reference "U3")
+					(unit 1)
+				)
+			)
+		)
 	)
