File: 03-engine_dyno/engine_dyno_v1/engine_dyno_v1.kicad_pcb (KiCad board)
At the start: 4 copper layers, 92 parts, among them J1 Screw_Terminal_01x02, J2 Screw_Terminal_01x02, J3 Screw_Terminal_01x02, J4 Screw_Terminal_01x05, J5 Screw_Terminal_01x03, J6 Screw_Terminal_01x05, J7 Screw_Terminal_01x03, P1 J1B1211CCD, Q1 PMOS, U1 LMR51430XDDCR, U10 INA827AIDGKR, U11 74LVC1G17, U12 AD630ARZ, U13 ADS1120IPWR, U14 OPA192IDBVR, U15 OPA192IDBVR, U16 74LVC1G17, U2 TVS1800DRV, U3 TPS2115APWR, U4 TPS60403DBVRG4, U5 AD5689RBRUZ, U6 Teensy4.1, U7 INA827AIDGKR, U8 AD630ARZ, U9 ADS1120IPWR

Commit message: added math and changes to schematic
Parts:
- moved U2 79.0 mm to (174.2, 85.8)
- moved U4 77.6 mm to (173.8, 80.7)
- moved U3 77.3 mm to (175.3, 74.3)
- moved U1 73.0 mm to (174.6, 91.2)
- moved C1 11.2 mm to (119.7, 117.3)
- moved C11 11.2 mm to (174.6, 108.5)
- moved C12 11.2 mm to (174.6, 110.5)
- moved C13 11.2 mm to (131.9, 63.7)
- moved C14 11.2 mm to (131.9, 65.7)
- moved C15 11.2 mm to (131.9, 67.7)
- moved C16 11.2 mm to (131.9, 69.7)
- moved C17 11.2 mm to (131.9, 71.6)
- moved C18 11.2 mm to (134.8, 63.7)
- moved C2 11.2 mm to (119.7, 119.3)
- moved C20 11.2 mm to (144.0, 117.3)
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
Commit message: general layout
Parts:
- moved P1 105.1 mm to (176.0, 109.4)
- moved C10 103.2 mm to (72.8, 123.5), turned to 180 degrees
- moved C11 102.6 mm to (72.8, 121.6), turned to 180 degrees
- moved C12 102.2 mm to (72.8, 119.6), turned to 180 degrees
- moved C1 86.8 mm to (190.9, 67.8), turned to -45 degrees
- moved D1 85.3 mm to (183.8, 66.1), turned to -90 degrees
- moved R2 84.9 mm to (193.0, 73.3), turned to 90 degrees
- moved F1 83.9 mm to (189.9, 64.7)
- moved C20 81.6 mm to (77.1, 70.6)
- moved C36 81.6 mm to (77.1, 72.5)
- moved R12 81.6 mm to (74.3, 70.6)
- moved R26 81.6 mm to (74.3, 72.6)
- moved U16 81.6 mm to (70.2, 72.0)
- moved J7 81.6 mm to (71.2, 64.2)
- moved C9 80.6 mm to (196.2, 87.2)
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Connections:
- C26 pad 2: /Hall2/HALL -> Net-(C26-Pad2)
- C36 pad 2: /Hall1/HALL -> Net-(C36-Pad2)
- R12 pad 1: Net-(R12-Pad1) -> /Hall1/SIG
- R12 pad 2: /Hall1/HALL -> Net-(C36-Pad2)
- R18 pad 1: Net-(R18-Pad1) -> /Hall2/SIG
- R18 pad 2: /Hall2/HALL -> Net-(C26-Pad2)
- U11 pad 2: /Hall2/SIG -> Net-(C26-Pad2)
- U11 pad 4: Net-(R18-Pad1) -> /Hall2/HALL
- U13 pad 2: /TMNR-5KM/CS! -> /MCU/CS_3
- U16 pad 2: /Hall1/SIG -> Net-(C36-Pad2)
- U16 pad 4: Net-(R12-Pad1) -> /Hall1/HALL
- U5 pad 16: +3V3 -> GND
- U6 pad 34: unconnected-(U6-GND-Pad34) -> GND
Routing:
- net +12V: track 0.00 -> 12.0 mm
- net Net-(D1-K): track 0.00 -> 8.48 mm
- net Net-(D1-A): track 0.00 -> 7.99 mm
- net /power/+12V_BAT: track 0.00 -> 6.33 mm
- net Net-(U1-SW): track 0.00 -> 4.72 mm
- net Net-(U1-FB): track 0.00 -> 2.68 mm
- net Net-(U1-CB): track 0.00 -> 2.62 mm
- net /MCU/A16: track 0.00 -> 0.67 mm

Commit message: some more changes
Parts:
- removed J2, J3: Screw_Terminal_01x02, TerminalBlock_RND:TerminalBlock_RND_205-00232_1x02_P5.08mm_Horizontal
- added C38: 10u, Capacitor_SMD:C_0402_1005Metric, F.Cu at (137.0, 99.0)
- C37, R14, R15, R16, R8: moved to B.Cu
- R11: value 100 -> 390
- R7: value 390 -> 1.5k
- moved J7 109.1 mm to (180.3, 63.8), turned to 180 degrees
- moved R12 101.0 mm to (175.2, 72.2), turned to -90 degrees
- moved U16 99.9 mm to (170.1, 74.7), turned to 180 degrees
- moved C36 98.1 mm to (175.2, 75.2), turned to 90 degrees
- moved R26 96.4 mm to (170.6, 71.7)
- moved R17 93.0 mm to (179.8, 106.5)
- moved C26 90.4 mm to (174.2, 104.1), turned to -90 degrees
- moved C20 89.5 mm to (166.5, 75.2), turned to 90 degrees
- moved R18 87.8 mm to (174.7, 106.5)
- moved C25 81.7 mm to (165.5, 107.0), turned to 90 degrees
- moved J5 80.2 mm to (170.1, 116.5), turned to 0 degrees
- moved U11 78.3 mm to (169.1, 106.5)
- moved C11 71.5 mm to (134.6, 85.6), turned to -90 degrees
- moved C12 68.0 mm to (137.0, 97.2)
- moved C10 66.4 mm to (133.9, 97.5), turned to 90 degrees
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Connections:
- U12 pad 15: /TMNR-5KM/AD630_OUT -> Net-(U12-CH_A-)
- U6 pad 11: unconnected-(U6-9_OUT1C-Pad11) -> /MCU/A16
- U6 pad 12: /MCU/CS_1 -> unconnected-(U6-10_CS_MQSR-Pad12)
- U6 pad 29: /MCU/CS_3 -> unconnected-(U6-37_CS-Pad29)
- U6 pad 31: /MCU/A15 -> unconnected-(U6-39_MISO1_OUT1A-Pad31)
- U6 pad 32: /MCU/A16 -> unconnected-(U6-40_A16-Pad32)
- U6 pad 37: unconnected-(U6-15_A1_RX3_SPDIF_IN-Pad37) -> /MCU/CS_1
- U6 pad 38: /Hall1/HALL -> unconnected-(U6-16_A2_RX4_SCL1-Pad38)
- U6 pad 39: /Hall2/HALL -> unconnected-(U6-17_A3_TX4_SDA1-Pad39)
- U6 pad 4: unconnected-(U6-2_OUT2-Pad4) -> /Hall1/HALL
- U6 pad 44: unconnected-(U6-22_A8_CTX1-Pad44) -> /MCU/A15
- U6 pad 45: unconnected-(U6-23_A9_CRX1_MCLK1-Pad45) -> /MCU/CS_3
- U6 pad 5: unconnected-(U6-3_LRCLK2-Pad5) -> /Hall2/HALL
- U8 pad 15: /Model1605/AD630_OUT -> Net-(U8-CH_A-)
Routing:
- net /MCU/+5V_USB: track 0.00 -> 128.7 mm, vias 0 -> 1
- net +5V: track 0.00 -> 56.1 mm, vias 0 -> 5
- net Net-(U7-VOUT): track 0.00 -> 20.5 mm
- net -5V: track 0.00 -> 18.4 mm, vias 0 -> 4
- net /MCU/MOSI: track 0.00 -> 16.7 mm
- net /Hall2/SIG: track 0.00 -> 14.1 mm
- net Net-(U8-SEL_A): track 0.00 -> 13.1 mm, vias 0 -> 1
- net +3V3: track 0.00 -> 13.0 mm, vias 0 -> 2
- net /TMNR-5KM/SIG+: track 0.00 -> 12.5 mm
- net /power/+5V_BUCK: track 0.00 -> 12.3 mm
- net /Hall1/SIG: track 0.00 -> 11.9 mm
- net Net-(U8-SEL_B): track 0.00 -> 11.8 mm, vias 0 -> 1
- net /Model1605/SIG+: track 0.00 -> 11.5 mm
- net Net-(C15-Pad1): track 0.00 -> 10.9 mm, vias 0 -> 2
- net /TMNR-5KM/SIG-: track 0.00 -> 10.8 mm
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- added copper zone on In2.Cu, net +5V
- added copper zone on In2.Cu, net -5V
- added copper zone on In1.Cu, net GND
Other:
- board outline added: 118.5 x 68.5 mm

Commit message: layout and 3d models
Parts:
- R14, R15, R16, R8: moved to F.Cu
- moved R25 61.2 mm to (130.9, 99.7), turned to -90 degrees
- moved R24 55.8 mm to (125.0, 97.5)
- moved R23 52.7 mm to (122.4, 97.5)
- moved C35 46.8 mm to (137.6, 113.0)
- moved C34 43.7 mm to (134.4, 113.0), turned to 180 degrees
- moved C30 42.2 mm to (125.0, 93.9), turned to 180 degrees
- moved C32 42.1 mm to (130.4, 93.9), turned to 180 degrees
- moved C33 38.7 mm to (126.8, 96.1), turned to 90 degrees
- moved C31 35.3 mm to (125.6, 99.9), turned to -90 degrees
- moved C28 35.2 mm to (118.0, 91.8)
- moved D1 32.9 mm to (165.3, 75.6)
- moved R7 32.6 mm to (130.0, 73.3)
- moved C37 32.1 mm to (170.2, 98.6)
- moved U4 31.8 mm to (166.2, 88.6), turned to -90 degrees
- moved C4 31.7 mm to (169.8, 89.4), turned to 90 degrees
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Connections:
- net Net-(P1-RD+) renamed /MCU/RD+
- net Net-(P1-RD-) renamed /MCU/RD-
- net Net-(P1-TD+) renamed /MCU/TD+
- net Net-(P1-TD-) renamed /MCU/TD-
- J4 pad 1: /Model1605/CAL -> /Model1605/SIG-
- J4 pad 2: /Model1605/EXC+ -> /Model1605/SIG+
- J4 pad 4: /Model1605/SIG+ -> /Model1605/EXC+
- J4 pad 5: /Model1605/SIG- -> /Model1605/CAL
- U6 pad 10: unconnected-(U6-8_TX2_IN1-Pad10) -> /Hall2/HALL
- U6 pad 11: /MCU/A16 -> /Hall1/HALL
- U6 pad 20: unconnected-(U6-28_RX7-Pad20) -> /MCU/A16
- U6 pad 44: /MCU/A15 -> /MCU/CS_3
- U6 pad 45: /MCU/CS_3 -> /MCU/A15
Routing:
- net /MCU/+5V_USB: track 128.7 -> 47.4 mm
- net /MCU/MOSI: track 16.7 -> 78.0 mm, vias 0 -> 1
- net /MCU/MISO: track 0.00 -> 60.6 mm, vias 0 -> 2
- net /Hall1/HALL: track 0.00 -> 46.7 mm
- net /Model1605/MID_REF: track 0.00 -> 44.0 mm, vias 0 -> 3
- net /Model1605/BIAS_REF: track 0.00 -> 43.8 mm, vias 0 -> 3
- net /MCU/SCK: track 9.93 -> 52.4 mm, vias 0 -> 1
- net /Hall2/HALL: track 0.00 -> 37.0 mm
- net Net-(U10-VOUT): track 0.00 -> 32.2 mm
- net /MCU/RD-: track 0.00 -> 31.3 mm
- net /MCU/RD+: track 0.00 -> 30.1 mm
- net /MCU/TD-: track 0.00 -> 24.9 mm
- net Net-(P1-GRN-): track 0.00 -> 22.7 mm
- net /MCU/TD+: track 0.00 -> 22.1 mm
- net +12V: track 17.5 -> 3.14 mm
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- added copper zone on F.Cu, net +12V
- added copper zone on In2.Cu, net +3V3
- added copper zone on F.Cu, net +5V
- added copper zone on F.Cu, net -5V
- added copper zone on F.Cu, net /MCU/+5V_USB
- added copper zone on F.Cu, net /power/+5V_BUCK
- added copper zone on B.Cu, net GND
- added copper zone on F.Cu, net GND
Other:
- board size 118.5 x 68.5 mm -> 101.3 x 69 mm
