File: 03-engine_dyno/engine_dyno_v1/Model1605.kicad_sch (KiCad schematic)
At the start: 24 parts, among them J2 Screw_Terminal_01x02, J4 Screw_Terminal_01x05, U15 OPA192IDBVR, U7 INA827AIDGKR, U8 AD630ARZ, U9 ADS1120IPWR

Commit message: beginnings of a pcb
Parts:
- C13, C14, C15, C16, C17, C18, C21, C22, C23, C24: footprint (none) -> Capacitor_SMD:C_0402_1005Metric
- J2: footprint (none) -> TerminalBlock_RND:TerminalBlock_RND_205-00232_1x02_P5.08mm_Horizontal
- J4: footprint (none) -> TerminalBlock_RND:TerminalBlock_RND_205-00235_1x05_P5.08mm_Horizontal
- R10, R13, R14, R15, R16, R7, R8, R9: footprint (none) -> Resistor_SMD:R_0402_1005Metric
Changed lines of the file:
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@@
 			)
 		)
-		(property "Footprint" ""
+		(property "Footprint" "Resistor_SMD:R_0402_1005Metric"
 			(at 207.01 60.96 0)
 			(effects
@@
 			)
 		)
-		(property "Footprint" ""
+		(property "Footprint" "Capacitor_SMD:C_0402_1005Metric"
 			(at 29.21 100.33 0)
 			(effects
@@
 			)
 		)
-		(property "Footprint" ""
+		(property "Footprint" "TerminalBlock_RND:TerminalBlock_RND_205-00232_1x02_P5.08mm_Horizontal"
 			(at 36.83 72.39 0)
 			(effects
@@
 			)
 		)
-		(property "Footprint" ""
+		(property "Footprint" "Capacitor_SMD:C_0402_1005Metric"
 			(at 219.71 66.04 0)
 			(effects
@@
 			)
 		)
-		(property "Footprint" ""
+		(property "Footprint" "Resistor_SMD:R_0402_1005Metric"
 			(at 67.31 72.39 0)
 			(effects
@@
 			)
 		)
-		(property "Footprint" ""
+		(property "Footprint" "Capacitor_SMD:C_0402_1005Metric"
 			(at 29.21 110.49 0)
 			(effects
@@
 			)
 		)
-		(property "Footprint" ""
+		(property "Footprint" "Resistor_SMD:R_0402_1005Metric"
 			(at 77.47 77.47 0)
 			(effects
@@
 			)
 		)
-		(property "Footprint" ""
+		(property "Footprint" "Resistor_SMD:R_0402_1005Metric"
 			(at 67.31 69.85 0)
 			(effects
@@
 			)
 		)
-		(property "Footprint" ""
+		(property "Footprint" "Resistor_SMD:R_0402_1005Metric"
 			(at 77.47 64.77 0)
 			(effects
@@
 			)
 		)
-		(property "Footprint" ""
+		(property "Footprint" "TerminalBlock_RND:TerminalBlock_RND_205-00235_1x05_P5.08mm_Horizontal"
 			(at 36.83 90.17 0)
 			(effects
@@
 			)
 		)
-		(property "Footprint" ""
+		(property "Footprint" "Capacitor_SMD:C_0402_1005Metric"
 			(at 237.49 48.26 0)
 			(effects
@@
 			)
 		)
-		(property "Footprint" ""
+		(property "Footprint" "Capacitor_SMD:C_0402_1005Metric"
 			(at 259.08 106.68 0)
 			(effects
@@
 			)
 		)
-		(property "Footprint" ""
+		(property "Footprint" "Resistor_SMD:R_0402_1005Metric"
 			(at 250.19 58.42 0)
 			(effects
@@
 			)
 		)
-		(property "Footprint" ""
+		(property "Footprint" "Capacitor_SMD:C_0402_1005Metric"
 			(at 210.82 55.88 0)
 			(effects
@@
 			)
 		)
-		(property "Footprint" ""
+		(property "Footprint" "Capacitor_SMD:C_0402_1005Metric"
 			(at 237.49 68.58 0)
 			(effects
@@
 			)
 		)
-		(property "Footprint" ""
+		(property "Footprint" "Capacitor_SMD:C_0402_1005Metric"
 			(at 165.1 82.55 0)
 			(effects
@@
 			)
 		)
-		(property "Footprint" ""
+		(property "Footprint" "Capacitor_SMD:C_0402_1005Metric"
 			(at 259.08 95.25 0)
 			(effects
@@
 			)
 		)
-		(property "Footprint" ""
+		(property "Footprint" "Capacitor_SMD:C_0402_1005Metric"
 			(at 165.1 125.73 0)
 			(effects
@@
 			)
 		)
-		(property "Footprint" ""
+		(property "Footprint" "Resistor_SMD:R_0402_1005Metric"
 			(at 45.72 115.57 0)
 			(effects
@@
 			)
 		)
-		(property "Footprint" ""
+		(property "Footprint" "Resistor_SMD:R_0402_1005Metric"
 			(at 214.63 60.96 0)
 			(effects

Commit message: added math and changes to schematic
Connections:
- net CS renamed CS!
- net DIN renamed MOSI
- net DOUT/~DRDY renamed MISO
- net DRDY renamed A14
- net SCLK renamed SCK
- no-connect marks 9 -> 10
Other:
- note added: "Full-scale bridge output = sensitivity × excitation = 2 mV/V × 5 Vrms = 10 mVrms"
- note added: "G = 5 + 80kΩ/RG [INA827 datasheet] RG = 390 Ω → G = 5 + 80k/390 = 210 Vout = 10 mVrms × 210 = 2.10 Vrms ≈ 2.97 Vpk BW check: GBW ≈ 15 MHz; BW(G=210) ≈ 15M/210 ≈ 71 kHz ≫ 3.277 kHz ✓"
- note added: "Gain strap ±1: |G| = RF_eff / RA RF_eff = RF‖RB = 10k‖10k = 5kΩ ; RA = 5kΩ → |G| = 1 Demod DC (full-wave, phase-aligned) = (2/π)·Vpk = 0.637 × 2.97 = 1.89 V Ripple at 2×fc = 2 × 3.277 kHz = 6.55 kHz Output swing needed ≈ 2.97 Vpk (verify vs ±5V swing, Fig 9)"
- note added: "Vref = 2.048 V (internal), PGA = 1 → FSR = ±2.048 V LSB = 2·Vref / 2^16 = 4.096/65536 = 62.5 µV Full-scale DC 1.89 V → 1.89/2.048 = 92% FSR ✓ (fits, no clip) Codes @ full torque ≈ 1.89 V / 62.5 µV ≈ 30,200"
- note added: "fc = 1 / (2π·R·√(C1·C2)) ; Q = ½·√(C1/C2) [unity-gain SK, R1=R2=R] R = 16 kΩ, C1 = 150 nF, C2 = 68 nF fc = 1/(2π·16k·√(150n·68n)) = 98.5 Hz Q = ½·√(150/68) = 0.74 (≈Butterworth) Ripple reject @6.55 kHz: (fc/f)² = (98.5/6550)² → −72.9 dB"

Commit message: minor changes
Parts:
- R7: value 390 -> 1.5k
Connections:
- net AD630_OUT: no longer U8.15 (RF)
- net at U8.19 (CH_B-), U8.20 (CH_A-): now also U8.15 (RF)
Other:
- note added: "G = 5 + 80kΩ/RG [INA827 datasheet] RG = 390 Ω → G = 5 + 80k/390 = 210 Vout = 10 mVrms × 210 = 2.10 Vrms ≈ 2.97 Vpk BW check: GBW ≈ 15 MHz; BW(G=210) ≈ 15M/210 ≈ 71 kHz ≫ 3.277 kHz"
- note removed: "G = 5 + 80kΩ/RG [INA827 datasheet] RG = 390 Ω → G = 5 + 80k/390 = 210 Vout = 10 mVrms × 210 = 2.10 Vrms ≈ 2.97 Vpk BW check: GBW ≈ 15 MHz; BW(G=210) ≈ 15M/210 ≈ 71 kHz ≫ 3.277 kHz ✓"
Changed lines of the file:
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@@
 		)
 	)
-	(text "G = 5 + 80kΩ/RG            [INA827 datasheet]\nRG = 390 Ω → G = 5 + 80k/390 = 210\nVout = 10 mVrms × 210 = 2.10 Vrms ≈ 2.97 Vpk\nBW check: GBW ≈ 15 MHz; BW(G=210) ≈ 15M/210 ≈ 71 kHz ≫ 3.277 kHz  ✓"
+	(text "G = 5 + 80kΩ/RG            [INA827 datasheet]\nRG = 390 Ω → G = 5 + 80k/390 = 210\nVout = 10 mVrms × 210 = 2.10 Vrms ≈ 2.97 Vpk\nBW check: GBW ≈ 15 MHz; BW(G=210) ≈ 15M/210 ≈ 71 kHz ≫ 3.277 kHz"
 		(exclude_from_sim no)
-		(at 54.864 134.62 0)
+		(at 53.594 129.286 0)
 		(effects
 			(font
@@
 	)
 	(junction
+		(at 90.17 97.79)
+		(diameter 0)
+		(color 0 0 0 0)
+	)
+	(junction
 		(at 232.41 48.26)
 		(diameter 0)
@@
 	(wire
 		(pts
-			(xy 90.17 95.25) (xy 90.17 100.33)
+			(xy 90.17 95.25) (xy 90.17 97.79)
 		)
 		(stroke
@@
 	(wire
 		(pts
-			(xy 162.56 115.57) (xy 165.1 115.57)
+			(xy 162.56 115.57) (xy 179.07 115.57)
 		)
 		(stroke
@@
 	(wire
 		(pts
+			(xy 90.17 97.79) (xy 90.17 100.33)
+		)
+		(stroke
+			(width 0)
+			(type default)
+		)
+	)
+	(wire
+		(pts
 			(xy 245.11 40.64) (xy 245.11 58.42)
 		)
@@
 	(wire
 		(pts
+			(xy 90.17 97.79) (xy 86.36 97.79)
+		)
+		(stroke
+			(width 0)
+			(type default)
+		)
+	)
+	(wire
+		(pts
 			(xy 162.56 102.87) (xy 165.1 102.87)
 		)
@@
 	(wire
 		(pts
+			(xy 86.36 140.97) (xy 179.07 140.97)
+		)
+		(stroke
+			(width 0)
+			(type default)
+		)
+	)
+	(wire
+		(pts
 			(xy 201.93 60.96) (xy 204.47 60.96)
 		)
@@
 	(wire
 		(pts
+			(xy 179.07 140.97) (xy 179.07 115.57)
+		)
+		(stroke
+			(width 0)
+			(type default)
+		)
+	)
+	(wire
+		(pts
 			(xy 99.06 92.71) (xy 101.6 92.71)
 		)
@@
 	(wire
 		(pts
+			(xy 86.36 97.79) (xy 86.36 140.97)
+		)
+		(stroke
+			(width 0)
+			(type default)
+		)
+	)
+	(wire
+		(pts
 			(xy 165.1 120.65) (xy 167.64 120.65)
 		)
@@
 		)
 	)
-	(label "AD630_OUT"
-		(at 165.1 115.57 0)
-		(effects
-			(font
-				(size 1.27 1.27)
-			)
-			(justify left bottom)
-		)
-	)
 	(hierarchical_label "MOSI"
 		(shape input)
@@
 			)
 		)
-		(property "Value" "390"
+		(property "Value" "1.5k"
 			(at 43.18 116.8399 0)
 			(effects

Commit message: some more changes
Parts:
- removed J2: Screw_Terminal_01x02, TerminalBlock_RND:TerminalBlock_RND_205-00232_1x02_P5.08mm_Horizontal, symbol Connector:Screw_Terminal_01x02
Changed lines of the file:
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@@
 	)
 	(junction
-		(at 52.07 72.39)
-		(diameter 0)
-		(color 0 0 0 0)
-	)
-	(junction
 		(at 219.71 40.64)
 		(diameter 0)
@@
 	)
 	(junction
-		(at 54.61 69.85)
-		(diameter 0)
-		(color 0 0 0 0)
-	)
-	(junction
 		(at 232.41 68.58)
 		(diameter 0)
@@
 	(wire
 		(pts
-			(xy 41.91 72.39) (xy 52.07 72.39)
-		)
-		(stroke
-			(width 0)
-			(type default)
-		)
-	)
-	(wire
-		(pts
 			(xy 219.71 63.5) (xy 219.71 60.96)
 		)
@@
 	(wire
 		(pts
-			(xy 41.91 69.85) (xy 54.61 69.85)
-		)
-		(stroke
-			(width 0)
-			(type default)
-		)
-	)
-	(wire
-		(pts
 			(xy 52.07 87.63) (xy 52.07 72.39)
 		)
@@
 		)
 	)
-	(label "GEN+"
-		(at 46.99 72.39 0)
-		(effects
-			(font
-				(size 1.27 1.27)
-			)
-			(justify left bottom)
-		)
-	)
 	(label "AD630_OUT"
 		(at 99.06 115.57 180)
@@
 		)
 	)
-	(label "GEN-"
-		(at 46.99 69.85 0)
-		(effects
-			(font
-				(size 1.27 1.27)
-			)
-			(justify left bottom)
-		)
-	)
 	(label "AD630_OUT"
 		(at 165.1 102.87 0)
@@
 	)
 	(symbol
-		(lib_id "Connector:Screw_Terminal_01x02")
-		(at 36.83 72.39 180)
-		(unit 1)
-		(exclude_from_sim no)
-		(in_bom yes)
-		(on_board yes)
-		(dnp no)
-		(property "Reference" "J2"
-			(at 36.83 67.056 0)
-			(effects
-				(font
-					(size 1.27 1.27)
-				)
-			)
-		)
-		(property "Value" "Screw_Terminal_01x02"
-			(at 36.83 64.77 0)
-			(effects
-				(font
-					(size 1.27 1.27)
-				)
-			)
-		)
-		(property "Footprint" "TerminalBlock_RND:TerminalBlock_RND_205-00232_1x02_P5.08mm_Horizontal"
-			(at 36.83 72.39 0)
-			(effects
-				(font
-					(size 1.27 1.27)
-				)
-				(hide yes)
-			)
-		)
-		(property "Datasheet" "~"
-			(at 36.83 72.39 0)
-			(effects
-				(font
-					(size 1.27 1.27)
-				)
-				(hide yes)
-			)
-		)
-		(property "Description" "Generic screw terminal, single row, 01x02, script generated (kicad-library-utils/schlib/autogen/connector/)"
-			(at 36.83 72.39 0)
-			(effects
-				(font
-					(size 1.27 1.27)
-				)
-				(hide yes)
-			)
-		)
-		(pin "1"
-		)
-		(pin "2"
-		)
-		(instances
-			(project "engine_dyno_v1"
-				(path "/d283b024-74fa-4d4c-9089-b2007a8f756c/d7a598d2-e16c-4272-a780-ed8480e4996a"
-					(reference "J2")
-					(unit 1)
-				)
-			)
-		)
-	)
-	(symbol
 		(lib_id "power:GND")
 		(at 29.21 97.79 180)
@@
 		(on_board yes)
 		(dnp no)
-		(fields_autoplaced yes)
 		(property "Reference" "U8"
 			(at 132.08 80.01 0)

Commit message: layout and 3d models
Connections:
- net CAL: now also J4.5 (Pin_5); no longer J4.1 (Pin_1)
- net EXC+: now also J4.4 (Pin_4); no longer J4.2 (Pin_2)
- net SIG+: now also J4.2 (Pin_2); no longer J4.4 (Pin_4)
- net SIG-: now also J4.1 (Pin_1); no longer J4.5 (Pin_5)
Other:
- note added: "Full-scale bridge = 2.0 mV/V × 5 Vrms = 10 mVrms G = 5 + 80kΩ/RG ; RG = 1.5kΩ → G = 58 INA out = 10 mVrms × 58 = 0.58 Vrms = 0.82 Vpk AD630 input window (−Vs+4 to +Vs−1) = −1 V to +4 V Signal −0.82 to +0.82 V"
- note removed: "G = 5 + 80kΩ/RG [INA827 datasheet] RG = 390 Ω → G = 5 + 80k/390 = 210 Vout = 10 mVrms × 210 = 2.10 Vrms ≈ 2.97 Vpk BW check: GBW ≈ 15 MHz; BW(G=210) ≈ 15M/210 ≈ 71 kHz ≫ 3.277 kHz"
- moved on the sheet: J4
Changed lines of the file:
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@@
 		)
 	)
-	(text "G = 5 + 80kΩ/RG            [INA827 datasheet]\nRG = 390 Ω → G = 5 + 80k/390 = 210\nVout = 10 mVrms × 210 = 2.10 Vrms ≈ 2.97 Vpk\nBW check: GBW ≈ 15 MHz; BW(G=210) ≈ 15M/210 ≈ 71 kHz ≫ 3.277 kHz"
+	(text "Full-scale bridge = 2.0 mV/V × 5 Vrms = 10 mVrms\nG = 5 + 80kΩ/RG ;  RG = 1.5kΩ → G = 58\nINA out = 10 mVrms × 58 = 0.58 Vrms = 0.82 Vpk\nAD630 input window (−Vs+4 to +Vs−1) = −1 V to +4 V\nSignal −0.82 to +0.82 V"
 		(exclude_from_sim no)
 		(at 53.594 129.286 0)
@@
 	(wire
 		(pts
+			(xy 39.37 90.17) (xy 54.61 90.17)
+		)
+		(stroke
+			(width 0)
+			(type default)
+		)
+	)
+	(wire
+		(pts
+			(xy 39.37 92.71) (xy 50.8 92.71)
+		)
+		(stroke
+			(width 0)
+			(type default)
+		)
+	)
+	(wire
+		(pts
 			(xy 200.66 121.92) (xy 203.2 121.92)
 		)
@@
 	(wire
 		(pts
-			(xy 41.91 90.17) (xy 54.61 90.17)
-		)
-		(stroke
-			(width 0)
-			(type default)
-		)
-	)
-	(wire
-		(pts
 			(xy 162.56 115.57) (xy 179.07 115.57)
 		)
@@
 	(wire
 		(pts
+			(xy 39.37 95.25) (xy 50.8 95.25)
+		)
+		(stroke
+			(width 0)
+			(type default)
+		)
+	)
+	(wire
+		(pts
 			(xy 219.71 40.64) (xy 245.11 40.64)
 		)
@@
 	(wire
 		(pts
-			(xy 41.91 92.71) (xy 50.8 92.71)
-		)
-		(stroke
-			(width 0)
-			(type default)
-		)
-	)
-	(wire
-		(pts
 			(xy 238.76 101.6) (xy 259.08 101.6)
 		)
@@
 	(wire
 		(pts
-			(xy 41.91 87.63) (xy 52.07 87.63)
-		)
-		(stroke
-			(width 0)
-			(type default)
-		)
-	)
-	(wire
-		(pts
 			(xy 219.71 55.88) (xy 219.71 40.64)
 		)
@@
 	(wire
 		(pts
-			(xy 41.91 95.25) (xy 50.8 95.25)
-		)
-		(stroke
-			(width 0)
-			(type default)
-		)
-	)
-	(wire
-		(pts
 			(xy 232.41 48.26) (xy 232.41 50.8)
 		)
@@
 	(wire
 		(pts
-			(xy 41.91 85.09) (xy 46.99 85.09)
+			(xy 39.37 85.09) (xy 46.99 85.09)
 		)
 		(stroke
@@
 		(pts
 			(xy 29.21 102.87) (xy 50.8 102.87)
+		)
+		(stroke
+			(width 0)
+			(type default)
+		)
+	)
+	(wire
+		(pts
+			(xy 39.37 87.63) (xy 52.07 87.63)
 		)
 		(stroke
@@
 	(symbol
 		(lib_id "Connector:Screw_Terminal_01x05")
-		(at 36.83 90.17 0)
-		(mirror y)
+		(at 34.29 90.17 180)
 		(unit 1)
 		(exclude_from_sim no)
@@
 		(dnp no)
 		(property "Reference" "J4"
-			(at 36.83 82.55 0)
+			(at 34.29 97.79 0)
 			(effects
 				(font
@@
 		)
 		(property "Value" "Screw_Terminal_01x05"
-			(at 36.83 80.518 0)
+			(at 34.29 82.042 0)
 			(effects
 				(font
@@
 		)
 		(property "Footprint" "TerminalBlock_RND:TerminalBlock_RND_205-00235_1x05_P5.08mm_Horizontal"
-			(at 36.83 90.17 0)
+			(at 34.29 90.17 0)
 			(effects
 				(font
@@
 		)
 		(property "Datasheet" "~"
-			(at 36.83 90.17 0)
+			(at 34.29 90.17 0)
 			(effects
 				(font
@@
 		)
 		(property "Description" "Generic screw terminal, single row, 01x05, script generated (kicad-library-utils/schlib/autogen/connector/)"
-			(at 36.83 90.17 0)
-			(effects
-				(font
+			(at 34.29 90.17 0)
+			(effects
+				(font

Commit message: im aboutta release
Other:
- note added: "Gain strap ±1: |G| = RF_eff / RA RF_eff = RF‖RB = 10k‖10k = 5kΩ ; RA = 5kΩ → |G| = 1 Demod DC (full-wave, phase-aligned) = (2/π)·Vpk = 0.637 × 0.82 = 0.52 V Ripple at 2×fc = 2 × 3.277 kHz = 6.55 kHz Output swing needed ≈ 0.82 Vpk (verify vs ±5V swing, Fig 9)"
- note removed: "Gain strap ±1: |G| = RF_eff / RA RF_eff = RF‖RB = 10k‖10k = 5kΩ ; RA = 5kΩ → |G| = 1 Demod DC (full-wave, phase-aligned) = (2/π)·Vpk = 0.637 × 2.97 = 1.89 V Ripple at 2×fc = 2 × 3.277 kHz = 6.55 kHz Output swing needed ≈ 2.97 Vpk (verify vs ±5V swing, Fig 9)"
Changed lines of the file:
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@@
 		)
 	)
-	(text "Gain strap ±1: |G| = RF_eff / RA\nRF_eff = RF‖RB = 10k‖10k = 5kΩ ; RA = 5kΩ → |G| = 1\nDemod DC (full-wave, phase-aligned) = (2/π)·Vpk = 0.637 × 2.97 = 1.89 V\nRipple at 2×fc = 2 × 3.277 kHz = 6.55 kHz\nOutput swing needed ≈ 2.97 Vpk (verify vs ±5V swing, Fig 9)"
+	(text "Gain strap ±1: |G| = RF_eff / RA\nRF_eff = RF‖RB = 10k‖10k = 5kΩ ; RA = 5kΩ → |G| = 1\nDemod DC (full-wave, phase-aligned) = (2/π)·Vpk = 0.637 × 0.82 = 0.52 V\nRipple at 2×fc = 2 × 3.277 kHz = 6.55 kHz\nOutput swing needed ≈ 0.82 Vpk (verify vs ±5V swing, Fig 9)"
 		(exclude_from_sim no)
 		(at 132.588 134.112 0)
