File: 03-engine_dyno/engine_dyno_v1/TMNR-5KM.kicad_sch (KiCad schematic)
At the start: 24 parts, among them J3 Screw_Terminal_01x02, J6 Screw_Terminal_01x05, U10 INA827AIDGKR, U12 AD630ARZ, U13 ADS1120IPWR, U14 OPA192IDBVR

Commit message: beginnings of a pcb
Parts:
- C19, C27, C28, C29, C30, C31, C32, C33, C34, C35: footprint (none) -> Capacitor_SMD:C_0402_1005Metric
- J3: footprint (none) -> TerminalBlock_RND:TerminalBlock_RND_205-00232_1x02_P5.08mm_Horizontal
- J6: footprint (none) -> TerminalBlock_RND:TerminalBlock_RND_205-00235_1x05_P5.08mm_Horizontal
- R11, R19, R20, R21, R22, R23, R24, R25: footprint (none) -> Resistor_SMD:R_0402_1005Metric
Connections:
- net CS renamed CS!
Changed lines of the file:
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@@
 		)
 	)
-	(hierarchical_label "CS"
+	(hierarchical_label "CS!"
 		(shape input)
 		(at 200.66 102.87 180)
@@
 			)
 		)
-		(property "Footprint" ""
+		(property "Footprint" "Capacitor_SMD:C_0402_1005Metric"
 			(at 259.08 91.44 0)
 			(effects
@@
 			)
 		)
-		(property "Footprint" ""
+		(property "Footprint" "Capacitor_SMD:C_0402_1005Metric"
 			(at 29.21 96.52 0)
 			(effects
@@
 			)
 		)
-		(property "Footprint" ""
+		(property "Footprint" "Resistor_SMD:R_0402_1005Metric"
 			(at 77.47 60.96 0)
 			(effects
@@
 			)
 		)
-		(property "Footprint" ""
+		(property "Footprint" "Capacitor_SMD:C_0402_1005Metric"
 			(at 165.1 121.92 0)
 			(effects
@@
 			)
 		)
-		(property "Footprint" ""
+		(property "Footprint" "TerminalBlock_RND:TerminalBlock_RND_205-00235_1x05_P5.08mm_Horizontal"
 			(at 36.83 86.36 0)
 			(effects
@@
 			)
 		)
-		(property "Footprint" ""
+		(property "Footprint" "Resistor_SMD:R_0402_1005Metric"
 			(at 250.19 54.61 0)
 			(effects
@@
 			)
 		)
-		(property "Footprint" ""
+		(property "Footprint" "Capacitor_SMD:C_0402_1005Metric"
 			(at 219.71 62.23 0)
 			(effects
@@
 			)
 		)
-		(property "Footprint" ""
+		(property "Footprint" "Resistor_SMD:R_0402_1005Metric"
 			(at 67.31 66.04 0)
 			(effects
@@
 			)
 		)
-		(property "Footprint" ""
+		(property "Footprint" "Capacitor_SMD:C_0402_1005Metric"
 			(at 210.82 52.07 0)
 			(effects
@@
 			)
 		)
-		(property "Footprint" ""
+		(property "Footprint" "Capacitor_SMD:C_0402_1005Metric"
 			(at 237.49 64.77 0)
 			(effects
@@
 			)
 		)
-		(property "Footprint" ""
+		(property "Footprint" "Resistor_SMD:R_0402_1005Metric"
 			(at 67.31 68.58 0)
 			(effects
@@
 			)
 		)
-		(property "Footprint" ""
+		(property "Footprint" "Resistor_SMD:R_0402_1005Metric"
 			(at 207.01 57.15 0)
 			(effects
@@
 			)
 		)
-		(property "Footprint" ""
+		(property "Footprint" "Resistor_SMD:R_0402_1005Metric"
 			(at 45.72 111.76 0)
 			(effects
@@
 			)
 		)
-		(property "Footprint" ""
+		(property "Footprint" "Capacitor_SMD:C_0402_1005Metric"
 			(at 237.49 44.45 0)
 			(effects
@@
 			)
 		)
-		(property "Footprint" ""
+		(property "Footprint" "Capacitor_SMD:C_0402_1005Metric"
 			(at 165.1 78.74 0)
 			(effects
@@
 			)
 		)
-		(property "Footprint" ""
+		(property "Footprint" "TerminalBlock_RND:TerminalBlock_RND_205-00232_1x02_P5.08mm_Horizontal"
 			(at 36.83 68.58 0)
 			(effects
@@
 			)
 		)
-		(property "Footprint" ""
+		(property "Footprint" "Capacitor_SMD:C_0402_1005Metric"
 			(at 259.08 102.87 0)
 			(effects
@@
 			)
 		)
-		(property "Footprint" ""
+		(property "Footprint" "Resistor_SMD:R_0402_1005Metric"
 			(at 214.63 57.15 0)
 			(effects
@@
 			)
 		)
-		(property "Footprint" ""
+		(property "Footprint" "Capacitor_SMD:C_0402_1005Metric"
 			(at 29.21 106.68 0)
 			(effects
@@
 			)
 		)
-		(property "Footprint" ""
+		(property "Footprint" "Resistor_SMD:R_0402_1005Metric"
 			(at 77.47 73.66 0)
 			(effects

Commit message: added math and changes to schematic
Connections:
- net DIN renamed MOSI
- net DOUT/~DRDY renamed MISO
- net DRDY renamed A15
- net SCLK renamed SCK
- no-connect marks 9 -> 10
Other:
- note added: "Full-scale = 1.3 mV/V × 2 Vrms = 2.6 mVrms"
- note added: "G = 5 + 80kΩ/RG RG = 100 Ω → G = 5 + 80k/100 = 805 Vout = 2.6 mVrms × 805 = 2.09 Vrms ≈ 2.96 Vpk BW check: BW(G=805) ≈ 15M/805 ≈ 18.6 kHz > 5 kHz ✓ (−0.3 dB @ 5 kHz)"
- note added: "Vref = 2.048 V internal, PGA = 1 → FSR = ±2.048 V LSB = 62.5 µV Full-scale DC 1.88 V → 92% FSR ✓ Codes @ full torque ≈ 30,100"
- note added: "fc = 1/(2π·R·√(C1·C2)) ; Q = ½·√(C1/C2) R = 16 kΩ, C1 = 150 nF, C2 = 68 nF fc = 98.5 Hz ; Q = 0.74 Ripple reject @10 kHz: (98.5/10000)² → −80.3 dB"
- note added: "|G| = RF_eff/RA = (10k‖10k)/5k = 1 Demod DC = (2/π)·Vpk = 0.637 × 2.96 = 1.88 V Ripple at 2×fc = 2 × 5 kHz = 10 kHz"
Changed lines of the file:
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@@
 	(rectangle
 		(start 14.224 50.8)
-		(end 181.356 135.89)
+		(end 181.356 136.398)
 		(stroke
 			(width 0)
@@
 	)
 	(rectangle
-		(start 188.722 30.48)
+		(start 188.722 21.844)
 		(end 272.034 79.248)
 		(stroke
@@
 	(rectangle
 		(start 183.896 81.534)
-		(end 279.908 149.352)
+		(end 279.908 152.908)
 		(stroke
 			(width 0)
@@
 		)
 	)
+	(text "fc = 1/(2π·R·√(C1·C2)) ;  Q = ½·√(C1/C2)\nR = 16 kΩ, C1 = 150 nF, C2 = 68 nF\nfc = 98.5 Hz ; Q = 0.74\nRipple reject @10 kHz: (98.5/10000)² → −80.3 dB"
+		(exclude_from_sim no)
+		(at 227.838 27.178 0)
+		(effects
+			(font
+				(size 1.27 1.27)
+			)
+		)
+	)
+	(text "G = 5 + 80kΩ/RG\nRG = 100 Ω → G = 5 + 80k/100 = 805\nVout = 2.6 mVrms × 805 = 2.09 Vrms ≈ 2.96 Vpk\nBW check: BW(G=805) ≈ 15M/805 ≈ 18.6 kHz > 5 kHz  ✓  (−0.3 dB @ 5 kHz)"
+		(exclude_from_sim no)
+		(at 55.88 124.714 0)
+		(effects
+			(font
+				(size 1.27 1.27)
+			)
+		)
+	)
+	(text "Full-scale = 1.3 mV/V × 2 Vrms = 2.6 mVrms"
+		(exclude_from_sim no)
+		(at 37.592 195.326 0)
+		(effects
+			(font
+				(size 1.27 1.27)
+			)
+		)
+	)
+	(text "Vref = 2.048 V internal, PGA = 1 → FSR = ±2.048 V\nLSB = 62.5 µV\nFull-scale DC 1.88 V → 92% FSR  ✓\nCodes @ full torque ≈ 30,100"
+		(exclude_from_sim no)
+		(at 221.742 148.336 0)
+		(effects
+			(font
+				(size 1.27 1.27)
+			)
+		)
+	)
+	(text "|G| = RF_eff/RA = (10k‖10k)/5k = 1\nDemod DC = (2/π)·Vpk = 0.637 × 2.96 = 1.88 V\nRipple at 2×fc = 2 × 5 kHz = 10 kHz"
+		(exclude_from_sim no)
+		(at 131.572 124.968 0)
+		(effects
+			(font
+				(size 1.27 1.27)
+			)
+		)
+	)
 	(text "Instrumentational Amplifier and Demodulator"
 		(exclude_from_sim no)
-		(at 158.75 134.366 0)
+		(at 157.734 134.62 0)
 		(effects
 			(font
@@
 	(text "ADC\n"
 		(exclude_from_sim no)
-		(at 277.114 148.082 0)
+		(at 276.86 151.384 0)
 		(effects
 			(font
@@
 	)
 	(no_connect
+		(at 46.99 81.28)
+	)
+	(no_connect
 		(at 101.6 101.6)
 	)
@@
 		)
 	)
-	(hierarchical_label "DOUT{slash}~DRDY"
+	(hierarchical_label "MISO"
 		(shape input)
 		(at 241.3 105.41 0)
@@
 		)
 	)
-	(hierarchical_label "DIN"
+	(hierarchical_label "MOSI"
 		(shape input)
 		(at 200.66 107.95 180)
@@
 		)
 	)
-	(hierarchical_label "DRDY"
+	(hierarchical_label "A15"
 		(shape input)
 		(at 241.3 102.87 0)
@@
 		)
 	)
-	(hierarchical_label "SCLK"
+	(hierarchical_label "SCK"
 		(shape input)
 		(at 200.66 110.49 180)

Commit message: minor changes
Parts:
- R11: value 100 -> 390
Connections:
- net AD630_OUT: no longer U12.15 (RF)
- net at U12.19 (CH_B-), U12.20 (CH_A-): now also U12.15 (RF)
Changed lines of the file:
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@@
 	)
 	(junction
+		(at 90.17 93.98)
+		(diameter 0)
+		(color 0 0 0 0)
+	)
+	(junction
 		(at 29.21 99.06)
 		(diameter 0)
@@
 	(wire
 		(pts
-			(xy 90.17 91.44) (xy 90.17 96.52)
+			(xy 90.17 91.44) (xy 90.17 93.98)
 		)
 		(stroke
@@
 	(wire
 		(pts
+			(xy 87.63 93.98) (xy 87.63 132.08)
+		)
+		(stroke
+			(width 0)
+			(type default)
+		)
+	)
+	(wire
+		(pts
 			(xy 217.17 57.15) (xy 219.71 57.15)
 		)
@@
 	(wire
 		(pts
-			(xy 162.56 111.76) (xy 165.1 111.76)
+			(xy 162.56 111.76) (xy 179.07 111.76)
 		)
 		(stroke
@@
 	(wire
 		(pts
+			(xy 87.63 132.08) (xy 179.07 132.08)
+		)
+		(stroke
+			(width 0)
+			(type default)
+		)
+	)
+	(wire
+		(pts
 			(xy 41.91 91.44) (xy 50.8 91.44)
 		)
@@
 	(wire
 		(pts
+			(xy 90.17 93.98) (xy 87.63 93.98)
+		)
+		(stroke
+			(width 0)
+			(type default)
+		)
+	)
+	(wire
+		(pts
 			(xy 232.41 44.45) (xy 232.41 46.99)
 		)
@@
 	(wire
 		(pts
+			(xy 179.07 132.08) (xy 179.07 111.76)
+		)
+		(stroke
+			(width 0)
+			(type default)
+		)
+	)
+	(wire
+		(pts
 			(xy 99.06 88.9) (xy 101.6 88.9)
 		)
@@
 	(wire
 		(pts
+			(xy 90.17 93.98) (xy 90.17 96.52)
+		)
+		(stroke
+			(width 0)
+			(type default)
+		)
+	)
+	(wire
+		(pts
 			(xy 77.47 68.58) (xy 90.17 68.58)
 		)
@@
 		)
 	)
-	(label "AD630_OUT"
-		(at 165.1 111.76 0)
-		(effects
-			(font
-				(size 1.27 1.27)
-			)
-			(justify left bottom)
-		)
-	)
 	(hierarchical_label "MISO"
 		(shape input)
@@
 			)
 		)
-		(property "Value" "100"
+		(property "Value" "390"
 			(at 43.18 113.0299 0)
 			(effects

Commit message: some more changes
Parts:
- removed J3: Screw_Terminal_01x02, TerminalBlock_RND:TerminalBlock_RND_205-00232_1x02_P5.08mm_Horizontal, symbol Connector:Screw_Terminal_01x02
Changed lines of the file:
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@@
 	)
 	(junction
-		(at 52.07 68.58)
-		(diameter 0)
-		(color 0 0 0 0)
-	)
-	(junction
 		(at 90.17 93.98)
 		(diameter 0)
@@
 	)
 	(junction
-		(at 54.61 66.04)
-		(diameter 0)
-		(color 0 0 0 0)
-	)
-	(junction
 		(at 232.41 64.77)
 		(diameter 0)
@@
 	(wire
 		(pts
-			(xy 41.91 68.58) (xy 52.07 68.58)
-		)
-		(stroke
-			(width 0)
-			(type default)
-		)
-	)
-	(wire
-		(pts
 			(xy 219.71 59.69) (xy 219.71 57.15)
 		)
@@
 	(wire
 		(pts
-			(xy 41.91 66.04) (xy 54.61 66.04)
-		)
-		(stroke
-			(width 0)
-			(type default)
-		)
-	)
-	(wire
-		(pts
 			(xy 52.07 83.82) (xy 52.07 68.58)
 		)
@@
 		)
 	)
-	(label "GEN-"
-		(at 46.99 66.04 0)
-		(effects
-			(font
-				(size 1.27 1.27)
-			)
-			(justify left bottom)
-		)
-	)
 	(label "CAL"
 		(at 46.99 81.28 0)
@@
 		)
 	)
-	(label "GEN+"
-		(at 46.99 68.58 0)
-		(effects
-			(font
-				(size 1.27 1.27)
-			)
-			(justify left bottom)
-		)
-	)
 	(label "AD630_OUT"
 		(at 99.06 111.76 180)
@@
 					(unit 1)
 				)
-			)
-		)
-	)
-	(symbol
-		(lib_id "Connector:Screw_Terminal_01x02")
-		(at 36.83 68.58 180)
-		(unit 1)
-		(exclude_from_sim no)
-		(in_bom yes)
-		(on_board yes)
-		(dnp no)
-		(property "Reference" "J3"
-			(at 36.83 63.246 0)
-			(effects
-				(font
-					(size 1.27 1.27)
-				)
-			)
-		)
-		(property "Value" "Screw_Terminal_01x02"
-			(at 36.83 60.96 0)
-			(effects
-				(font
-					(size 1.27 1.27)
-				)
-			)
-		)
-		(property "Footprint" "TerminalBlock_RND:TerminalBlock_RND_205-00232_1x02_P5.08mm_Horizontal"
-			(at 36.83 68.58 0)
-			(effects
-				(font
-					(size 1.27 1.27)
-				)
-				(hide yes)
-			)
-		)
-		(property "Datasheet" "~"
-			(at 36.83 68.58 0)
-			(effects
-				(font
-					(size 1.27 1.27)
-				)
-				(hide yes)
-			)
-		)
-		(property "Description" "Generic screw terminal, single row, 01x02, script generated (kicad-library-utils/schlib/autogen/connector/)"
-			(at 36.83 68.58 0)
-			(effects
-				(font
-					(size 1.27 1.27)
-				)
-				(hide yes)
-			)
-		)
-		(pin "1"
-		)
-		(pin "2"
-		)
-		(instances
-			(project "engine_dyno_v1"
-				(path "/d283b024-74fa-4d4c-9089-b2007a8f756c/f78dad16-88c4-435c-93ac-abdbe766ab03"
-					(reference "J3")
-					(unit 1)
-				)

Commit message: layout and 3d models
Other:
- note added: "Full-scale bridge = 1.3 mV/V × 2 Vrms = 2.6 mVrms G = 5 + 80kΩ/RG ; RG = 390Ω → G = 210 INA out = 2.6 mVrms × 210 = 0.55 Vrms = 0.77 Vpk Signal −0.77 to +0.77 V"
- note removed: "G = 5 + 80kΩ/RG RG = 100 Ω → G = 5 + 80k/100 = 805 Vout = 2.6 mVrms × 805 = 2.09 Vrms ≈ 2.96 Vpk BW check: BW(G=805) ≈ 15M/805 ≈ 18.6 kHz > 5 kHz ✓ (−0.3 dB @ 5 kHz)"
Changed lines of the file:
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@@
 		)
 	)
-	(text "G = 5 + 80kΩ/RG\nRG = 100 Ω → G = 5 + 80k/100 = 805\nVout = 2.6 mVrms × 805 = 2.09 Vrms ≈ 2.96 Vpk\nBW check: BW(G=805) ≈ 15M/805 ≈ 18.6 kHz > 5 kHz  ✓  (−0.3 dB @ 5 kHz)"
+	(text "Full-scale bridge = 1.3 mV/V × 2 Vrms = 2.6 mVrms\nG = 5 + 80kΩ/RG ;  RG = 390Ω → G = 210\nINA out = 2.6 mVrms × 210 = 0.55 Vrms = 0.77 Vpk\nSignal −0.77 to +0.77 V"
 		(exclude_from_sim no)
 		(at 55.88 124.714 0)

Commit message: im aboutta release
Other:
- note added: "|G| = RF_eff/RA = (10k‖10k)/5k = 1 Demod DC = (2/π)·Vpk = 0.637 × 0.77 = 0.49 V Ripple at 2×fc = 2 × 5 kHz = 10 kHz"
- note removed: "|G| = RF_eff/RA = (10k‖10k)/5k = 1 Demod DC = (2/π)·Vpk = 0.637 × 2.96 = 1.88 V Ripple at 2×fc = 2 × 5 kHz = 10 kHz"
Changed lines of the file:
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@@
 		)
 	)
-	(text "|G| = RF_eff/RA = (10k‖10k)/5k = 1\nDemod DC = (2/π)·Vpk = 0.637 × 2.96 = 1.88 V\nRipple at 2×fc = 2 × 5 kHz = 10 kHz"
+	(text "|G| = RF_eff/RA = (10k‖10k)/5k = 1\nDemod DC = (2/π)·Vpk = 0.637 × 0.77 = 0.49 V\nRipple at 2×fc = 2 × 5 kHz = 10 kHz"
 		(exclude_from_sim no)
 		(at 131.572 124.968 0)
