File: 05-shock dyno/digitalprocessing.kicad_sch (KiCad schematic)
At the start: 9 parts, among them U1 INA827AIDGK, U2 AD5626BRMZ

Commit message: layout updates
Parts:
- C15: footprint (none) -> Capacitor_SMD:C_0402_1005Metric
- C31, C32, C33, R21, R22: footprint (none) -> Capacitor_SMD:C_0603_1608Metric
- R7: footprint (none) -> Capacitor_SMD:C_0805_2012Metric
- U1: footprint INA827AIDGK:SOP65P490X110-8N -> 00-footprints:INA827AIDGK
- U2: footprint AD5626BRMZ:SOP65P490X110-8N -> 00-footprints:AD5626BRMZ
Other:
- moved on the sheet: C15, U2

Commit message: v1 layout
Parts:
- renumbered C15 to C19, C31 to C20, C33 to C21, C32 to C22, R21 to R16, R22 to R17, R7 to R18, U2 to U3, U1 to U4
Connections:
- net GNDA renamed GND
- net amp_ref renamed force_-
- net force renamed force_+
- net loadcell+_f renamed loadcell_f+
- net loadcell-_f renamed loadcell_f-
