File: 05-shock dyno/power.kicad_sch (KiCad schematic)
At the start: 26 parts, among them IC2 SPX3819S-L_TR, IC3 TPS54331D, U3 REF5025ID

Commit message: layout updates
Parts:
- removed C20: 1nF, symbol Device:C
- removed C21: 47pF, symbol Device:C
- removed C22: 0.01uF, symbol Device:C
- removed C23, C24: 4.7uF, symbol Device:C
- removed C25: 0.01µF, symbol Device:C
- removed D3: B340, Diode_SMD:D_SMC, symbol Diode:B340
- removed IC3: TPS54331D, symbol TPS54331D:TPS54331D
- removed L1: 18uH, symbol Device:L
- removed R10: 10.2k, symbol Device:R
- removed R11: 1.96k, symbol Device:R
- removed R12: 29.4K, symbol Device:R
- removed R13: 332K, symbol Device:R
- removed R14: 68.1K, symbol Device:R
- added PS1: TSR_1-2450, TSR-1-24120, symbol TSR_1-2450:TSR_1-2450
- C16: value 0.1uF -> 10uF; footprint (none) -> Capacitor_SMD:C_1206_3216Metric
- C17, C28: footprint (none) -> Capacitor_SMD:C_0805_2012Metric
- C18: value 47uF -> 22uF; footprint (none) -> Capacitor_SMD:C_1210_3225Metric
- C19: value 47uF -> 0.1uF; footprint (none) -> Capacitor_SMD:C_1206_3216Metric
- C26, C29, R8, R9: footprint (none) -> Capacitor_SMD:C_0603_1608Metric
- D2: value D_Schottky -> B340B-13-F; footprint (none) -> 00-footprints:DIOM5336X250N
- IC2: footprint (none) -> 00-footprints:SOIC127P600X175-8N
- U3: footprint REF5025ID:SOIC127P599X175-8N -> 00-footprints:REF5025
Connections:
- net 11.1V: now also C16.2, C19.2, PS1.1 (VIN+)
- net 5V: now also PS1.3 (VOUT+); no longer C19.1
- net GNDA: now also PS1.2 (GND)
- net PGND: now also C16.1, C19.1; no longer C19.2
Other:
- note removed: "Vout: 4.96V"
- note removed: "rating over 5V"
- moved on the sheet: C17, C26, IC2, R8, R9

Commit message: v1 layout
Parts:
- PS1: footprint TSR-1-24120 -> 00-footprints:TSR-1-24120
- renumbered C17 to C12, C26 to C13, C16 to C14, C18 to C15, C19 to C16, C28 to C17, C29 to C18, D2 to D1, IC2 to IC3, R8 to R14, R9 to R15, U3 to U2
Connections:
- net PGND is gone; now on net GND: C14.1, C15.2, C16.1
- net GNDA renamed GND
