File: 05-shock dyno/sgprocessing.kicad_sch (KiCad schematic)
At the start: 17 parts, among them IC1 ADS131M04IPWR, IC4 OPA320AIDBVR

Commit message: v1 layout
Parts:
- renumbered C9 to C10, C10 to C11, C7 to C6, C1 to C7, C6 to C8, C8 to C9, IC4 to IC2, R1 to R10, R3 to R11, R4 to R12, R5 to R13, R15 to R8, R16 to R9
Connections:
- net GNDD is gone; now on net GND: C4.1, C5.2, IC1.19 (DGND)
- net PGND is gone; now on net GND: IC2.2 (V-)
- net pos_bias_nyq+ is gone; now on net position_nyq-: IC1.5 (AIN1N)
- net pos_bias_nyq- is gone; now on net position_nyq-: C10.2, C11.1, R13.2
- net position_nyq+: now also IC1.6 (AIN1P)
- net position_nyq-: no longer IC1.6 (AIN1P)
- net GNDA renamed GND
- net amp_ref renamed force_-
- net force renamed force_+
- net force_nyq+ renamed amp_ref_nyq+
