File: 05-shock dyno/ethernet.kicad_sch (KiCad schematic)
At the start: 9 parts, among them T1 749013011

Commit message: layout updates
Parts:
- C11, C12, C13, C2, R2, R6: footprint (none) -> Capacitor_SMD:C_0402_1005Metric
- C30: footprint (none) -> Capacitor_SMD:C_1206_3216Metric
- D1: footprint (none) -> Package_TO_SOT_SMD:SOT-23-5
- T1: footprint (none) -> 00-footprints:749013011
Changed lines of the file:
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@@
 			)
 		)
-		(property "Footprint" ""
+		(property "Footprint" "Capacitor_SMD:C_1206_3216Metric"
 			(at 176.53 92.4052 0)
 			(effects
@@
 			)
 		)
-		(property "Footprint" ""
+		(property "Footprint" "Capacitor_SMD:C_0402_1005Metric"
 			(at 167.64 99.568 90)
 			(effects
@@
 			)
 		)
-		(property "Footprint" ""
+		(property "Footprint" "Capacitor_SMD:C_0402_1005Metric"
 			(at 82.2452 105.41 0)
 			(effects
@@
 			)
 		)
-		(property "Footprint" ""
+		(property "Footprint" "Capacitor_SMD:C_0402_1005Metric"
 			(at 167.64 86.868 90)
 			(effects
@@
 			)
 		)
-		(property "Footprint" ""
+		(property "Footprint" "Capacitor_SMD:C_0402_1005Metric"
 			(at 82.2452 92.71 0)
 			(effects
@@
 			)
 		)
-		(property "Footprint" ""
+		(property "Footprint" "Capacitor_SMD:C_0402_1005Metric"
 			(at 89.8652 92.71 0)
 			(effects
@@
 			)
 		)
-		(property "Footprint" ""
+		(property "Footprint" "Package_TO_SOT_SMD:SOT-23-5"
 			(at 139.7 214.3 0)
 			(effects
@@
 			)
 		)
-		(property "Footprint" ""
+		(property "Footprint" "Capacitor_SMD:C_0402_1005Metric"
 			(at 89.8652 105.41 0)
 			(effects
@@
 			)
 		)
-		(property "Footprint" ""
+		(property "Footprint" "00-footprints:749013011"
 			(at 149.86 177.47 0)
 			(effects

Commit message: v1 layout
Parts:
- renumbered C2 to C23, C12 to C24, C11 to C25, C13 to C26, C30 to C27, D1 to D2, R2 to R19, R6 to R20
Connections:
- net GNDD renamed GND
