File: 05-shock dyno/05-shock dyno.kicad_sch (KiCad schematic)
At the start: 20 parts, among them J1 RJ45, J2 Conn_01x02, J3 Conn_01x03, J4 Conn_01x04, U4 Teensy4.1

Commit message: layout updates
Parts:
- removed H1, H2, H3, H4: MountingHole_Pad, symbol Mechanical:MountingHole_Pad
- removed J2: Conn_01x02, symbol Connector_Generic:Conn_01x02
- added J5: XT30PW-M, 00-footprints:AMASS_XT30PW-M, symbol XT30PW-M:XT30PW-M
- BT1: footprint (none) -> Battery:BatteryHolder_LINX_BAT-HLD-012-SMT
- C14, R17, R18, R19, R20, R23, R24, R25: footprint (none) -> Capacitor_SMD:C_0402_1005Metric
- C27: footprint (none) -> Capacitor_SMD:C_1206_3216Metric
- J1: footprint (none) -> Connector_RJ:RJ45_Amphenol_RJHSE5380
- J3: footprint (none) -> Connector_JST:JST_XH_B3B-XH-A_1x03_P2.50mm_Vertical
- J4: footprint (none) -> Connector_JST:JST_XH_B4B-XH-A_1x04_P2.50mm_Vertical
- NT2: footprint (none) -> NetTie:NetTie-2_SMD_Pad0.5mm
- U4: footprint 22XT_Main:Teensy41 -> 00-footprints:MODULE_DEV-16771
Connections:
- net 11.1V_Battery: now also J5.P
- net PGND: now also J5.N
Other:
- note removed: "Ethernet TVS Diode"

Commit message: v1 layout
Parts:
- removed NT2: NetTie_3_Tee, NetTie:NetTie-2_SMD_Pad0.5mm, symbol Device:NetTie_3_Tee
- J2: renamed from J1; footprint Connector_RJ:RJ45_Amphenol_RJHSE5380 -> 00-footprints:TE_RJ45-8N-B
- U1: renamed from U4; footprint 00-footprints:MODULE_DEV-16771 -> 00-footprints:Teensy41
- renumbered C27 to C1, C14 to C2, J3 to J1, J5 to J3, R17 to R1, R18 to R2, R19 to R3, R20 to R4, R23 to R5, R25 to R6, R24 to R7
Connections:
- net GNDA: no longer J1.3 (Pin_3), J4.2 (Pin_2)
- net GNDD: no longer BT1.2 (-), C1.1, C2.2, U1.1 (GND), U1.34 (GND), U1.47 (GND), U1.52 (GND), U1.64 (GND)
- net PGND: no longer J3.N
- new net GND: BT1.2 (-), C1.1, C2.2, J1.3 (Pin_3), J3.N, J4.2 (Pin_2), U1.1 (GND), U1.34 (GND), U1.47 (GND), U1.52 (GND), U1.64 (GND)

Commit message: v2 layout
Parts:
- added H1, H2, H3, H4: MountingHole_Pad, MountingHole:MountingHole_4.3mm_M4, symbol Mechanical:MountingHole_Pad
Connections:
- net GND: now also H1.1, H2.1, H3.1, H4.1

Commit message: fixes
Parts:
- H1, H2, H3, H4: footprint MountingHole:MountingHole_4.3mm_M4 -> MountingHole:MountingHole_4.3mm_M4_DIN965_Pad
Changed lines of the file:
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@@
 			)
 		)
-		(property "Footprint" "MountingHole:MountingHole_4.3mm_M4"
+		(property "Footprint" "MountingHole:MountingHole_4.3mm_M4_DIN965_Pad"
 			(at 248.92 26.67 0)
 			(effects
@@
 			)
 		)
-		(property "Footprint" "MountingHole:MountingHole_4.3mm_M4"
+		(property "Footprint" "MountingHole:MountingHole_4.3mm_M4_DIN965_Pad"
 			(at 240.03 26.67 0)
 			(effects
@@
 			)
 		)
-		(property "Footprint" "MountingHole:MountingHole_4.3mm_M4"
+		(property "Footprint" "MountingHole:MountingHole_4.3mm_M4_DIN965_Pad"
 			(at 250.19 35.56 0)
 			(effects
@@
 			)
 		)
-		(property "Footprint" "MountingHole:MountingHole_4.3mm_M4"
+		(property "Footprint" "MountingHole:MountingHole_4.3mm_M4_DIN965_Pad"
 			(at 240.03 35.56 0)
 			(effects
