File: 05-shock dyno/05-shock dyno.kicad_pcb (KiCad board)
At the start: 4 copper layers, 133.5 x 97.2 mm, 64 parts, among them IC1 ADS131M04IPWR, IC2 SPX3819S-L_TR, IC4 OPA320AIDBVR, J1 RJ45, J3 Conn_01x03, J4 Conn_01x04, J5 XT30PW-M, T1 749013011, U1 INA827AIDGK, U2 AD5626BRMZ, U3 REF5025ID, U4 Teensy4.1

Commit message: v1 layout
Parts:
- removed NT2: NetTie_3_Tee, NetTie:NetTie-2_SMD_Pad0.5mm
- J2: renamed from J1; footprint Connector_RJ:RJ45_Amphenol_RJHSE5380 -> 00-footprints:TE_RJ45-8N-B
- U1: renamed from U4; footprint 00-footprints:MODULE_DEV-16771 -> 00-footprints:Teensy41
- moved U2 160.9 mm to (65.7, 123.8), turned to 180 degrees
- moved R1 154.9 mm to (84.8, 64.2), turned to 90 degrees
- moved C1 154.7 mm to (86.5, 68.2), turned to 180 degrees
- moved C18 154.3 mm to (71.5, 123.0), turned to 90 degrees
- moved R2 153.4 mm to (87.0, 64.2), turned to 90 degrees
- moved R4 152.5 mm to (89.2, 64.2), turned to 90 degrees
- moved J2 151.9 mm to (69.8, 60.9)
- moved R3 150.2 mm to (91.0, 64.2), turned to 90 degrees
- moved C17 145.1 mm to (74.0, 123.0), turned to 90 degrees
- moved IC3 127.6 mm to (144.2, 101.5)
- moved C24 122.5 mm to (110.5, 50.8)
- moved C26 122.5 mm to (110.5, 52.8)
- moved C13 121.0 mm to (137.2, 102.7), turned to 90 degrees
- moved R20 118.2 mm to (101.8, 66.5), turned to -90 degrees
- moved R19 118.0 mm to (99.0, 66.5), turned to -90 degrees
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- renumbered C27 to C1, C9 to C10, C10 to C11, C17 to C12, C26 to C13, C16 to C14, C18 to C15, C19 to C16, C28 to C17, C29 to C18, C15 to C19, C14 to C2, C31 to C20, C33 to C21, C32 to C22, C2 to C23, C12 to C24, C11 to C25, C13 to C26, C30 to C27, C7 to C6, C1 to C7, C6 to C8, C8 to C9, D2 to D1, D1 to D2, IC4 to IC2, IC2 to IC3, J3 to J1, J5 to J3, R17 to R1, R1 to R10, R3 to R11, R4 to R12, R5 to R13, R8 to R14, R9 to R15, R21 to R16, R22 to R17, R7 to R18, R2 to R19, R18 to R2, R6 to R20, R19 to R3, R20 to R4, R23 to R5, R25 to R6, R24 to R7, R15 to R8, R16 to R9, U3 to U2, U2 to U3, U1 to U4
Connections:
- net amp_ref renamed force_-
- net force renamed force_+
- net force_nyq+ renamed amp_ref_nyq+
- net loadcell+_f renamed loadcell_f+
- net loadcell-_f renamed loadcell_f-
- BT1 pad 2: GNDD -> GND
- C1 pad 1: GNDD -> GND
- C10 pad 2: pos_bias_nyq- -> position_nyq-
- C11 pad 1: pos_bias_nyq- -> position_nyq-
- C11 pad 2: GNDA -> GND
- C12 pad 2: GNDA -> GND
- C14 pad 1: PGND -> GND
- C15 pad 2: PGND -> GND
- C16 pad 1: PGND -> GND
- C17 pad 2: GNDA -> GND
- C18 pad 2: GNDA -> GND
- C19 pad 2: GNDA -> GND
- C2 pad 2: GNDD -> GND
- C20 pad 1: GNDA -> GND
- C22 pad 1: GNDA -> GND
- C23 pad 2: GNDD -> GND
- C24 pad 2: GNDD -> GND
- C25 pad 2: GNDD -> GND
- C26 pad 2: GNDD -> GND
- C27 pad 1: GNDD -> GND
- C3 pad 2: GNDA -> GND
- C4 pad 1: GNDD -> GND
- C5 pad 2: GNDD -> GND
- C6 pad 1: GNDA -> GND
- C8 pad 2: GNDA -> GND
- C9 pad 1: GNDA -> GND
- D2 pad 2: GNDD -> GND
- IC1 pad 19: GNDD -> GND
- IC1 pad 2: GNDA -> GND
- IC1 pad 5: pos_bias_nyq+ -> position_nyq-
- IC1 pad 6: position_nyq- -> position_nyq+
- IC2 pad 2: PGND -> GND
- IC3 pad 5: GNDA -> GND
- IC3 pad 6: GNDA -> GND
- IC3 pad 7: GNDA -> GND
- IC3 pad 8: GNDA -> GND
- J1 pad 3: GNDA -> GND
- J3 pad N: PGND -> GND
- J4 pad 2: GNDA -> GND
- PS1 pad 2: GNDA -> GND
- R13 pad 1: GNDA -> GND
- R13 pad 2: pos_bias_nyq- -> position_nyq-
- R15 pad 2: GNDA -> GND
- R9 pad 1: GNDA -> GND
- U1 pad 1: GNDD -> GND
- U1 pad 34: GNDD -> GND
- U2 pad 4: GNDA -> GND
- U3 pad 7: GNDA -> GND
- U4 pad 5: GNDA -> GND
Routing:
- net 3v3: track 0.00 -> 89.0 mm, vias 0 -> 2
- net 3v3_teensy: track 0.00 -> 88.3 mm, vias 0 -> 4
- net GND: track 0.00 -> 67.1 mm, vias 0 -> 34
- net !LDAC: track 0.00 -> 51.9 mm, vias 0 -> 2
- net MOSI1: track 0.00 -> 48.9 mm
- net CLR_DAC: track 0.00 -> 43.6 mm, vias 0 -> 2
- net Net-(BT1-+): track 0.00 -> 40.2 mm
- net amp_ref_nyq-: track 0.00 -> 39.6 mm
- net amp_ref_nyq+: track 0.00 -> 39.4 mm
- net RD+: track 0.00 -> 38.9 mm
- net RD-: track 0.00 -> 38.8 mm
- net TX+: track 0.00 -> 38.4 mm
- net TX-: track 0.00 -> 38.3 mm
- net TD-: track 0.00 -> 38.1 mm
- net TD+: track 0.00 -> 38.1 mm
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- added copper zone on In2.Cu, net 5V
- added copper zone on In1.Cu, net GND
Other:
- board size 133.5 x 97.2 mm -> 101.5 x 89.2 mm

Commit message: v2 layout
Parts:
- added G***: BJR_LOGO, 22XT_Main:BJR_LOGO, B.Cu at (140.2, 45.4)
- added H1: MountingHole_Pad, MountingHole:MountingHole_4.3mm_M4, F.Cu at (148.5, 47.1)
- added H2: MountingHole_Pad, MountingHole:MountingHole_4.3mm_M4, F.Cu at (60.5, 47.1)
- added H3: MountingHole_Pad, MountingHole:MountingHole_4.3mm_M4, F.Cu at (148.5, 98.3)
- added H4: MountingHole_Pad, MountingHole:MountingHole_4.3mm_M4, F.Cu at (60.5, 98.3)
- moved J3 87.0 mm to (67.8, 54.8), turned to 0 degrees
- moved D1 57.7 mm to (78.7, 61.8), turned to 180 degrees
- moved C8 53.9 mm to (63.0, 87.2), turned to 90 degrees
- moved C27 53.0 mm to (146.8, 55.6), turned to 180 degrees
- moved R1 52.8 mm to (137.0, 56.4), turned to 0 degrees
- moved C1 51.7 mm to (135.8, 52.6), turned to 0 degrees
- moved C14 51.4 mm to (79.3, 51.4), turned to 0 degrees
- moved J2 49.7 mm to (119.0, 53.3), turned to 180 degrees
- moved R20 49.4 mm to (150.0, 55.8), turned to 90 degrees
- moved R2 48.0 mm to (134.4, 56.4), turned to 180 degrees
- moved R3 47.0 mm to (137.0, 54.8), turned to 0 degrees
- moved C6 46.6 mm to (68.6, 87.2)
- moved J4 46.5 mm to (61.5, 71.1), turned to 0 degrees
- moved J1 46.5 mm to (83.6, 91.4), turned to 180 degrees
- moved R11 46.3 mm to (64.6, 87.2), turned to -90 degrees
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Routing:
- net 3v3_teensy: track 88.3 -> 9.37 mm, vias 4 -> 1
- net 3v3: track 89.0 -> 16.3 mm, vias 2 -> 4
- net ADC_CLK: track 27.1 -> 72.5 mm, vias 0 -> 2
- net SCLK1: track 34.2 -> 72.4 mm, vias 0 -> 2
- net amp_ref_nyq-: track 39.6 -> 7.23 mm, vias 0 -> 1
- net MOSI1: track 48.9 -> 77.6 mm, vias 0 -> 1
- net amp_ref_nyq+: track 39.4 -> 67.2 mm, vias 0 -> 2
- net CS_ADC: track 26.8 -> 53.5 mm, vias 4 -> 2
- net CS_DAC: track 35.9 -> 21.4 mm, vias 2 -> 1
- net GND: track 67.1 -> 55.4 mm, vias 34 -> 39
- net Net-(T1-TXCT): track 13.6 -> 2.55 mm
- net loadcell_f+: track 19.6 -> 8.81 mm
- net CLR_DAC: track 43.6 -> 53.7 mm, vias 2 -> 1
- net loadcell_f-: track 19.7 -> 10.2 mm
- net 11.1V: track 25.8 -> 17.0 mm
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- added copper zone on In2.Cu, net 3v3
- added copper zone on F.Cu, net 3v3_teensy
Other:
- board size 101.5 x 89.2 mm -> 100 x 63.2 mm
- board text added: "2.5V"
- board text added: "3V3"
- board text added: "Blue Jay Racing @ JHU 23XT Shock Dyno V1"
- board text added: "GND"
- board text added: "Max Gao"
- board text added: "POS"
- board text added: "SIG+"
- board text added: "SIG-"
- board text added: "Sophie Noureddine"

Commit message: fixes
Parts:
- H1, H2, H3, H4: footprint MountingHole:MountingHole_4.3mm_M4 -> MountingHole:MountingHole_4.3mm_M4_DIN965_Pad
- moved C24 1.88 mm to (148.5, 70.6)
- moved C26 1.88 mm to (148.5, 72.2)
- moved C23 1.73 mm to (145.8, 70.6)
- moved C25 1.73 mm to (145.8, 72.0)
- moved R7 1.59 mm to (118.1, 85.0), turned to 0 degrees
- moved C3 1.00 mm to (119.3, 88.2)
- moved C4 0.40 mm to (131.8, 89.0)
Routing:
- net amp_ref_nyq-: track 7.23 -> 66.8 mm, vias 1 -> 2
- net MISO1: track 37.8 -> 45.5 mm, vias 0 -> 2
- net MOSI1: track 77.6 -> 85.0 mm, vias 1 -> 2
- net GND: track 55.4 -> 58.3 mm, vias 39 -> 41
- net position: track 7.91 -> 10.4 mm
- net 3v3: track 16.3 -> 17.3 mm
- net SYNC_ADC: track 19.4 -> 20.3 mm, vias 0 -> 2
- net Net-(T1-TCT): track 4.64 -> 5.39 mm
- net Net-(T1-RCT): track 4.63 -> 5.15 mm

Commit message: update
Parts:
- moved J3 0.35 mm to (67.8, 54.5)
Routing:
- net !LDAC: track 45.6 -> 48.7 mm, vias 1 -> 2
- net force_-: track 15.6 -> 18.7 mm, vias 0 -> 2
- net TX+: track 31.1 -> 32.7 mm
- net TX-: track 31.3 -> 32.8 mm
- net force_+: track 5.90 -> 7.21 mm
- net amp_ref_nyq-: track 66.8 -> 68.0 mm
- net amp_ref_nyq+: track 67.2 -> 68.1 mm
- net CLR_DAC: track 53.7 -> 54.3 mm
- net 3v3_teensy: vias 1 -> 0

Commit message: fix
Routing:
- net GND: track 58.4 -> 56.5 mm, vias 41 -> 40
- net amp_ref_nyq-: track 68.0 -> 66.8 mm
- net ADC_CLK: track 72.3 -> 72.9 mm
