File: 04-magnetometer/magnetometer_v1/magnetometer_v1.kicad_sch (KiCad schematic)
At the start: 29 parts, among them IC1 STM32F072CBT6, IC2 TMAG5170A1QDGKR, IC3 TCAN1042GVDRQ1, J1 Conn_02x03_Odd_Even, J2 USB4110-GF-A, SW1 SW_Push, SW2 SW_Push, U1 SPX3819M5-L-3-3/TR

Commit message: add manual power source selection
Parts:
- removed J1: Conn_02x03_Odd_Even, symbol Connector_Generic:Conn_02x03_Odd_Even
- added F1: 125 mA, symbol Device:Polyfuse
- added J1: Conn_01x04, symbol Connector_Generic:Conn_01x04
- added SW3: SW_SPDT, symbol Switch:SW_SPDT
Connections:
- net 5v: now also J1.1 (Pin_1), SW3.1 (A); no longer C13.2, C2.1, IC3.3 (VCC), U1.1 (VIN), U1.3 (EN)
- net CAN+: now also J1.2 (Pin_2)
- net CAN-: now also J1.3 (Pin_3)
- net GND: now also J1.4 (Pin_4)
- net VBUS: now reaches J2.A4-B9 (VBUS)
- net VBUS: now also J2.A9-B4 (VBUS), F1.2
- new net: F1.1, SW3.3 (C)
- new net VIN_SEL: C13.2, C2.1, IC3.3 (VCC), SW3.2 (B), U1.1 (VIN), U1.3 (EN)
- no-connect marks 33 -> 31
Other:
- note added: "5v to 3v3 ldo"
- note added: "dnp unless terminating node"
- note added: "stm32f072cb and caps"
- note removed: "5v to 3v3 LDO"
- note removed: "STM32F072CB and caps"
- moved on the sheet: C1, C13, C14, C15, C2, C3, IC3, J2, R2, R3, R4, R5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

Commit message: update power protection
Parts:
- removed F1: 125 mA, symbol Device:Polyfuse
- added D1: D_Schottky, symbol Device:D_Schottky
Connections:
- net 5v: now also D1.1 (K); no longer J1.1 (Pin_1)
- net VBUS: now also SW3.3 (C)
- new net: D1.2 (A), J1.1 (Pin_1)
Other:
- moved on the sheet: C1, C13, C14, C15, C2, C3, IC3, J1, J2, R2, R3, R4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

Commit message: update stm caps
Parts:
- removed C10: 1uF, symbol Device:C
- added C17: 100nF, symbol Device:C
- C7: value 10nF -> 4.7uF
Connections:
- net 3v3: now also C17.2
- net GND: now also C17.1
Other:
- note added: "pin 1, 9, 24, 36, 48"
- note removed: "pin 1, 48"
- note removed: "pin 24"
- note removed: "pin 36"
- note removed: "pin 9"
- moved on the sheet: C11, C16, C4, C5, C6, C7, C8, C9, R1, SW1, SW2, SW3

Commit message: pdr updates
Parts:
- removed J1: Conn_01x04, symbol Connector_Generic:Conn_01x04
- added C10: 4.7uF, symbol Device:C
- added D2: D_TVS_Dual_AAC, symbol Device:D_TVS_Dual_AAC
- added D3: LED, symbol Device:LED
- added J1: Conn_02x04_Counter_Clockwise, symbol Connector_Generic:Conn_02x04_Counter_Clockwise
- added JP1: Jumper_2_Bridged, symbol Jumper:Jumper_2_Bridged
- added R6: 330, symbol Device:R
- added R7, R8: 10k, symbol Device:R
Connections:
- net !CS: now also R7.2
- net 3v3: now also R6.2, R7.1, R8.2
- net 5v: now also J1.5 (Pin_5)
- net CAN+: now also D2.1 (A1), J1.2 (Pin_2), J1.6 (Pin_6)
- net CAN-: now also D2.2 (A2), J1.3 (Pin_3), J1.7 (Pin_7)
- net GND: now also C13.2, C10.2, D2.3 (common), D3.1 (K), J1.4 (Pin_4), J1.8 (Pin_8); no longer C13.1
- net VIN_SEL: now also C13.1, C10.1, JP1.2 (B); no longer C13.2, SW3.2 (B)
- net !ALERT: now reaches IC2.8 (ALERT_N)
- net !ALERT: now also IC1.10 (PA0), R8.1
- net at D1.2 (A): now also J1.1 (Pin_1)
- new net: D3.2 (A), R6.1
- new net: JP1.1 (A), SW3.2 (B)
- no-connect marks 31 -> 29
Other:
- moved on the sheet: C12, C13, C16, D1, IC1B, IC2, R1, SW1, SW2, SW3

Commit message: start layout
Parts:
- removed J1: Conn_02x04_Counter_Clockwise, symbol Connector_Generic:Conn_02x04_Counter_Clockwise
- added J1: Conn_02x04_Odd_Even, Connector_PinHeader_2.54mm:PinHeader_2x04_P2.54mm_Vertical, symbol Connector_Generic:Conn_02x04_Odd_Even
- C1, C10, C11, C12, C13, C14, C15, C16, C17, C2, C3, C4, C5, C6, C7, C8, C9: footprint (none) -> Capacitor_SMD:C_0402_1005Metric
- D1: footprint (none) -> Diode_SMD:D_SOD-323
- D2: footprint (none) -> Package_TO_SOT_SMD:SOT-23-3
- D3: footprint (none) -> LED_SMD:LED_0402_1005Metric
- IC1: footprint LQFP48-7x7mm -> mag-fp:STM32F072CBT6
- IC2: footprint (none) -> mag-fp:TMAG5170A2QDGKR
- IC3: footprint SOIC127P600X175-8N -> mag-fp:TCAN1042GVDRQ1
- J2: footprint (none) -> mag-fp:USB4110-GF-A_GCT
- JP1: footprint (none) -> Connector_PinHeader_2.54mm:PinHeader_1x02_P2.54mm_Vertical
- R1, R2, R3, R4, R5, R6, R7, R8: footprint (none) -> Resistor_SMD:R_0402_1005Metric
- SW1, SW2: footprint (none) -> mag-fp:SW_NANOT-AS_CNK
- SW3: footprint (none) -> mag-fp:SW_JS102011SCQN
- U1: footprint (none) -> mag-fp:SPX3819M5-L-3-3TR
Connections:
- net 5v: now also J1.8 (Pin_8)
- net CAN+: now also D2.2 (A2), J1.5 (Pin_5), J1.6 (Pin_6); no longer D2.1 (A1)
- net CAN-: now also D2.1 (A1), J1.3 (Pin_3), J1.4 (Pin_4); no longer D2.2 (A2)
- net GND: now also J1.2 (Pin_2), J1.7 (Pin_7)
- net at D1.2 (A): now also J1.1 (Pin_1)

Commit message: preliminary routing
Parts:
- removed C16: 10pF, Capacitor_SMD:C_0402_1005Metric, symbol Device:C
- removed R1: 10k, Resistor_SMD:R_0402_1005Metric, symbol Device:R
- removed SW1, SW2: SW_Push, mag-fp:SW_NANOT-AS_CNK, symbol Switch:SW_Push
- added C18: 10pF, Capacitor_SMD:C_0402_1005Metric, symbol Device:C
- added R9: 10k, Resistor_SMD:R_0402_1005Metric, symbol Device:R
- added U2, U3: NANOT100AS, mag-fp:SW_NANOT-AS_CNK, symbol mag-symbols:NANOT100AS
Connections:
- net 3v3: now also C18.2, U3.1
- net BOOT0: now also C18.1, R9.1, U3.2
- net GND: now also R9.2, U2.2
- net NRST: now also U2.1
Other:
- moved on the sheet: C12, D1, D2, D3, IC2, J1, JP1, R6, R7, R8, SW3
