File: 04-magnetometer/magnetometer_v1/magnetometer_v1.kicad_sch (KiCad schematic)
At the start: 38 parts, among them IC1 STM32F072CBT6, IC2 TMAG5170A1QDGKR, IC3 TCAN1042GVDRQ1, J1 Conn_02x04_Odd_Even, J2 USB4110-GF-A, SW3 SW_SPDT, U1 SPX3819M5-L-3-3/TR, U2 NANOT100AS, U3 NANOT100AS

Commit message: add mounting holes
Parts:
- added H1, H2, H3, H4: MountingHole_Pad, MountingHole:MountingHole_2.2mm_M2_DIN965_Pad, symbol Mechanical:MountingHole_Pad
Connections:
- net GND: now also H1.1, H2.1, H3.1, H4.1

Commit message: add power planes and modify layout
Connections:
- net VIN_JUMP: now reaches JP1.1 (A), SW3.2 (B)
Other:
- moved on the sheet: JP1
Changed lines of the file:
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@@
 	(wire
 		(pts
-			(xy 135.89 187.96) (xy 130.81 187.96)
+			(xy 158.75 187.96) (xy 153.67 187.96)
 		)
 		(stroke
@@
 	(wire
 		(pts
-			(xy 120.65 187.96) (xy 116.84 187.96)
-		)
-		(stroke
-			(width 0)
-			(type default)
-		)
-	)
-	(wire
-		(pts
 			(xy 107.95 168.91) (xy 113.03 168.91)
 		)
@@
 	(global_label "VIN_SEL"
 		(shape output)
-		(at 135.89 187.96 0)
+		(at 158.75 187.96 0)
+		(fields_autoplaced yes)
+		(effects
+			(font
+				(size 1.27 1.27)
+			)
+			(justify left)
+		)
+		(property "Intersheetrefs" "${INTERSHEET_REFS}"
+			(at 169.1133 187.96 0)
+			(effects
+				(font
+					(size 1.27 1.27)
+				)
+				(justify left)
+				(hide yes)
+			)
+		)
+	)
+	(global_label "VIN_JUMP"
+		(shape output)
+		(at 116.84 187.96 0)
 		(fields_autoplaced yes)
 		(effects
@@
 		)
 		(property "Intersheetrefs" "${INTERSHEET_REFS}"
-			(at 146.2533 187.96 0)
+			(at 128.8362 187.96 0)
 			(effects
 				(font
@@
 		)
 	)
+	(global_label "VIN_JUMP"
+		(shape input)
+		(at 143.51 187.96 180)
+		(fields_autoplaced yes)
+		(effects
+			(font
+				(size 1.27 1.27)
+			)
+			(justify right)
+		)
+		(property "Intersheetrefs" "${INTERSHEET_REFS}"
+			(at 131.5138 187.96 0)
+			(effects
+				(font
+					(size 1.27 1.27)
+				)
+				(justify right)
+				(hide yes)
+			)
+		)
+	)
 	(global_label "SCLK"
 		(shape output)
@@
 	(symbol
 		(lib_id "Jumper:Jumper_2_Bridged")
-		(at 125.73 187.96 0)
+		(at 148.59 187.96 0)
 		(unit 1)
 		(exclude_from_sim no)
@@
 		(fields_autoplaced yes)
 		(property "Reference" "JP1"
-			(at 125.73 182.88 0)
+			(at 148.59 182.88 0)
 			(effects
 				(font
@@
 		)
 		(property "Value" "Jumper_2_Bridged"
-			(at 125.73 185.42 0)
+			(at 148.59 185.42 0)
 			(effects
 				(font
@@
 		)
 		(property "Footprint" "Connector_PinHeader_2.54mm:PinHeader_1x02_P2.54mm_Vertical"
-			(at 125.73 187.96 0)
+			(at 148.59 187.96 0)
 			(effects
 				(font
@@
 		)
 		(property "Datasheet" "~"
-			(at 125.73 187.96 0)
+			(at 148.59 187.96 0)
 			(effects
 				(font
@@
 		)
 		(property "Description" "Jumper, 2-pole, closed/bridged"
-			(at 125.73 187.96 0)
+			(at 148.59 187.96 0)
 			(effects
 				(font

Commit message: made review changes
Changed lines of the file:
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@@
 	)
 	(junction
-		(at 114.3 33.02)
+		(at 109.22 34.29)
 		(diameter 0)
 		(color 0 0 0 0)
@@
 	)
 	(junction
-		(at 114.3 34.29)
-		(diameter 0)
-		(color 0 0 0 0)
-	)
-	(junction
 		(at 113.03 151.13)
 		(diameter 0)
@@
 	(wire
 		(pts
-			(xy 109.22 33.02) (xy 114.3 33.02)
-		)
-		(stroke
-			(width 0)
-			(type default)
-		)
-	)
-	(wire
-		(pts
 			(xy 143.51 118.11) (xy 143.51 119.38)
 		)
@@
 	(wire
 		(pts
-			(xy 114.3 33.02) (xy 114.3 34.29)
-		)
-		(stroke
-			(width 0)
-			(type default)
-		)
-	)
-	(wire
-		(pts
 			(xy 104.14 78.74) (xy 118.11 78.74)
 		)
@@
 	(wire
 		(pts
-			(xy 114.3 33.02) (xy 114.3 31.75)
-		)
-		(stroke
-			(width 0)
-			(type default)
-		)
-	)
-	(wire
-		(pts
 			(xy 251.46 118.11) (xy 248.92 118.11)
 		)
@@
 	(wire
 		(pts
-			(xy 109.22 34.29) (xy 114.3 34.29)
-		)
-		(stroke
-			(width 0)
-			(type default)
-		)
-	)
-	(wire
-		(pts
 			(xy 248.92 114.3) (xy 259.08 114.3)
 		)
@@
 	(wire
 		(pts
-			(xy 109.22 31.75) (xy 109.22 33.02)
+			(xy 109.22 31.75) (xy 109.22 34.29)
 		)
 		(stroke
@@
 	(wire
 		(pts
-			(xy 109.22 39.37) (xy 114.3 39.37)
-		)
-		(stroke
-			(width 0)
-			(type default)
-		)
-	)
-	(wire
-		(pts
 			(xy 215.9 142.24) (xy 215.9 147.32)
 		)
@@
 	(wire
 		(pts
-			(xy 114.3 34.29) (xy 114.3 39.37)
-		)
-		(stroke
-			(width 0)
-			(type default)
-		)
-	)
-	(wire
-		(pts
-			(xy 109.22 31.75) (xy 114.3 31.75)
-		)
-		(stroke
+			(xy 109.22 34.29) (xy 109.22 39.37)
+		)
+		(stroke

Commit message: generate gerber and bom
Parts:
- renumbered C18 to C16, JP1 to J3, R9 to R1, SW3 to U4
Changed lines of the file:
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@@
 		(dnp no)
 		(fields_autoplaced yes)
-		(property "Reference" "R9"
+		(property "Reference" "R1"
 			(at 148.59 113.03 90)
 			(effects
@@
 			(project "magnetometer_v1"
 				(path "/5ed894ec-debc-4dbe-bce4-314c8814571c"
-					(reference "R9")
+					(reference "R1")
 					(unit 1)
 				)
@@
 		(on_board yes)
 		(dnp no)
-		(property "Reference" "C18"
+		(property "Reference" "C16"
 			(at 125.73 130.048 90)
 			(effects
@@
 			(project "magnetometer_v1"
 				(path "/5ed894ec-debc-4dbe-bce4-314c8814571c"
-					(reference "C18")
+					(reference "C16")
 					(unit 1)
 				)
@@
 		(dnp no)
 		(fields_autoplaced yes)
-		(property "Reference" "JP1"
+		(property "Reference" "J3"
 			(at 148.59 182.88 0)
 			(effects
@@
 			(project "magnetometer_v1"
 				(path "/5ed894ec-debc-4dbe-bce4-314c8814571c"
-					(reference "JP1")
+					(reference "J3")
 					(unit 1)
 				)
@@
 		(dnp no)
 		(fields_autoplaced yes)
-		(property "Reference" "SW3"
+		(property "Reference" "U4"
 			(at 111.76 179.07 0)
 			(effects
@@
 			(project ""
 				(path "/5ed894ec-debc-4dbe-bce4-314c8814571c"
-					(reference "SW3")
+					(reference "U4")
 					(unit 1)
 				)
