File: MeshNetBoard(COPY).kicad_pcb (KiCad board)
At the start: 4 copper layers, 65 x 30 mm, 41 parts, among them J2 Conn_01x02, J3 Micro_SD_Card_Det_Hirose_DM3AT, Q1 Q_PMOS_GSD, SW1 SW_Push, SW2 SW_SPST, U1 XIAO-ESP32-S3-DIP, U2 TPS631000DRLR, U4 MAX9031AU, U5 MCP73831-2-OT

Commit message: help me
Parts:
- moved C6 57.6 mm to (154.1, 23.1)
- moved D6 57.6 mm to (157.6, 20.1)
- moved R13 57.6 mm to (162.1, 23.1)
- moved C7 57.6 mm to (158.8, 22.6)
- moved R9 57.6 mm to (153.4, 26.5)
- moved U1 57.6 mm to (141.7, 29.2)
- moved U5 57.6 mm to (157.5, 25.6)
- moved SW2 52.2 mm to (154.7, 51.9)
- moved JP1 44.0 mm to (65.5, 62.7)
- moved J2 35.9 mm to (138.4, 61.0)
- moved C5 35.0 mm to (28.8, 41.6)
- moved R8 35.0 mm to (25.6, 41.6)
- moved C4 35.0 mm to (31.1, 41.6)
- moved J3 35.0 mm to (30.5, 31.0)
- moved D1 30.1 mm to (77.9, 61.3)
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Routing:
- net +BATT: track 70.6 -> 1.77 mm
- net 3v3: track 51.5 -> 0.00 mm, vias 3 -> 0
- net GND: track 46.6 -> 0.00 mm, vias 13 -> 0
- net MOSI: track 43.1 -> 0.00 mm
- net MISO: track 35.8 -> 0.00 mm
- net SCK: track 34.0 -> 0.00 mm
- net SD_DATA: track 27.5 -> 0.00 mm
- net Net-(D2-A): track 25.4 -> 0.00 mm
- net GPIO44: track 21.4 -> 0.00 mm
- net Net-(J2-Pin_1): track 19.3 -> 0.00 mm
- net Net-(U4-+): track 15.5 -> 0.00 mm
- net 5v: track 14.1 -> 0.00 mm
- net Net-(JP1-B): track 12.4 -> 0.00 mm
- net Net-(Q1-D): track 11.2 -> 0.00 mm
- net LED4: track 8.14 -> 0.00 mm
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