File: WSG_1.0/WSG_1.0/WSG_ADC.kicad_sch (KiCad schematic)
At the start: 35 parts, among them J2 USB4110-GF-A, J4 Conn_01x02, U10 TPS22916BYFPR, U11 W25N04KVZEIR, U12 USBLC6-2SC6, U7 PQ25180YBGT, U8 TPS63802DLAR, U9 TPS7A2025PDBVR

Commit message: forgot to commit, started layout and started implementing sophie's/cyan's feedback for the schematic
Parts:
- C10, C12, C14, C15, C16, C17, C18, C19, C33, C8: footprint (none) -> Capacitor_SMD:C_01005_0402Metric_Pad0.57x0.30mm_HandSolder
- F1: footprint (none) -> Fuse:Fuse_0805_2012Metric_Pad1.15x1.40mm_HandSolder
- J2: footprint USB4110-GF-A_GCT -> Connector_USB:USB_C_Receptacle_GCT_USB4110
- J4: footprint (none) -> footprints:JST_S2B-PH-K-S_LF__SN_-2pin_male
- L1: footprint (none) -> Inductor_SMD:L_Coilcraft_XxL4020
- MOSFET1: footprint SOT23_DIO -> Package_TO_SOT_SMD:SOT-23
- R14, R20, R22, R23, R24, R25, R26, R31, R32, R33, R36, R37, R5: footprint (none) -> Resistor_SMD:R_01005_0402Metric_Pad0.57x0.30mm_HandSolder
- U10: footprint YFP0004ABAB -> footprints:IC_TPS22916BYFPR
- U11: footprint W25N04KVZEIR:IC_W25N04KVZEIR -> footprints:SON127P500X600X80-9N
- U7: footprint YBG0008-IPC_A -> footprints:IC_BQ25180YBGR
- U8: footprint DLA0010A -> Package_DFN_QFN:DFN-10-1EP_2x3mm_P0.5mm_EP0.64x2.4mm
- U9: footprint DBV0005A-IPC_A -> Package_TO_SOT_SMD:SOT-23-5
Changed lines of the file:
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@@
 			)
 		)
-		(property "Footprint" "USB4110-GF-A_GCT"
+		(property "Footprint" "Connector_USB:USB_C_Receptacle_GCT_USB4110"
 			(at 43.18 29.21 0)
 			(hide yes)
@@
 			)
 		)
-		(property "Footprint" ""
+		(property "Footprint" "footprints:JST_S2B-PH-K-S_LF__SN_-2pin_male"
 			(at 176.53 25.4 0)
 			(hide yes)
@@
 			)
 		)
-		(property "Footprint" ""
+		(property "Footprint" "Resistor_SMD:R_01005_0402Metric_Pad0.57x0.30mm_HandSolder"
 			(at 171.45 133.858 90)
 			(hide yes)
@@
 			)
 		)
-		(property "Footprint" ""
+		(property "Footprint" "Fuse:Fuse_0805_2012Metric_Pad1.15x1.40mm_HandSolder"
 			(at 96.52 7.62 0)
 			(hide yes)
@@
 			)
 		)
-		(property "Footprint" "SOT23_DIO"
+		(property "Footprint" "Package_TO_SOT_SMD:SOT-23"
 			(at 33.02 83.82 0)
 			(hide yes)
@@
 			)
 		)
-		(property "Footprint" ""
+		(property "Footprint" "Capacitor_SMD:C_01005_0402Metric_Pad0.57x0.30mm_HandSolder"
 			(at 191.4652 66.04 0)
 			(hide yes)
@@
 			)
 		)
-		(property "Footprint" ""
+		(property "Footprint" "Resistor_SMD:R_01005_0402Metric_Pad0.57x0.30mm_HandSolder"
 			(at 21.082 27.94 90)
 			(hide yes)
@@
 			)
 		)
-		(property "Footprint" ""
+		(property "Footprint" "Capacitor_SMD:C_01005_0402Metric_Pad0.57x0.30mm_HandSolder"
 			(at 171.1452 121.92 0)
 			(hide yes)
@@
 			)
 		)
-		(property "Footprint" ""
+		(property "Footprint" "Capacitor_SMD:C_01005_0402Metric_Pad0.57x0.30mm_HandSolder"
 			(at 248.6152 151.13 0)
 			(hide yes)
@@
 			)
 		)
-		(property "Footprint" ""
+		(property "Footprint" "Capacitor_SMD:C_01005_0402Metric_Pad0.57x0.30mm_HandSolder"
 			(at 228.2952 85.09 0)
 			(hide yes)
@@
 			)
 		)
-		(property "Footprint" ""
+		(property "Footprint" "Capacitor_SMD:C_01005_0402Metric_Pad0.57x0.30mm_HandSolder"
 			(at 129.2352 121.92 0)
 			(hide yes)
@@
 			)
 		)
-		(property "Footprint" ""
+		(property "Footprint" "Resistor_SMD:R_01005_0402Metric_Pad0.57x0.30mm_HandSolder"
 			(at 103.632 35.56 90)
 			(hide yes)
@@
 			)
 		)
-		(property "Footprint" ""
+		(property "Footprint" "Capacitor_SMD:C_01005_0402Metric_Pad0.57x0.30mm_HandSolder"
 			(at 163.5252 168.91 0)
 			(hide yes)
@@
 			)
 		)
-		(property "Footprint" "DBV0005A-IPC_A"
+		(property "Footprint" "Package_TO_SOT_SMD:SOT-23-5"
 			(at 210.82 151.13 0)
 			(hide yes)
@@
 			)
 		)
-		(property "Footprint" "YBG0008-IPC_A"
+		(property "Footprint" "footprints:IC_BQ25180YBGR"
 			(at 129.54 121.92 0)
 			(hide yes)
@@
 			)
 		)
-		(property "Footprint" ""
+		(property "Footprint" "Capacitor_SMD:C_01005_0402Metric_Pad0.57x0.30mm_HandSolder"
 			(at 209.2452 151.13 0)
 			(hide yes)
@@
 			)
 		)
-		(property "Footprint" ""
+		(property "Footprint" "Resistor_SMD:R_01005_0402Metric_Pad0.57x0.30mm_HandSolder"
 			(at 39.37 183.642 90)
 			(hide yes)
@@
 			)
 		)
-		(property "Footprint" ""
+		(property "Footprint" "Resistor_SMD:R_01005_0402Metric_Pad0.57x0.30mm_HandSolder"
 			(at 185.42 102.108 90)
 			(hide yes)
@@
 			)
 		)
-		(property "Footprint" ""
+		(property "Footprint" "Resistor_SMD:R_01005_0402Metric_Pad0.57x0.30mm_HandSolder"
 			(at 90.678 153.67 90)
 			(hide yes)
@@
 			)
 		)
-		(property "Footprint" ""
+		(property "Footprint" "Resistor_SMD:R_01005_0402Metric_Pad0.57x0.30mm_HandSolder"
 			(at 175.26 60.198 90)
 			(hide yes)
@@
 			)
 		)
-		(property "Footprint" ""
+		(property "Footprint" "Inductor_SMD:L_Coilcraft_XxL4020"
 			(at 50.8 105.41 0)
 			(hide yes)
@@
 			)
 		)
-		(property "Footprint" "W25N04KVZEIR:IC_W25N04KVZEIR"
+		(property "Footprint" "footprints:SON127P500X600X80-9N"
 			(at 138.43 179.07 0)
 			(hide yes)
@@
 			)
 		)
-		(property "Footprint" ""
+		(property "Footprint" "Capacitor_SMD:C_01005_0402Metric_Pad0.57x0.30mm_HandSolder"
 			(at 182.5752 127 0)
 			(hide yes)
@@
 			)
 		)
-		(property "Footprint" ""
+		(property "Footprint" "Resistor_SMD:R_01005_0402Metric_Pad0.57x0.30mm_HandSolder"
 			(at 90.678 143.51 90)
 			(hide yes)
@@
 			)
 		)
-		(property "Footprint" "YFP0004ABAB"
+		(property "Footprint" "footprints:IC_TPS22916BYFPR"
 			(at 63.5 180.34 0)
 			(hide yes)
@@
 			)
 		)
-		(property "Footprint" ""
+		(property "Footprint" "Resistor_SMD:R_01005_0402Metric_Pad0.57x0.30mm_HandSolder"
 			(at 182.118 62.23 90)
 			(hide yes)
@@
 			)
 		)
-		(property "Footprint" ""
+		(property "Footprint" "Capacitor_SMD:C_01005_0402Metric_Pad0.57x0.30mm_HandSolder"
 			(at 84.7852 128.27 0)
 			(hide yes)
@@
 			)
 		)
-		(property "Footprint" ""
+		(property "Footprint" "Capacitor_SMD:C_01005_0402Metric_Pad0.57x0.30mm_HandSolder"
 			(at 23.8252 128.27 0)
 			(hide yes)
@@
 			)
 		)
-		(property "Footprint" ""
+		(property "Footprint" "Resistor_SMD:R_01005_0402Metric_Pad0.57x0.30mm_HandSolder"
 			(at 185.42 90.678 90)
 			(hide yes)
@@
 			)
 		)
-		(property "Footprint" ""
+		(property "Footprint" "Resistor_SMD:R_01005_0402Metric_Pad0.57x0.30mm_HandSolder"
 			(at 185.42 110.998 90)
 			(hide yes)
@@
 			)
 		)
-		(property "Footprint" ""
+		(property "Footprint" "Resistor_SMD:R_01005_0402Metric_Pad0.57x0.30mm_HandSolder"
 			(at 25.4 85.598 90)
 			(hide yes)
@@
 			)
 		)
-		(property "Footprint" ""
+		(property "Footprint" "Resistor_SMD:R_01005_0402Metric_Pad0.57x0.30mm_HandSolder"
 			(at 219.71 79.248 90)
 			(hide yes)
@@
 			)
 		)
-		(property "Footprint" "DLA0010A"
+		(property "Footprint" "Package_DFN_QFN:DFN-10-1EP_2x3mm_P0.5mm_EP0.64x2.4mm"
 			(at 52.07 135.89 0)
 			(hide yes)

Commit message: placement mostly done
Parts:
- removed J2: USB4110-GF-A, Connector_USB:USB_C_Receptacle_GCT_USB4110, symbol my-symbols:USB4110-GF-A
- removed R22, R23: 5.1k, Resistor_SMD:R_01005_0402Metric_Pad0.57x0.30mm_HandSolder, symbol Device:R
- added C34: 1uF, Capacitor_SMD:C_01005_0402Metric_Pad0.57x0.30mm_HandSolder, symbol Device:C
- added J2: USB_C_Receptacle_USB2.0_16P, Connector_USB:USB_C_Receptacle_GCT_USB4110, symbol Connector:USB_C_Receptacle_USB2.0_16P
- added R39: 100k, Resistor_SMD:R_01005_0402Metric_Pad0.57x0.30mm_HandSolder, symbol Device:R
- added R40, R41: 5.1k, Resistor_SMD:R_01005_0402Metric_Pad0.57x0.30mm_HandSolder, symbol Device:R
- L1: footprint Inductor_SMD:L_Coilcraft_XxL4020 -> (none)
- U10: value TPS22916BYFPR -> TPS22916CYFPR
Connections:
- net 3V3: now also C34.2
- net CHG_INT: now also U7.A1 (INT_N); no longer U7.1 (INT_N)
- net GND: now also U7.D2 (GND), C34.1, J2.A1 (GND), J2.A12 (GND), J2.B1 (GND), J2.B12 (GND), J2.SH (SHIELD), R39.1, R40.1, R41.1; no longer J4.2 (Pin_2), U7.8 (GND), U8.2 (MODE)
- net I2C_SCL: now also U7.B1 (SCL); no longer U7.3 (SCL)
- net I2C_SDA: now also U7.C1 (SDA); no longer U7.5 (SDA)
- net SYS: now also U7.B2 (SYS); no longer U7.4 (SYS)
- net USB_DM: now also J2.A7 (D-), J2.B7 (D-)
- net USB_DP: now also J2.A6 (D+), J2.B6 (D+)
- net VBAT: now also U7.C2 (BAT); no longer U7.6 (BAT)
- net VBUS: now also J2.A4 (VBUS), J2.A9 (VBUS), J2.B4 (VBUS), J2.B9 (VBUS)
- net VIN_P: now also U7.A2 (IN); no longer U7.2 (IN)
- net at R14.1: now also U7.D1 (TS_MR); no longer U7.7 (TS_MR)
- new net: J2.B5 (CC2), R41.2
- new net: J2.A5 (CC1), R40.2
- new net BATT_N: J4.2 (Pin_2)
- new net BUCK_MODE: R39.2, U8.2 (MODE)
Other:
- note added: "load switch B faster slew time, C smoother"
- note removed: "load switch"

Commit message: sketch pcb finished
Parts:
- removed R31: 1M, Resistor_SMD:R_01005_0402Metric_Pad0.57x0.30mm_HandSolder, symbol Device:R
- added FB1: 0, Resistor_SMD:R_0402_1005Metric_Pad0.72x0.64mm_HandSolder, symbol Device:R
- C10, C12, C16, C17, C18, C19, C33, C34, C8: footprint Capacitor_SMD:C_01005_0402Metric_Pad0.57x0.30mm_HandSolder -> Capacitor_SMD:C_0402_1005Metric_Pad0.74x0.62mm_HandSolder
- C14: value 10uF -> 22uF; footprint Capacitor_SMD:C_01005_0402Metric_Pad0.57x0.30mm_HandSolder -> Capacitor_SMD:C_0603_1608Metric_Pad1.08x0.95mm_HandSolder; MPN (none) -> GRM188R60J226MEA0J
- C15: footprint Capacitor_SMD:C_01005_0402Metric_Pad0.57x0.30mm_HandSolder -> Capacitor_SMD:C_0603_1608Metric_Pad1.08x0.95mm_HandSolder; MPN (none) -> GRM188R60J226MEA0J
- F1: value Polyfuse -> 0ZCJ0075AF2E; footprint Fuse:Fuse_0805_2012Metric_Pad1.15x1.40mm_HandSolder -> Fuse:Fuse_1206_3216Metric
- L1: footprint (none) -> Inductor_SMD:L_Coilcraft_XxL4020; MPN (none) -> XFL4020-471MEC
- R14, R24, R25, R26, R33, R36, R37, R39, R40, R41, R5: footprint Resistor_SMD:R_01005_0402Metric_Pad0.57x0.30mm_HandSolder -> Resistor_SMD:R_0402_1005Metric_Pad0.72x0.64mm_HandSolder
- R20: value 560k -> 511k; footprint Resistor_SMD:R_01005_0402Metric_Pad0.57x0.30mm_HandSolder -> Resistor_SMD:R_0402_1005Metric_Pad0.72x0.64mm_HandSolder
- R32: value 100k -> 91k; footprint Resistor_SMD:R_01005_0402Metric_Pad0.57x0.30mm_HandSolder -> Resistor_SMD:R_0402_1005Metric_Pad0.72x0.64mm_HandSolder
- U11: footprint footprints:SON127P500X600X80-9N -> footprints:IC_W25N04KVZEIR
- U7: value PQ25180YBGT -> BQ25180YBGR
- U8: footprint Package_DFN_QFN:DFN-10-1EP_2x3mm_P0.5mm_EP0.64x2.4mm -> footprints:DLA0010A
Connections:
- net 3V3: now also FB1.2; no longer C34.2, U10.A2 (VIN)
- new net: C34.2, FB1.1, U10.A2 (VIN)
Other:
- note added: "VBAT_SENSE = VBAT/2"
- note added: "firmware constant = 2x"
- note added: "volatile registers watchdog enabled by default (160s)"
