File: WSG_1.0/WSG_1.0/WSG_ESP.kicad_sch (KiCad schematic)
At the start: 1 part, among them U12 ESP32-S3

Commit message: finished schematic
Parts:
- removed U12: ESP32-S3, Package_DFN_QFN:QFN-56-1EP_7x7mm_P0.4mm_EP4x4mm, symbol MCU_Espressif:ESP32-S3
- added C30: 1uF, symbol Device:C
- added C31: 0.1uF, symbol Device:C
- added C32: 10uF, symbol Device:C
- added R29, R30: 10k, symbol Device:R
- added SW1, SW2: SW_Push, symbol Switch:SW_Push
- added U13: ESP32-S3-MINI-1, RF_Module:ESP32-S2-MINI-1, symbol RF_Module:ESP32-S3-MINI-1
Connections:
- new net: R30.2, SW1.2, U13.4 (IO0)
- new net 3V3: C31.1, C32.1, R29.1, R30.1, U13.3 (3V3)
- new net ADC_CS: U13.15 (IO11)
- new net ADC_DRDY: U13.12 (IO8)
- new net ADC_MISO: U13.11 (IO7)
- new net ADC_MOSI: U13.10 (IO6)
- new net ADC_RST: U13.13 (IO9)
- new net ADC_SCLK: U13.9 (IO5)
- new net AFE_EN: U13.33 (IO37)
- new net CHG_INT: U13.32 (IO36)
- new net DAC_CS: U13.8 (IO4)
- new net EN: C30.2, R29.2, SW2.1, U13.45 (EN)
- new net EXC_EN: U13.34 (IO38)
- new net FLASH_CLK: U13.25 (IO21)
- new net FLASH_CS: U13.14 (IO10)
- new net FLASH_MISO: U13.28 (IO33)
- new net FLASH_MOSI: U13.26 (IO26)
- new net GND: C30.1, C31.2, C32.2, SW1.1, SW2.2, U13.1 (GND), U13.2 (GND), U13.42 (GND), U13.43 (GND), U13.46 (GND), U13.47 (GND), U13.48 (GND), U13.49 (GND), U13.50 (GND), U13.51 (GND), U13.52 (GND), U13.53 (GND), U13.54 (GND), U13.55 (GND), U13.56 (GND), U13.57 (GND), U13.58 (GND), U13.59 (GND), U13.60 (GND), U13.61 (GND), U13.62 (GND), U13.63 (GND), U13.64 (GND), U13.65 (GND)
- new net I2C_SCL: U13.31 (IO35)
- new net I2C_SDA: U13.29 (IO34)
- new net SHUNT_EN: U13.35 (IO39)
- new net USB_DM: U13.23 (USB_D-)
- new net USB_DP: U13.24 (USB_D+)
- new net VBAT_SENSE: U13.6 (IO2)
- no-connect marks 0 -> 18

Commit message: forgot to commit, started layout and started implementing sophie's/cyan's feedback for the schematic
Parts:
- C30, C31, C32: footprint (none) -> Capacitor_SMD:C_01005_0402Metric_Pad0.57x0.30mm_HandSolder
- R29, R30: footprint (none) -> Resistor_SMD:R_01005_0402Metric_Pad0.57x0.30mm_HandSolder
- SW1, SW2: footprint (none) -> Button_Switch_SMD:SW_DIP_SPSTx01_Slide_6.7x4.1mm_W6.73mm_P2.54mm_LowProfile_JPin
Changed lines of the file:
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@@
 			)
 		)
-		(property "Footprint" ""
+		(property "Footprint" "Button_Switch_SMD:SW_DIP_SPSTx01_Slide_6.7x4.1mm_W6.73mm_P2.54mm_LowProfile_JPin"
 			(at 132.08 55.88 0)
 			(hide yes)
@@
 			)
 		)
-		(property "Footprint" ""
+		(property "Footprint" "Resistor_SMD:R_01005_0402Metric_Pad0.57x0.30mm_HandSolder"
 			(at 149.86 44.958 90)
 			(hide yes)
@@
 			)
 		)
-		(property "Footprint" ""
+		(property "Footprint" "Resistor_SMD:R_01005_0402Metric_Pad0.57x0.30mm_HandSolder"
 			(at 125.73 70.358 90)
 			(hide yes)
@@
 			)
 		)
-		(property "Footprint" ""
+		(property "Footprint" "Capacitor_SMD:C_01005_0402Metric_Pad0.57x0.30mm_HandSolder"
 			(at 150.8252 58.42 0)
 			(hide yes)
@@
 			)
 		)
-		(property "Footprint" ""
+		(property "Footprint" "Capacitor_SMD:C_01005_0402Metric_Pad0.57x0.30mm_HandSolder"
 			(at 180.34 57.4548 0)
 			(hide yes)
@@
 			)
 		)
-		(property "Footprint" ""
+		(property "Footprint" "Button_Switch_SMD:SW_DIP_SPSTx01_Slide_6.7x4.1mm_W6.73mm_P2.54mm_LowProfile_JPin"
 			(at 124.46 73.66 0)
 			(hide yes)
@@
 			)
 		)
-		(property "Footprint" ""
+		(property "Footprint" "Capacitor_SMD:C_01005_0402Metric_Pad0.57x0.30mm_HandSolder"
 			(at 165.1 59.3852 0)
 			(hide yes)

Commit message: placement mostly done
Parts:
- added R34, R35, R38: 10k, Resistor_SMD:R_01005_0402Metric_Pad0.57x0.30mm_HandSolder, symbol Device:R
- U13: value ESP32-S3-MINI-1 -> ESP32-S3-MINI-1-N8; footprint RF_Module:ESP32-S2-MINI-1 -> footprints:XCVR_ESP32-S3-MINI-1-N8
Connections:
- net ADC_CS: now also U13.18 (IO14); no longer U13.15 (IO11)
- net FLASH_CLK: now also U13.16 (IO12); no longer U13.25 (IO21)
- net FLASH_MISO: now also U13.17 (IO13); no longer U13.28 (IO33)
- net FLASH_MOSI: now also U13.15 (IO11); no longer U13.26 (IO26)
- net GND: now also R34.2, R35.2, R38.2
- net VBAT_SENSE: now also U13.5 (IO1); no longer U13.6 (IO2)
- net BUCK_MODE: now reaches U13.19 (IO15)
- net at U13.41 (IO45): now also R34.1
- net at U13.44 (IO46): now also R35.1
- net at U13.7 (IO3): now also R38.1
- net SHUNT_EN: no longer names the net of U13.35 (IO39)
- no-connect marks 18 -> 15

Commit message: sketch pcb finished
Parts:
- C30, C31: footprint Capacitor_SMD:C_01005_0402Metric_Pad0.57x0.30mm_HandSolder -> Capacitor_SMD:C_0402_1005Metric_Pad0.74x0.62mm_HandSolder
- C32: value 10uF -> 22uF; footprint Capacitor_SMD:C_01005_0402Metric_Pad0.57x0.30mm_HandSolder -> Capacitor_SMD:C_0603_1608Metric_Pad1.08x0.95mm_HandSolder; MPN (none) -> GRM188R60J226MEA0J
- R29, R30, R34, R35, R38: footprint Resistor_SMD:R_01005_0402Metric_Pad0.57x0.30mm_HandSolder -> Resistor_SMD:R_0402_1005Metric_Pad0.72x0.64mm_HandSolder
- SW1, SW2: footprint Button_Switch_SMD:SW_DIP_SPSTx01_Slide_6.7x4.1mm_W6.73mm_P2.54mm_LowProfile_JPin -> Button_Switch_SMD:SW_SPST_SKQG_WithStem
Changed lines of the file:
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@@
 			)
 		)
-		(property "Footprint" "Button_Switch_SMD:SW_DIP_SPSTx01_Slide_6.7x4.1mm_W6.73mm_P2.54mm_LowProfile_JPin"
+		(property "Footprint" "Button_Switch_SMD:SW_SPST_SKQG_WithStem"
 			(at 132.08 55.88 0)
 			(hide yes)
@@
 			)
 		)
-		(property "Footprint" "Resistor_SMD:R_01005_0402Metric_Pad0.57x0.30mm_HandSolder"
+		(property "Footprint" "Resistor_SMD:R_0402_1005Metric_Pad0.72x0.64mm_HandSolder"
 			(at 149.86 44.958 90)
 			(hide yes)
@@
 			)
 		)
-		(property "Footprint" "Resistor_SMD:R_01005_0402Metric_Pad0.57x0.30mm_HandSolder"
+		(property "Footprint" "Resistor_SMD:R_0402_1005Metric_Pad0.72x0.64mm_HandSolder"
 			(at 125.73 70.358 90)
 			(hide yes)
@@
 			)
 		)
-		(property "Footprint" "Resistor_SMD:R_01005_0402Metric_Pad0.57x0.30mm_HandSolder"
+		(property "Footprint" "Resistor_SMD:R_0402_1005Metric_Pad0.72x0.64mm_HandSolder"
 			(at 151.13 75.692 90)
 			(hide yes)
@@
 			)
 		)
-		(property "Footprint" "Capacitor_SMD:C_01005_0402Metric_Pad0.57x0.30mm_HandSolder"
+		(property "Footprint" "Capacitor_SMD:C_0402_1005Metric_Pad0.74x0.62mm_HandSolder"
 			(at 150.8252 58.42 0)
 			(hide yes)
@@
 			)
 		)
-		(property "Footprint" "Capacitor_SMD:C_01005_0402Metric_Pad0.57x0.30mm_HandSolder"
+		(property "Footprint" "Capacitor_SMD:C_0402_1005Metric_Pad0.74x0.62mm_HandSolder"
 			(at 180.34 57.4548 0)
 			(hide yes)
@@
 			)
 		)
-		(property "Footprint" "Resistor_SMD:R_01005_0402Metric_Pad0.57x0.30mm_HandSolder"
+		(property "Footprint" "Resistor_SMD:R_0402_1005Metric_Pad0.72x0.64mm_HandSolder"
 			(at 200.66 119.888 90)
 			(hide yes)
@@
 			)
 		)
-		(property "Footprint" "Button_Switch_SMD:SW_DIP_SPSTx01_Slide_6.7x4.1mm_W6.73mm_P2.54mm_LowProfile_JPin"
+		(property "Footprint" "Button_Switch_SMD:SW_SPST_SKQG_WithStem"
 			(at 124.46 73.66 0)
 			(hide yes)
@@
 			)
 		)
-		(property "Value" "10uF"
+		(property "Value" "22uF"
 			(at 168.91 54.61 90)
 			(show_name no)
@@
 			)
 		)
-		(property "Footprint" "Capacitor_SMD:C_01005_0402Metric_Pad0.57x0.30mm_HandSolder"
+		(property "Footprint" "Capacitor_SMD:C_0603_1608Metric_Pad1.08x0.95mm_HandSolder"
 			(at 165.1 59.3852 0)
 			(hide yes)
@@
 		(property "Description" "Unpolarized capacitor"
 			(at 168.91 58.42 0)
+			(hide yes)
+			(show_name no)
+			(do_not_autoplace no)
+			(effects
+				(font
+					(size 1.27 1.27)
+				)
+			)
+		)
+		(property "MPN" "GRM188R60J226MEA0J"
+			(at 168.91 58.42 90)
 			(hide yes)
 			(show_name no)
@@
 			)
 		)
-		(property "Footprint" "Resistor_SMD:R_01005_0402Metric_Pad0.57x0.30mm_HandSolder"
+		(property "Footprint" "Resistor_SMD:R_0402_1005Metric_Pad0.72x0.64mm_HandSolder"
 			(at 200.66 116.078 90)
 			(hide yes)
