File: WSG_1.0/WSG_1.0/WSG_1.0.kicad_pcb (KiCad board)
At the start: 4 copper layers, 117.5 x 94 mm, 17 parts, among them J2 USB4110-GF-A, U1 ADS131A04IPBS, U10 TPS22916BYFPR, U11 W25N04KVZEIR, U12 USBLC6-2SC6, U13 ESP32-S3-MINI-1, U2 DAC60501MDGSR, U3 INA827AIDGK, U4 INA827AIDGK, U5 INA827AIDGK, U6 TMP235A2DBZR, U7 PQ25180YBGT, U8 TPS63802DLAR, U9 TPS7A2025PDBVR, Y1 SiT8008AI-13-33S-16.384000

Commit message: placement mostly done
Parts:
- added C1: 0.1uF, Capacitor_SMD:C_01005_0402Metric_Pad0.57x0.30mm_HandSolder, B.Cu at (145.1, 81.9)
- added C10: 10uF, Capacitor_SMD:C_01005_0402Metric_Pad0.57x0.30mm_HandSolder, F.Cu at (71.3, 157.8)
- added C11: 0.1uF, Capacitor_SMD:C_01005_0402Metric_Pad0.57x0.30mm_HandSolder, F.Cu at (154.5, 74.8)
- added C12: 1uF, Capacitor_SMD:C_01005_0402Metric_Pad0.57x0.30mm_HandSolder, F.Cu at (74.2, 157.0)
- added C13: 0.1uF, Capacitor_SMD:C_01005_0402Metric_Pad0.57x0.30mm_HandSolder, B.Cu at (145.4, 75.8)
- added C14: 10uF, Capacitor_SMD:C_01005_0402Metric_Pad0.57x0.30mm_HandSolder, F.Cu at (77.5, 155.1)
- added C15: 22uF, Capacitor_SMD:C_01005_0402Metric_Pad0.57x0.30mm_HandSolder, F.Cu at (77.3, 160.0)
- added C16: 1uF, Capacitor_SMD:C_01005_0402Metric_Pad0.57x0.30mm_HandSolder, F.Cu at (100.6, 80.0)
- added C17: 1uF, Capacitor_SMD:C_01005_0402Metric_Pad0.57x0.30mm_HandSolder, F.Cu at (130.8, 83.0)
- added C18: 0.1uF, Capacitor_SMD:C_01005_0402Metric_Pad0.57x0.30mm_HandSolder, F.Cu at (119.3, 87.7)
- added C19: 100nF, Capacitor_SMD:C_01005_0402Metric_Pad0.57x0.30mm_HandSolder, F.Cu at (98.6, 79.9)
- added C2: 10nF, Capacitor_SMD:C_01005_0402Metric_Pad0.57x0.30mm_HandSolder, F.Cu at (155.3, 84.9)
- added C20: 1uF, Capacitor_SMD:C_01005_0402Metric_Pad0.57x0.30mm_HandSolder, F.Cu at (137.5, 85.7)
- added C21: 270nF, Capacitor_SMD:C_01005_0402Metric_Pad0.57x0.30mm_HandSolder, F.Cu at (135.7, 85.7)
- added C22: 1uF, Capacitor_SMD:C_01005_0402Metric_Pad0.57x0.30mm_HandSolder, F.Cu at (138.0, 74.2)
- added C23: 1uF, Capacitor_SMD:C_01005_0402Metric_Pad0.57x0.30mm_HandSolder, F.Cu at (136.4, 85.7)
- added C24: 1uF, Capacitor_SMD:C_01005_0402Metric_Pad0.57x0.30mm_HandSolder, F.Cu at (134.0, 85.7)
- added C25: 1uF, Capacitor_SMD:C_01005_0402Metric_Pad0.57x0.30mm_HandSolder, F.Cu at (138.9, 85.7)
- added C26: 150nF, Capacitor_SMD:C_01005_0402Metric_Pad0.57x0.30mm_HandSolder, F.Cu at (148.9, 88.4)
- added C27: 0.1uF, Capacitor_SMD:C_01005_0402Metric_Pad0.57x0.30mm_HandSolder, F.Cu at (148.9, 90.0)
- added C28: 0.1uF, Capacitor_SMD:C_01005_0402Metric_Pad0.57x0.30mm_HandSolder, F.Cu at (143.3, 83.5)
- added C29: 0.1uF, Capacitor_SMD:C_01005_0402Metric_Pad0.57x0.30mm_HandSolder, F.Cu at (154.5, 88.3)
- added C3: 10nF, Capacitor_SMD:C_01005_0402Metric_Pad0.57x0.30mm_HandSolder, F.Cu at (158.1, 73.9)
- added C30: 1uF, Capacitor_SMD:C_01005_0402Metric_Pad0.57x0.30mm_HandSolder, F.Cu at (153.4, 159.7)
- added C31: 0.1uF, Capacitor_SMD:C_01005_0402Metric_Pad0.57x0.30mm_HandSolder, F.Cu at (153.4, 161.3)
- added C32: 10uF, Capacitor_SMD:C_01005_0402Metric_Pad0.57x0.30mm_HandSolder, F.Cu at (153.9, 163.2)
- added C33: 100nF, Capacitor_SMD:C_01005_0402Metric_Pad0.57x0.30mm_HandSolder, F.Cu at (101.5, 77.7)
- added C34: 1uF, Capacitor_SMD:C_01005_0402Metric_Pad0.57x0.30mm_HandSolder, F.Cu at (119.9, 81.7)
- added C35: 1uF, Capacitor_SMD:C_01005_0402Metric_Pad0.57x0.30mm_HandSolder, F.Cu at (138.1, 73.6)
- added C4: 0.1uF, Capacitor_SMD:C_01005_0402Metric_Pad0.57x0.30mm_HandSolder, F.Cu at (151.4, 83.0)
- added C5: 0.1uF, Capacitor_SMD:C_01005_0402Metric_Pad0.57x0.30mm_HandSolder, F.Cu at (153.3, 83.0)
- added C6: 0.1uF, Capacitor_SMD:C_01005_0402Metric_Pad0.57x0.30mm_HandSolder, B.Cu at (145.2, 78.6)
- added C7: 10nF, Capacitor_SMD:C_01005_0402Metric_Pad0.57x0.30mm_HandSolder, F.Cu at (153.4, 83.8)
- added C8: 1uF, Capacitor_SMD:C_01005_0402Metric_Pad0.57x0.30mm_HandSolder, F.Cu at (71.4, 156.8)
- added C9: 10nF, Capacitor_SMD:C_01005_0402Metric_Pad0.57x0.30mm_HandSolder, F.Cu at (154.9, 79.5)
- added F1: Polyfuse, Fuse:Fuse_0805_2012Metric_Pad1.15x1.40mm_HandSolder, F.Cu at (63.8, 158.1)
- added H1: MountingHole, MountingHole:MountingHole_3.2mm_M3, F.Cu at (57.2, 76.7)
- added H2: MountingHole, MountingHole:MountingHole_3.2mm_M3, F.Cu at (57.2, 84.6)
- added J1: Conn_01x10, Connector_PinHeader_2.00mm:PinHeader_2x05_P2.00mm_Horizontal, F.Cu at (157.9, 76.0)
- added J4: Conn_01x02, footprints:JST_S2B-PH-K-S_LF__SN_-2pin_male, F.Cu at (56.5, 142.0)
- added L1: 470nH, Inductor_SMD:L_Coilcraft_XxL4020, F.Cu at (80.5, 157.5)
- added R1: 100, Resistor_SMD:R_01005_0402Metric_Pad0.57x0.30mm_HandSolder, F.Cu at (133.2, 74.2)
- added R10: 1k, Resistor_SMD:R_01005_0402Metric_Pad0.57x0.30mm_HandSolder, F.Cu at (154.8, 78.2)
- added R11: 845, Resistor_SMD:R_01005_0402Metric_Pad0.57x0.30mm_HandSolder, F.Cu at (149.6, 77.9)
- added R12: 350, Resistor_SMD:R_01005_0402Metric_Pad0.57x0.30mm_HandSolder, F.Cu at (155.5, 81.7)
- added R13: 1k, Resistor_SMD:R_01005_0402Metric_Pad0.57x0.30mm_HandSolder, F.Cu at (155.1, 83.0)
- added R14: 10.2k, Resistor_SMD:R_01005_0402Metric_Pad0.57x0.30mm_HandSolder, F.Cu at (66.7, 158.8)
- added R15: 100, Resistor_SMD:R_01005_0402Metric_Pad0.57x0.30mm_HandSolder, F.Cu at (136.5, 73.6)
- added R16: 350, Resistor_SMD:R_01005_0402Metric_Pad0.57x0.30mm_HandSolder, F.Cu at (156.0, 79.7)
- added R17: 1k, Resistor_SMD:R_01005_0402Metric_Pad0.57x0.30mm_HandSolder, F.Cu at (154.9, 80.1)
- added R18: 100, Resistor_SMD:R_01005_0402Metric_Pad0.57x0.30mm_HandSolder, F.Cu at (134.8, 73.6)
- added R19: 100, Resistor_SMD:R_01005_0402Metric_Pad0.57x0.30mm_HandSolder, F.Cu at (133.2, 73.6)
- added R2: 100, Resistor_SMD:R_01005_0402Metric_Pad0.57x0.30mm_HandSolder, F.Cu at (134.8, 74.2)
- added R20: 560k, Resistor_SMD:R_01005_0402Metric_Pad0.57x0.30mm_HandSolder, F.Cu at (74.1, 159.0)
- added R21: 845, Resistor_SMD:R_01005_0402Metric_Pad0.57x0.30mm_HandSolder, F.Cu at (149.6, 75.0)
- added R24: 100k, Resistor_SMD:R_01005_0402Metric_Pad0.57x0.30mm_HandSolder, F.Cu at (119.2, 84.6)
- added R25: 1M, Resistor_SMD:R_01005_0402Metric_Pad0.57x0.30mm_HandSolder, B.Cu at (101.5, 77.7)
- added R26: 1M, Resistor_SMD:R_01005_0402Metric_Pad0.57x0.30mm_HandSolder, F.Cu at (99.9, 77.7)
- added R27: 100, Resistor_SMD:R_01005_0402Metric_Pad0.57x0.30mm_HandSolder, F.Cu at (138.1, 85.7)
- added R28: 100k, Resistor_SMD:R_01005_0402Metric_Pad0.57x0.30mm_HandSolder, F.Cu at (142.8, 79.3)
- added R29: 10k, Resistor_SMD:R_01005_0402Metric_Pad0.57x0.30mm_HandSolder, F.Cu at (156.6, 160.0)
- added R3: 100, Resistor_SMD:R_01005_0402Metric_Pad0.57x0.30mm_HandSolder, F.Cu at (136.4, 74.2)
- added R30: 10k, Resistor_SMD:R_01005_0402Metric_Pad0.57x0.30mm_HandSolder, F.Cu at (156.6, 161.7)
- added R31: 1M, Resistor_SMD:R_01005_0402Metric_Pad0.57x0.30mm_HandSolder, B.Cu at (100.0, 77.7)
- added R32: 100k, Resistor_SMD:R_01005_0402Metric_Pad0.57x0.30mm_HandSolder, F.Cu at (74.2, 158.0)
- added R33: 10k, Resistor_SMD:R_01005_0402Metric_Pad0.57x0.30mm_HandSolder, F.Cu at (66.4, 157.3)
- added R34: 10k, Resistor_SMD:R_01005_0402Metric_Pad0.57x0.30mm_HandSolder, F.Cu at (119.9, 74.7)
- added R35: 10k, Resistor_SMD:R_01005_0402Metric_Pad0.57x0.30mm_HandSolder, F.Cu at (119.9, 76.3)
- added R36: 10k, Resistor_SMD:R_01005_0402Metric_Pad0.57x0.30mm_HandSolder, F.Cu at (120.0, 86.5)
- added R37: 10k, Resistor_SMD:R_01005_0402Metric_Pad0.57x0.30mm_HandSolder, F.Cu at (118.7, 86.2)
- added R38: 10k, Resistor_SMD:R_01005_0402Metric_Pad0.57x0.30mm_HandSolder, F.Cu at (119.9, 78.0)
- added R39: 100k, Resistor_SMD:R_01005_0402Metric_Pad0.57x0.30mm_HandSolder, F.Cu at (107.0, 89.1)
- added R4: 350, Resistor_SMD:R_01005_0402Metric_Pad0.57x0.30mm_HandSolder, F.Cu at (131.1, 83.8)
- added R40: 5.1k, Resistor_SMD:R_01005_0402Metric_Pad0.57x0.30mm_HandSolder, F.Cu at (63.5, 155.7)
- added R41: 5.1k, Resistor_SMD:R_01005_0402Metric_Pad0.57x0.30mm_HandSolder, B.Cu at (63.6, 158.7)
- added R5: 100k, Resistor_SMD:R_01005_0402Metric_Pad0.57x0.30mm_HandSolder, F.Cu at (73.4, 150.9)
- added R6: 350, Resistor_SMD:R_01005_0402Metric_Pad0.57x0.30mm_HandSolder, F.Cu at (151.5, 88.4)
- added R7: 350, Resistor_SMD:R_01005_0402Metric_Pad0.57x0.30mm_HandSolder, F.Cu at (155.2, 84.1)
- added R8: 845, Resistor_SMD:R_01005_0402Metric_Pad0.57x0.30mm_HandSolder, F.Cu at (149.5, 81.1)
- added R9: 1k, Resistor_SMD:R_01005_0402Metric_Pad0.57x0.30mm_HandSolder, F.Cu at (153.2, 82.1)
- added SW1: SW_Push, Button_Switch_SMD:SW_DIP_SPSTx01_Slide_6.7x4.1mm_W6.73mm_P2.54mm_LowProfile_JPin, F.Cu at (163.0, 155.7)
- added SW2: SW_Push, Button_Switch_SMD:SW_DIP_SPSTx01_Slide_6.7x4.1mm_W6.73mm_P2.54mm_LowProfile_JPin, F.Cu at (163.0, 161.5)
- J2: value USB4110-GF-A -> USB_C_Receptacle_USB2.0_16P
- U1: value ADS131A04IPBS -> ADS131A04IPBSR
- U10: value TPS22916BYFPR -> TPS22916CYFPR
- U13: value ESP32-S3-MINI-1 -> ESP32-S3-MINI-1-N8; footprint RF_Module:ESP32-S2-MINI-1 -> footprints:XCVR_ESP32-S3-MINI-1-N8
- U2: value DAC60501MDGSR -> DAC60501ZDGSR
- moved U10 87.2 mm to (144.2, 90.5)
- moved U2 76.8 mm to (147.2, 84.5)
- moved U5 75.2 mm to (147.0, 75.0), turned to 180 degrees
- moved U6 74.4 mm to (158.3, 87.2)
- moved U4 69.5 mm to (147.0, 77.8), turned to 180 degrees
- moved U1 68.9 mm to (136.8, 79.7)
- moved U3 63.6 mm to (146.9, 81.2), turned to 180 degrees
- moved U9 61.4 mm to (165.6, 87.5)
- moved MOSFET1 54.9 mm to (69.2, 149.7), turned to 180 degrees
- moved U11 53.2 mm to (98.8, 87.7), turned to 180 degrees
- moved U13 30.3 mm to (110.3, 80.2)
- moved Y1 23.1 mm to (135.1, 90.2)
- moved D1 17.6 mm to (64.9, 151.8), turned to -90 degrees
- moved U12 17.0 mm to (64.9, 162.7)
- moved U7 7.11 mm to (69.0, 158.0)
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Connections:
- J2 pad A1: (no net) -> GND
- J2 pad A12: (no net) -> GND
- J2 pad A4: (no net) -> VBUS
- J2 pad A9: (no net) -> VBUS
- J2 pad B1: (no net) -> GND
- J2 pad B12: (no net) -> GND
- J2 pad B4: (no net) -> VBUS
- J2 pad B9: (no net) -> VBUS
- J2 pad SH: (no net) -> GND
- U13 pad 15: ADC_CS -> FLASH_MOSI
- U13 pad 16: unconnected-(U13-IO12-Pad16) -> FLASH_CLK
- U13 pad 17: unconnected-(U13-IO13-Pad17) -> FLASH_MISO
- U13 pad 18: unconnected-(U13-IO14-Pad18) -> ADC_CS
- U13 pad 19: unconnected-(U13-IO15-Pad19) -> BUCK_MODE
- U13 pad 25: FLASH_CLK -> unconnected-(U13-IO21-Pad25)
- U13 pad 26: FLASH_MOSI -> unconnected-(U13-IO26-Pad26)
- U13 pad 28: FLASH_MISO -> unconnected-(U13-IO33-Pad28)
- U13 pad 35: SHUNT_EN -> unconnected-(U13-IO39-Pad35)
- U13 pad 41: unconnected-(U13-IO45-Pad41) -> Net-(U13-IO45)
- U13 pad 44: unconnected-(U13-IO46-Pad44) -> Net-(U13-IO46)
- U13 pad 5: unconnected-(U13-IO1-Pad5) -> VBAT_SENSE
- U13 pad 6: VBAT_SENSE -> unconnected-(U13-IO2-Pad6)
- U13 pad 7: unconnected-(U13-IO3-Pad7) -> Net-(U13-IO3)
- U7 pad A1: (no net) -> CHG_INT
- U7 pad A2: (no net) -> VIN_P
- U7 pad B1: (no net) -> I2C_SCL
- U7 pad B2: (no net) -> SYS
- U7 pad C1: (no net) -> I2C_SDA
- U7 pad C2: (no net) -> VBAT
- U7 pad D1: (no net) -> Net-(U7-TS_MR)
- U7 pad D2: (no net) -> GND
- U8 pad 2: GND -> BUCK_MODE
Routing:
- net (no net): track 0.00 -> 0.10 mm, vias 0 -> 1
Other:
- board text added: "digital"
- board text added: "power"

Commit message: sketch pcb finished
Parts:
- removed R31: 1M, Resistor_SMD:R_01005_0402Metric_Pad0.57x0.30mm_HandSolder
- added FB1: 0, Resistor_SMD:R_0402_1005Metric_Pad0.72x0.64mm_HandSolder, F.Cu at (127.9, 83.9)
- added U14: TPD4E1U06DBVR, footprints:SOT95P280X145-6N, F.Cu at (131.6, 86.5)
- C1, C10, C11, C12, C13, C16, C17, C18, C19, C2, C20, C22, C23, C25, C27, C28, C3, C30, C31, C33, C34, C4, C5, C6, C7, C8, C9: footprint Capacitor_SMD:C_01005_0402Metric_Pad0.57x0.30mm_HandSolder -> Capacitor_SMD:C_0402_1005Metric_Pad0.74x0.62mm_HandSolder
- C14, C32: value 10uF -> 22uF; footprint Capacitor_SMD:C_01005_0402Metric_Pad0.57x0.30mm_HandSolder -> Capacitor_SMD:C_0603_1608Metric_Pad1.08x0.95mm_HandSolder
- C15: footprint Capacitor_SMD:C_01005_0402Metric_Pad0.57x0.30mm_HandSolder -> Capacitor_SMD:C_0603_1608Metric_Pad1.08x0.95mm_HandSolder
- C21: value 270nF -> 0.1uF; footprint Capacitor_SMD:C_01005_0402Metric_Pad0.57x0.30mm_HandSolder -> Capacitor_SMD:C_0402_1005Metric_Pad0.74x0.62mm_HandSolder; moved to B.Cu
- C24, C26, C29, C35: footprint Capacitor_SMD:C_01005_0402Metric_Pad0.57x0.30mm_HandSolder -> Capacitor_SMD:C_0402_1005Metric_Pad0.74x0.62mm_HandSolder; moved to B.Cu
- F1: value Polyfuse -> 0ZCJ0075AF2E; footprint Fuse:Fuse_0805_2012Metric_Pad1.15x1.40mm_HandSolder -> Fuse:Fuse_1206_3216Metric
- R1, R14, R15, R2, R24, R36, R37: footprint Resistor_SMD:R_01005_0402Metric_Pad0.57x0.30mm_HandSolder -> Resistor_SMD:R_0402_1005Metric_Pad0.72x0.64mm_HandSolder; moved to B.Cu
- R10, R11, R12, R13, R16, R17, R18, R19, R21, R26, R27, R28, R29, R3, R30, R33, R34, R35, R38, R39, R4, R40, R41, R5, R6, R7, R8, R9: footprint Resistor_SMD:R_01005_0402Metric_Pad0.57x0.30mm_HandSolder -> Resistor_SMD:R_0402_1005Metric_Pad0.72x0.64mm_HandSolder
- R20: value 560k -> 511k; footprint Resistor_SMD:R_01005_0402Metric_Pad0.57x0.30mm_HandSolder -> Resistor_SMD:R_0402_1005Metric_Pad0.72x0.64mm_HandSolder
- R25: footprint Resistor_SMD:R_01005_0402Metric_Pad0.57x0.30mm_HandSolder -> Resistor_SMD:R_0402_1005Metric_Pad0.72x0.64mm_HandSolder; moved to F.Cu
- R32: value 100k -> 91k; footprint Resistor_SMD:R_01005_0402Metric_Pad0.57x0.30mm_HandSolder -> Resistor_SMD:R_0402_1005Metric_Pad0.72x0.64mm_HandSolder
- SW1, SW2: footprint Button_Switch_SMD:SW_DIP_SPSTx01_Slide_6.7x4.1mm_W6.73mm_P2.54mm_LowProfile_JPin -> Button_Switch_SMD:SW_SPST_SKQG_WithStem
- U11: footprint footprints:SON127P500X600X80-9N -> footprints:IC_W25N04KVZEIR; moved to B.Cu
- U3, U4, U5: value INA827AIDGK -> INA827AIDGKR
- U7: value PQ25180YBGT -> BQ25180YBGR
- U8: footprint Package_DFN_QFN:DFN-10-1EP_2x3mm_P0.5mm_EP0.64x2.4mm -> footprints:DLA0010A
- moved SW1 104.2 mm to (95.0, 76.8), turned to 90 degrees
- moved C32 103.3 mm to (100.7, 74.7), turned to 180 degrees
- moved R30 100.3 mm to (101.9, 77.6), turned to -90 degrees
- moved C31 100.0 mm to (101.3, 76.0), turned to 180 degrees
- moved SW2 93.6 mm to (125.9, 75.6)
- moved R29 92.9 mm to (121.0, 74.2), turned to 90 degrees
- moved C30 92.6 mm to (119.4, 73.6), turned to 180 degrees
- moved H1 82.7 mm to (136.0, 101.6), turned to -90 degrees
- moved C12 73.2 mm to (103.6, 90.0), turned to 180 degrees
- moved H2 72.9 mm to (128.1, 101.6), turned to -90 degrees
- moved R32 72.0 mm to (102.0, 91.6), turned to -90 degrees
- moved C14 71.3 mm to (107.1, 90.3), turned to 180 degrees
- moved U8 71.1 mm to (103.9, 92.3)
- moved R20 70.8 mm to (102.0, 93.9), turned to -90 degrees
- moved MOSFET1 70.4 mm to (99.6, 86.2)
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Connections:
- C21 pad 1: GND -> 3V3A
- C21 pad 2: VNCP_C -> GND
- C34 pad 2: 3V3 -> Net-(U10-VIN)
- U1 pad 11: VNCP_C -> GND
- U10 pad A2: 3V3 -> Net-(U10-VIN)
Routing:
- net GND: track 0.00 -> 64.6 mm, vias 0 -> 55
- net BATT_N: track 0.00 -> 44.0 mm
- net AIN3P: track 0.00 -> 14.6 mm
- net 3V3: track 0.00 -> 13.3 mm, vias 0 -> 12
- net EN: track 0.00 -> 12.5 mm
- net USB_DM: track 0.00 -> 10.4 mm, vias 0 -> 2
- net FLASH_MISO: track 0.00 -> 7.74 mm, vias 0 -> 1
- net USB_DP: track 0.00 -> 7.44 mm, vias 0 -> 2
- net VREF_1V65: track 0.00 -> 7.24 mm
- net BATT_P: track 0.00 -> 7.16 mm, vias 0 -> 1
- net VBUS: track 0.00 -> 5.89 mm, vias 0 -> 2
- net SIG0: track 0.00 -> 4.62 mm
- net VBAT_SENSE: track 0.00 -> 4.50 mm
- net FLASH_CS: track 0.00 -> 4.34 mm, vias 0 -> 1
- net INP0: track 0.00 -> 4.02 mm
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- added copper zone on In2.Cu, net 3V3
- added copper zone on In2.Cu, net 3V3A
- added copper zone on B.Cu, net GND
- added copper zone on F.Cu, net GND
- added copper zone on In1.Cu, net GND
Other:
- board size 117.5 x 94 mm -> 53.8 x 34.1 mm
- board text removed: "digital"
- board text removed: "power"
