File: WSG_1.0/WSG_1.0/WSG_1_0_ESP.kicad_sch (KiCad schematic)
At the start: 22 parts, among them SW3 SW_Push, SW4 SW_Push, U15 ESP32-S3-MINI-1U-N8

Commit message: ~1/2 done with routing, neeed to undo some
Other:
- moved on the sheet: R23, R29, R30, R38, R57, R58
Changed lines of the file:
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@@
 	(wire
 		(pts
-			(xy 95.25 71.12) (xy 111.76 71.12)
+			(xy 96.52 71.12) (xy 111.76 71.12)
 		)
 		(stroke
@@
 	(wire
 		(pts
-			(xy 95.25 71.12) (xy 95.25 69.85)
+			(xy 96.52 71.12) (xy 96.52 69.85)
 		)
 		(stroke
@@
 	(wire
 		(pts
-			(xy 88.9 90.17) (xy 95.25 90.17)
+			(xy 78.74 90.17) (xy 95.25 90.17)
 		)
 		(stroke
@@
 	(global_label "DAC_CS"
 		(shape input)
-		(at 87.63 69.85 180)
+		(at 88.9 69.85 180)
 		(fields_autoplaced yes)
 		(effects
@@
 		)
 		(property "Intersheetrefs" "${INTERSHEET_REFS}"
-			(at 77.5691 69.85 0)
+			(at 78.8391 69.85 0)
 			(hide yes)
 			(show_name no)
@@
 	(global_label "3V3A"
 		(shape input)
-		(at 46.99 113.03 180)
+		(at 38.1 113.03 180)
 		(fields_autoplaced yes)
 		(effects
@@
 		)
 		(property "Intersheetrefs" "${INTERSHEET_REFS}"
-			(at 39.4086 113.03 0)
+			(at 30.5186 113.03 0)
 			(hide yes)
 			(show_name no)
@@
 	(global_label "3V3A"
 		(shape input)
-		(at 46.99 102.87 180)
+		(at 38.1 102.87 180)
 		(fields_autoplaced yes)
 		(effects
@@
 		)
 		(property "Intersheetrefs" "${INTERSHEET_REFS}"
-			(at 39.4086 102.87 0)
+			(at 30.5186 102.87 0)
 			(hide yes)
 			(show_name no)
@@
 	(global_label "ADC_RST"
 		(shape input)
-		(at 54.61 83.82 0)
+		(at 45.72 83.82 0)
 		(fields_autoplaced yes)
 		(effects
@@
 		)
 		(property "Intersheetrefs" "${INTERSHEET_REFS}"
-			(at 65.6385 83.82 0)
+			(at 56.7485 83.82 0)
 			(hide yes)
 			(show_name no)
@@
 	(global_label "ADC_CS"
 		(shape input)
-		(at 54.61 102.87 0)
+		(at 45.72 102.87 0)
 		(fields_autoplaced yes)
 		(effects
@@
 		)
 		(property "Intersheetrefs" "${INTERSHEET_REFS}"
-			(at 64.6709 102.87 0)
+			(at 55.7809 102.87 0)
 			(hide yes)
 			(show_name no)
@@
 	(global_label "3V3A"
 		(shape input)
-		(at 46.99 83.82 180)
+		(at 38.1 83.82 180)
 		(fields_autoplaced yes)
 		(effects
@@
 		)
 		(property "Intersheetrefs" "${INTERSHEET_REFS}"
-			(at 39.4086 83.82 0)
+			(at 30.5186 83.82 0)
 			(hide yes)
 			(show_name no)
@@
 	(global_label "3V3"
 		(shape input)
-		(at 46.99 93.98 180)
+		(at 38.1 93.98 180)
 		(fields_autoplaced yes)
 		(effects
@@
 		)
 		(property "Intersheetrefs" "${INTERSHEET_REFS}"
-			(at 40.4972 93.98 0)
+			(at 31.6072 93.98 0)
 			(hide yes)
 			(show_name no)
@@
 	(global_label "FLASH_CS"
 		(shape input)
-		(at 54.61 93.98 0)
+		(at 45.72 93.98 0)
 		(fields_autoplaced yes)
 		(effects
@@
 		)
 		(property "Intersheetrefs" "${INTERSHEET_REFS}"
-			(at 66.7876 93.98 0)
+			(at 57.8976 93.98 0)
 			(hide yes)
 			(show_name no)
@@
 	(global_label "ADC_RST"
 		(shape input)
-		(at 81.28 90.17 180)
+		(at 71.12 90.17 180)
 		(fields_autoplaced yes)
 		(effects
@@
 		)
 		(property "Intersheetrefs" "${INTERSHEET_REFS}"
-			(at 70.2515 90.17 0)
+			(at 60.0915 90.17 0)
 			(hide yes)
 			(show_name no)
@@
 	(global_label "DAC_CS"
 		(shape input)
-		(at 54.61 113.03 0)
+		(at 45.72 113.03 0)
 		(fields_autoplaced yes)
 		(effects
@@
 		)
 		(property "Intersheetrefs" "${INTERSHEET_REFS}"
-			(at 64.6709 113.03 0)
+			(at 55.7809 113.03 0)
 			(hide yes)
 			(show_name no)
@@
 	(symbol
 		(lib_id "Device:R")
-		(at 50.8 102.87 270)
+		(at 41.91 102.87 270)
 		(unit 1)
 		(body_style 1)
@@
 		(fields_autoplaced yes)
 		(property "Reference" "R29"
-			(at 50.8 96.52 90)
+			(at 41.91 96.52 90)
 			(show_name no)
 			(do_not_autoplace no)
@@
 		)
 		(property "Value" "100k"
-			(at 50.8 99.06 90)
+			(at 41.91 99.06 90)
 			(show_name no)
 			(do_not_autoplace no)
@@
 		)
 		(property "Footprint" "Resistor_SMD:R_0402_1005Metric_Pad0.72x0.64mm_HandSolder"
-			(at 50.8 101.092 90)
+			(at 41.91 101.092 90)
 			(hide yes)
 			(show_name no)
@@
 		)
 		(property "Datasheet" ""
-			(at 50.8 102.87 0)
+			(at 41.91 102.87 0)
 			(hide yes)
 			(show_name no)
@@
 		)
 		(property "Description" "Resistor"
-			(at 50.8 102.87 0)
+			(at 41.91 102.87 0)
 			(hide yes)
 			(show_name no)
@@
 	(symbol
 		(lib_id "Device:R")
-		(at 91.44 69.85 270)
+		(at 92.71 69.85 270)
 		(unit 1)
 		(body_style 1)
@@
 		(dnp no)
 		(property "Reference" "R58"
-			(at 91.186 71.12 90)
+			(at 92.456 71.12 90)
 			(show_name no)
 			(do_not_autoplace no)
@@
 		)
 		(property "Value" "1k"
-			(at 91.186 68.58 90)
+			(at 92.456 68.58 90)
 			(show_name no)
 			(do_not_autoplace no)
@@
 		)
 		(property "Footprint" "Resistor_SMD:R_0402_1005Metric_Pad0.72x0.64mm_HandSolder"
-			(at 91.44 68.072 90)
+			(at 92.71 68.072 90)
 			(hide yes)
 			(show_name no)
@@
 		)
 		(property "Datasheet" ""
-			(at 91.44 69.85 0)
+			(at 92.71 69.85 0)
 			(hide yes)
 			(show_name no)
@@
 		)
 		(property "Description" "Resistor"
-			(at 91.44 69.85 0)
+			(at 92.71 69.85 0)
 			(hide yes)
 			(show_name no)
@@
 	(symbol
 		(lib_id "Device:R")
-		(at 50.8 83.82 270)
+		(at 41.91 83.82 270)
 		(unit 1)
 		(body_style 1)
@@
 		(fields_autoplaced yes)
 		(property "Reference" "R38"
-			(at 50.8 77.47 90)
+			(at 41.91 77.47 90)
 			(show_name no)
 			(do_not_autoplace no)
@@
 		)
 		(property "Value" "100k"
-			(at 50.8 80.01 90)
+			(at 41.91 80.01 90)
 			(show_name no)
 			(do_not_autoplace no)
@@
 		)
 		(property "Footprint" "Resistor_SMD:R_0402_1005Metric_Pad0.72x0.64mm_HandSolder"
-			(at 50.8 82.042 90)
+			(at 41.91 82.042 90)
 			(hide yes)
 			(show_name no)
@@
 		)
 		(property "Datasheet" ""
-			(at 50.8 83.82 0)
+			(at 41.91 83.82 0)
 			(hide yes)
 			(show_name no)
@@
 		)
 		(property "Description" "Resistor"
-			(at 50.8 83.82 0)
+			(at 41.91 83.82 0)
 			(hide yes)
 			(show_name no)
@@
 	(symbol
 		(lib_id "Device:R")
-		(at 85.09 90.17 90)
+		(at 74.93 90.17 90)
 		(unit 1)
 		(body_style 1)
@@
 		(dnp no)
 		(property "Reference" "R57"
-			(at 84.074 88.9 90)
+			(at 73.914 88.9 90)
 			(show_name no)
 			(do_not_autoplace no)
@@
 		)
 		(property "Value" "1k"
-			(at 84.074 91.44 90)
+			(at 73.914 91.44 90)
 			(show_name no)
 			(do_not_autoplace no)
@@
 		)
 		(property "Footprint" "Resistor_SMD:R_0402_1005Metric_Pad0.72x0.64mm_HandSolder"
-			(at 85.09 91.948 90)
+			(at 74.93 91.948 90)
 			(hide yes)
 			(show_name no)
@@
 		)
 		(property "Datasheet" ""
-			(at 85.09 90.17 0)
+			(at 74.93 90.17 0)
 			(hide yes)
 			(show_name no)
@@
 		)
 		(property "Description" "Resistor"
-			(at 85.09 90.17 0)
+			(at 74.93 90.17 0)
 			(hide yes)
 			(show_name no)
@@
 	(symbol
 		(lib_id "Device:R")
-		(at 50.8 93.98 270)
+		(at 41.91 93.98 270)
 		(unit 1)
 		(body_style 1)
@@
 		(fields_autoplaced yes)
 		(property "Reference" "R23"
-			(at 50.8 87.63 90)
+			(at 41.91 87.63 90)
 			(show_name no)
 			(do_not_autoplace no)
@@
 		)
 		(property "Value" "100k"
-			(at 50.8 90.17 90)
+			(at 41.91 90.17 90)
 			(show_name no)
 			(do_not_autoplace no)
@@
 		)
 		(property "Footprint" "Resistor_SMD:R_0402_1005Metric_Pad0.72x0.64mm_HandSolder"
-			(at 50.8 92.202 90)
+			(at 41.91 92.202 90)
 			(hide yes)
 			(show_name no)
@@
 		)
 		(property "Datasheet" ""
-			(at 50.8 93.98 0)
+			(at 41.91 93.98 0)
 			(hide yes)
 			(show_name no)
@@
 		)
 		(property "Description" "Resistor"
-			(at 50.8 93.98 0)
+			(at 41.91 93.98 0)
 			(hide yes)
 			(show_name no)
@@
 	(symbol
 		(lib_id "Device:R")
-		(at 50.8 113.03 270)
+		(at 41.91 113.03 270)
 		(unit 1)
 		(body_style 1)
@@
 		(fields_autoplaced yes)
 		(property "Reference" "R30"
-			(at 50.8 106.68 90)
+			(at 41.91 106.68 90)
 			(show_name no)
 			(do_not_autoplace no)
@@
 		)
 		(property "Value" "100k"
-			(at 50.8 109.22 90)
+			(at 41.91 109.22 90)
 			(show_name no)
 			(do_not_autoplace no)
@@
 		)
 		(property "Footprint" "Resistor_SMD:R_0402_1005Metric_Pad0.72x0.64mm_HandSolder"
-			(at 50.8 111.252 90)
+			(at 41.91 111.252 90)
 			(hide yes)
 			(show_name no)
@@
 		)
 		(property "Datasheet" ""
-			(at 50.8 113.03 0)
+			(at 41.91 113.03 0)
 			(hide yes)
 			(show_name no)
@@
 		)
 		(property "Description" "Resistor"
-			(at 50.8 113.03 0)
+			(at 41.91 113.03 0)
 			(hide yes)
 			(show_name no)

Commit message: adjuts placement slightly, reroute
Connections:
- net USB_DM renamed USB_DN
Changed lines of the file:
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@@
 		)
 	)
-	(global_label "USB_DM"
+	(global_label "USB_DN"
 		(shape input)
 		(at 92.71 116.84 180)
@@
 		)
 		(property "Intersheetrefs" "${INTERSHEET_REFS}"
-			(at 82.2258 116.84 0)
+			(at 82.3467 116.84 0)
 			(hide yes)
 			(show_name no)

Commit message: organized schematic, new layouT
Parts:
- SW3, SW4: footprint Button_Switch_SMD:SW_SPST_CK_KMS2xxG -> footprints:NANOT100AS_butt
Other:
- note added: "MHF III antenna not U.FL"
Changed lines of the file:
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@@
 	(generator_version "10.0")
 	(paper "A4")
+	(text "MHF III antenna not U.FL"
+		(exclude_from_sim no)
+		(at 155.448 41.91 0)
+		(effects
+			(font
+				(size 1.27 1.27)
+			)
+		)
+	)
 	(junction
 		(at 179.07 123.19)
@@
 			)
 		)
-		(property "Footprint" "Button_Switch_SMD:SW_SPST_CK_KMS2xxG"
+		(property "Footprint" "footprints:NANOT100AS_butt"
 			(at 184.15 118.11 0)
 			(hide yes)
@@
 			)
 		)
-		(property "Footprint" "Button_Switch_SMD:SW_SPST_CK_KMS2xxG"
+		(property "Footprint" "footprints:NANOT100AS_butt"
 			(at 83.82 53.34 0)
 			(hide yes)

Commit message: no drc errors
Other:
- moved on the sheet: R45
Changed lines of the file:
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@@
 	(global_label "EN"
 		(shape input)
-		(at 119.38 36.83 0)
+		(at 185.42 144.78 0)
 		(fields_autoplaced yes)
 		(effects
@@
 		)
 		(property "Intersheetrefs" "${INTERSHEET_REFS}"
-			(at 124.8447 36.83 0)
+			(at 190.8847 144.78 0)
 			(hide yes)
 			(show_name no)
@@
 	(global_label "3V3"
 		(shape input)
-		(at 111.76 36.83 180)
-		(fields_autoplaced yes)
-		(effects
-			(font
-				(size 1.27 1.27)
-			)
-			(justify right)
-		)
-		(property "Intersheetrefs" "${INTERSHEET_REFS}"
-			(at 105.2672 36.83 0)
+		(at 177.8 144.78 180)
+		(fields_autoplaced yes)
+		(effects
+			(font
+				(size 1.27 1.27)
+			)
+			(justify right)
+		)
+		(property "Intersheetrefs" "${INTERSHEET_REFS}"
+			(at 171.3072 144.78 0)
 			(hide yes)
 			(show_name no)
@@
 	(symbol
 		(lib_id "Device:R")
-		(at 115.57 36.83 90)
+		(at 181.61 144.78 90)
 		(unit 1)
 		(body_style 1)
@@
 		(fields_autoplaced yes)
 		(property "Reference" "R45"
-			(at 115.57 30.48 90)
+			(at 181.61 138.43 90)
 			(show_name no)
 			(do_not_autoplace no)
@@
 		)
 		(property "Value" "10k"
-			(at 115.57 33.02 90)
+			(at 181.61 140.97 90)
 			(show_name no)
 			(do_not_autoplace no)
@@
 		)
 		(property "Footprint" "Resistor_SMD:R_0402_1005Metric_Pad0.72x0.64mm_HandSolder"
-			(at 115.57 38.608 90)
+			(at 181.61 146.558 90)
 			(hide yes)
 			(show_name no)
@@
 		)
 		(property "Datasheet" ""
-			(at 115.57 36.83 0)
+			(at 181.61 144.78 0)
 			(hide yes)
 			(show_name no)
@@
 		)
 		(property "Description" "Resistor"
-			(at 115.57 36.83 0)
-			(hide yes)
-			(show_name no)
+			(at 181.61 144.78 0)
+			(hide yes)
+			(show_name no)
