File: WSG_1.0/WSG_1.0/WSG_1_0_ESP.kicad_sch (KiCad schematic)
At the start: 22 parts, among them SW3 SW_Push, SW4 SW_Push, U15 ESP32-S3-MINI-1U-N8

Commit message: labeled schematic flags, now doing routing stuff
Other:
- note added: "VBAT_SENSE: battery voltage divider"
Changed lines of the file:
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@@
+		)
+	)
+	(text "VBAT_SENSE: battery voltage divider"
+		(exclude_from_sim no)
+		(at 160.528 37.846 0)
+		(effects
+			(font
+				(size 1.27 1.27)
+			)
 		)
 	)
@@
 	)
 	(global_label "BUCK_MODE"
-		(shape input)
+		(shape output)
 		(at 93.98 113.03 180)
 		(fields_autoplaced yes)

Commit message: production files generated
Parts:
- C36: MPN GRM188R60J226MEA0J -> CL10A226MQ8NRNE
Changed lines of the file:
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@@
 			)
 		)
-		(property "MPN" "GRM188R60J226MEA0J"
+		(property "MPN" "CL10A226MQ8NRNE"
 			(at 91.44 44.45 90)
 			(hide yes)

Commit message: diff pair
Connections:
- net USB-: now reaches R34.2, U15.23 (IO19)
- net USB+: now reaches R35.2, U15.24 (IO20)
Other:
- moved on the sheet: R34, R35
Changed lines of the file:
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@@
 	(wire
 		(pts
-			(xy 101.6 115.57) (xy 93.98 115.57)
+			(xy 100.33 113.03) (xy 100.33 101.6)
 		)
 		(stroke
@@
 	(wire
 		(pts
-			(xy 100.33 113.03) (xy 100.33 101.6)
+			(xy 93.98 135.89) (xy 93.98 137.16)
 		)
 		(stroke
@@
 	(wire
 		(pts
-			(xy 93.98 135.89) (xy 93.98 137.16)
+			(xy 95.25 140.97) (xy 92.71 140.97)
 		)
 		(stroke
@@
 	(wire
 		(pts
-			(xy 95.25 140.97) (xy 92.71 140.97)
+			(xy 73.66 120.65) (xy 91.44 120.65)
 		)
 		(stroke
@@
 	(wire
 		(pts
-			(xy 95.25 120.65) (xy 92.71 120.65)
+			(xy 95.25 82.55) (xy 93.98 82.55)
 		)
 		(stroke
@@
 	(wire
 		(pts
-			(xy 95.25 82.55) (xy 93.98 82.55)
+			(xy 111.76 78.74) (xy 95.25 78.74)
 		)
 		(stroke
@@
 	(wire
 		(pts
-			(xy 111.76 78.74) (xy 95.25 78.74)
+			(xy 109.22 111.76) (xy 111.76 111.76)
 		)
 		(stroke
@@
 	(wire
 		(pts
-			(xy 102.87 111.76) (xy 104.14 111.76)
+			(xy 96.52 71.12) (xy 96.52 69.85)
 		)
 		(stroke
@@
 	(wire
 		(pts
-			(xy 96.52 71.12) (xy 96.52 69.85)
+			(xy 96.52 87.63) (xy 96.52 93.98)
 		)
 		(stroke
@@
 	(wire
 		(pts
-			(xy 96.52 87.63) (xy 96.52 93.98)
+			(xy 173.99 124.46) (xy 152.4 124.46)
 		)
 		(stroke
@@
 	(wire
 		(pts
-			(xy 173.99 124.46) (xy 152.4 124.46)
+			(xy 97.79 95.25) (xy 95.25 95.25)
 		)
 		(stroke
@@
 	(wire
 		(pts
-			(xy 97.79 95.25) (xy 95.25 95.25)
+			(xy 106.68 109.22) (xy 111.76 109.22)
 		)
 		(stroke
@@
 	(wire
 		(pts
+			(xy 106.68 116.84) (xy 106.68 109.22)
+		)
+		(stroke
+			(width 0)
+			(type default)
+		)
+	)
+	(wire
+		(pts
 			(xy 153.67 134.62) (xy 153.67 137.16)
 		)
@@
 	(wire
 		(pts
-			(xy 93.98 116.84) (xy 92.71 116.84)
+			(xy 76.2 116.84) (xy 88.9 116.84)
 		)
 		(stroke
@@
 	(wire
 		(pts
-			(xy 95.25 58.42) (xy 95.25 60.96)
+			(xy 99.06 120.65) (xy 109.22 120.65)
 		)
 		(stroke
@@
 	(wire
 		(pts
-			(xy 100.33 135.89) (xy 93.98 135.89)
+			(xy 95.25 58.42) (xy 95.25 60.96)
 		)
 		(stroke
@@
 	(wire
 		(pts
-			(xy 100.33 97.79) (xy 97.79 97.79)
+			(xy 100.33 135.89) (xy 93.98 135.89)
 		)
 		(stroke
@@
 	(wire
 		(pts
-			(xy 90.17 78.74) (xy 91.44 78.74)
+			(xy 100.33 97.79) (xy 97.79 97.79)
 		)
 		(stroke
@@
 	(wire
 		(pts
-			(xy 101.6 109.22) (xy 101.6 115.57)
+			(xy 90.17 78.74) (xy 91.44 78.74)
 		)
 		(stroke
@@
 	(wire
 		(pts
-			(xy 102.87 116.84) (xy 95.25 116.84)
-		)
-		(stroke
-			(width 0)
-			(type default)
-		)
-	)
-	(wire
-		(pts
 			(xy 156.21 132.08) (xy 152.4 132.08)
 		)
@@
 	(wire
 		(pts
-			(xy 93.98 115.57) (xy 93.98 116.84)
+			(xy 109.22 120.65) (xy 109.22 111.76)
 		)
 		(stroke
@@
 	(wire
 		(pts
-			(xy 101.6 109.22) (xy 104.14 109.22)
-		)
-		(stroke
-			(width 0)
-			(type default)
-		)
-	)
-	(wire
-		(pts
 			(xy 109.22 67.31) (xy 109.22 68.58)
 		)
@@
 	(wire
 		(pts
-			(xy 95.25 116.84) (xy 95.25 120.65)
-		)
-		(stroke
-			(width 0)
-			(type default)
-		)
-	)
-	(wire
-		(pts
 			(xy 109.22 68.58) (xy 111.76 68.58)
 		)
@@
 	(wire
 		(pts
-			(xy 102.87 111.76) (xy 102.87 116.84)
-		)
-		(stroke
-			(width 0)
-			(type default)
-		)
-	)
-	(wire
-		(pts
 			(xy 95.25 86.36) (xy 95.25 90.17)
 		)
@@
 	(wire
 		(pts
+			(xy 96.52 116.84) (xy 106.68 116.84)
+		)
+		(stroke
+			(width 0)
+			(type default)
+		)
+	)
+	(wire
+		(pts
 			(xy 97.79 83.82) (xy 97.79 86.36)
 		)
@@
 		)
 	)
+	(label "USB+"
+		(at 102.87 120.65 0)
+		(effects
+			(font
+				(size 1.27 1.27)
+			)
+			(justify left bottom)
+		)
+	)
+	(label "USB-"
+		(at 100.33 116.84 0)
+		(effects
+			(font
+				(size 1.27 1.27)
+			)
+			(justify left bottom)
+		)
+	)
 	(global_label "FLASH_MOSI"
 		(shape output)
@@
 	(global_label "USB_DN"
 		(shape bidirectional)
-		(at 92.71 116.84 180)
+		(at 76.2 116.84 180)
 		(fields_autoplaced yes)
 		(effects
@@
 		)
 		(property "Intersheetrefs" "${INTERSHEET_REFS}"
-			(at 81.2354 116.84 0)
+			(at 64.7254 116.84 0)
 			(hide yes)
 			(show_name no)
@@
 	(global_label "USB_DP"
 		(shape bidirectional)
-		(at 92.71 120.65 180)
+		(at 73.66 120.65 180)
 		(fields_autoplaced yes)
 		(effects
@@
 		)
 		(property "Intersheetrefs" "${INTERSHEET_REFS}"
-			(at 81.2959 120.65 0)
+			(at 62.2459 120.65 0)
 			(hide yes)
 			(show_name no)
@@
 	(symbol
 		(lib_id "Device:R")
-		(at 107.95 109.22 90)
+		(at 92.71 116.84 90)
 		(unit 1)
 		(body_style 1)
@@
 		(fields_autoplaced yes)
 		(property "Reference" "R34"
-			(at 107.95 102.87 90)
+			(at 92.71 110.49 90)
 			(show_name no)
 			(do_not_autoplace no)
@@
 		)
 		(property "Value" "22"
-			(at 107.95 105.41 90)
+			(at 92.71 113.03 90)
 			(show_name no)
 			(do_not_autoplace no)
@@
 		)
 		(property "Footprint" "Resistor_SMD:R_0402_1005Metric_Pad0.72x0.64mm_HandSolder"
-			(at 107.95 110.998 90)
+			(at 92.71 118.618 90)
 			(hide yes)
 			(show_name no)
@@
 		)
 		(property "Datasheet" ""
-			(at 107.95 109.22 0)
+			(at 92.71 116.84 0)
 			(hide yes)
 			(show_name no)
@@
 		)
 		(property "Description" "Resistor"
-			(at 107.95 109.22 0)
+			(at 92.71 116.84 0)
 			(hide yes)
 			(show_name no)
@@
 	(symbol
 		(lib_id "Device:R")
-		(at 107.95 111.76 90)
+		(at 95.25 120.65 90)
 		(unit 1)
 		(body_style 1)
@@
 		(dnp no)
 		(property "Reference" "R35"
-			(at 107.696 114.808 90)
+			(at 94.996 123.698 90)
 			(show_name no)
 			(do_not_autoplace no)
@@
 		)
 		(property "Value" "22"
-			(at 107.696 117.348 90)
+			(at 94.996 126.238 90)
 			(show_name no)
 			(do_not_autoplace no)
@@
 		)
 		(property "Footprint" "Resistor_SMD:R_0402_1005Metric_Pad0.72x0.64mm_HandSolder"
-			(at 107.95 113.538 90)
+			(at 95.25 122.428 90)
 			(hide yes)
 			(show_name no)
@@
 		)
 		(property "Datasheet" ""
-			(at 107.95 111.76 0)
+			(at 95.25 120.65 0)
 			(hide yes)
 			(show_name no)
@@
 		)
 		(property "Description" "Resistor"
-			(at 107.95 111.76 0)
+			(at 95.25 120.65 0)
 			(hide yes)
 			(show_name no)
