File: 02-main_board[main_board_v1]/analog processing.kicad_sch (KiCad schematic)
At the start: 27 parts, among them IC1 AD7175-8BCPZ-RL7

Commit message: Updated with changes from PDR
Parts:
- added R22: 10k, symbol Device:R
Connections:
- net 5V_ref is gone; now on net 5V_stable: C9.1, IC1.40 (REF+)
- net !CS_adc: now also R22.1
- net 3.3V_teensy: now also R22.2
- net 5V renamed 5V_stable
Changed lines of the file:
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@@
 	(rectangle
 		(start 25.4 27.94)
-		(end 140.97 139.7)
+		(end 140.97 147.32)
 		(stroke
 			(width 0)
@@
 	)
 	(junction
+		(at 86.36 133.35)
+		(diameter 0)
+		(color 0 0 0 0)
+	)
+	(junction
 		(at 179.07 104.14)
 		(diameter 0)
@@
 	(wire
 		(pts
+			(xy 86.36 133.35) (xy 86.36 119.38)
+		)
+		(stroke
+			(width 0)
+			(type default)
+		)
+	)
+	(wire
+		(pts
 			(xy 73.66 45.72) (xy 73.66 46.99)
 		)
@@
 	(wire
 		(pts
+			(xy 86.36 135.89) (xy 86.36 133.35)
+		)
+		(stroke
+			(width 0)
+			(type default)
+		)
+	)
+	(wire
+		(pts
 			(xy 172.72 46.99) (xy 179.07 46.99)
 		)
@@
 		(pts
 			(xy 125.73 93.98) (xy 115.57 93.98)
+		)
+		(stroke
+			(width 0)
+			(type default)
+		)
+	)
+	(wire
+		(pts
+			(xy 85.09 133.35) (xy 86.36 133.35)
 		)
 		(stroke
@@
 	(global_label "!CS_adc"
 		(shape input)
-		(at 86.36 119.38 270)
+		(at 86.36 135.89 270)
 		(fields_autoplaced yes)
 		(effects
@@
 		)
 		(property "Intersheetrefs" "${INTERSHEET_REFS}"
-			(at 86.36 129.8037 90)
+			(at 86.36 146.3137 90)
 			(effects
 				(font
@@
 		)
 	)
-	(global_label "5V"
-		(shape input)
-		(at 49.53 91.44 180)
-		(fields_autoplaced yes)
-		(effects
-			(font
-				(size 1.27 1.27)
-			)
-			(justify right)
-		)
-		(property "Intersheetrefs" "${INTERSHEET_REFS}"
-			(at 44.2467 91.44 0)
-			(effects
-				(font
-					(size 1.27 1.27)
-				)
-				(justify right)
-				(hide yes)
-			)
-		)
-	)
 	(global_label "filtered_6"
 		(shape output)
@@
 		)
 	)
+	(global_label "3.3V_teensy"
+		(shape input)
+		(at 77.47 133.35 180)
+		(fields_autoplaced yes)
+		(effects
+			(font
+				(size 1.27 1.27)
+			)
+			(justify right)
+		)
+		(property "Intersheetrefs" "${INTERSHEET_REFS}"
+			(at 63.3572 133.35 0)
+			(effects
+				(font
+					(size 1.27 1.27)
+				)
+				(justify right)
+				(hide yes)
+			)
+		)
+	)
 	(global_label "MOSI_adc"
 		(shape input)
@@
 		)
 	)
+	(global_label "5V_stable"
+		(shape input)
+		(at 49.53 91.44 180)
+		(fields_autoplaced yes)
+		(effects
+			(font
+				(size 1.27 1.27)
+			)
+			(justify right)
+		)
+		(property "Intersheetrefs" "${INTERSHEET_REFS}"
+			(at 37.4735 91.44 0)
+			(effects
+				(font
+					(size 1.27 1.27)
+				)
+				(justify right)
+				(hide yes)
+			)
+		)
+	)
 	(global_label "MISO_adc"
 		(shape input)
@@
 		)
 	)
-	(global_label "5V_ref"
+	(global_label "5V_stable"
 		(shape input)
 		(at 73.66 45.72 90)
@@
 		)
 		(property "Intersheetrefs" "${INTERSHEET_REFS}"
-			(at 73.66 36.8686 90)
+			(at 73.66 33.6635 90)
 			(effects
 				(font
@@
 					(unit 1)
 				)
+			)
+		)
+	)
+	(symbol
+		(lib_id "Device:R")
+		(at 81.28 133.35 270)
+		(unit 1)
+		(exclude_from_sim no)
+		(in_bom yes)
+		(on_board yes)
+		(dnp no)
+		(property "Reference" "R22"
+			(at 81.28 135.89 90)
+			(effects
+				(font
+					(size 1.27 1.27)
+				)
+			)
+		)
+		(property "Value" "10k"
+			(at 81.28 138.43 90)
+			(effects
+				(font
+					(size 1.27 1.27)
+				)
+			)
+		)
+		(property "Footprint" ""
+			(at 81.28 131.572 90)
+			(effects
+				(font
+					(size 1.27 1.27)
+				)
+				(hide yes)
+			)
+		)
+		(property "Datasheet" "~"
+			(at 81.28 133.35 0)
+			(effects
+				(font
+					(size 1.27 1.27)
+				)
+				(hide yes)
+			)
+		)
+		(property "Description" "Resistor"
+			(at 81.28 133.35 0)
+			(effects
+				(font
+					(size 1.27 1.27)
+				)
+				(hide yes)
+			)
+		)
+		(pin "1"
+		)
+		(pin "2"
+		)
+		(instances
+			(project ""
+				(path "/0ba8c130-372e-4349-9fc9-4ef188509568/92ce0411-43bd-4a5b-b429-16cad50bc1ec"
+					(reference "R22")
+					(unit 1)
+				)

Commit message: first rev
Parts:
- C10, C11, C12, C13, C14, C15, C16, C17, C18, C19, C20, C21, C22, C23, C9: footprint (none) -> Capacitor_SMD:C_0402_1005Metric
- IC1: footprint QFN50P600X600X80-41N-D -> footprints:AD7175-8BCPZ-RL7
- R10, R22, R3, R4, R5, R6, R7, R8, R9: footprint (none) -> Resistor_SMD:R_0402_1005Metric
- TP5, TP6, TP7: footprint (none) -> TestPoint:TestPoint_Pad_1.0x1.0mm
Connections:
- net filtered_1: now also IC1.31 (AIN9); no longer IC1.4 (AIN2)
- net filtered_2: now also IC1.32 (AIN10); no longer IC1.5 (AIN3)
- net filtered_3: now also IC1.33 (AIN11); no longer IC1.26 (AIN4)
- net filtered_4: now also IC1.34 (AIN12); no longer IC1.27 (AIN5)
- net filtered_5: now also IC1.35 (AIN13); no longer IC1.28 (AIN6)
- net filtered_6: now also IC1.36 (AIN14); no longer IC1.29 (AIN7)
- net filtered_7: now also IC1.37 (AIN15); no longer IC1.30 (AIN8)
- net filtered_8: now also IC1.38 (GPO3); no longer IC1.31 (AIN9)
Other:
- moved on the sheet: C9
