File: 02-main_board[main_board_v1]/analog processing.kicad_sch (KiCad schematic)
At the start: 28 parts, among them IC1 AD7175-8BCPZ-RL7

Commit message: this is what i ordered
Parts:
- C10, C11, C12, C13, C14, C16, C17, C18, C20, C21, C22, C23, C24: MPN (none) -> CC0603KRX7R9BB104; Manufacturer (none) -> YAGEO
- C15, C19: MPN (none) -> CL10A105KA8NFNC; Manufacturer (none) -> Samsung Electro-Mechanics
- IC1: MPN (none) -> AD7175-8BCPZ-RL7; Manufacturer (none) -> Analog Devices; Manufacturer_Name Analog Devices -> (none)
- R10, R11, R12, R13, R14, R7, R8, R9: MPN (none) -> RC0603FR-072K2L; Manufacturer (none) -> YAGEO
- R15: MPN (none) -> CRCW060310K0FKEA; Manufacturer (none) -> Vishay Dale
