File: 02-main_board[main_board_v1]/esp32.kicad_sch (KiCad schematic)
At the start: 5 parts, among them Q1 XIAO_ESP32S3

Commit message: Updated with changes from PDR
Parts:
- added R21: 10k, symbol Device:R
Connections:
- net CS_esp32: now also R21.2
- net JTAG_esp32 renamed handshake_esp32
- new net 3.3V_teensy: R21.1
Other:
- moved on the sheet: TP8, TP9
Changed lines of the file:
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@@
+		(color 0 0 0 0)
+	)
+	(junction
+		(at 41.91 57.15)
+		(diameter 0)
 		(color 0 0 0 0)
 	)
@@
 	(no_connect
 		(at 78.74 62.23)
+	)
+	(wire
+		(pts
+			(xy 41.91 58.42) (xy 41.91 57.15)
+		)
+		(stroke
+			(width 0)
+			(type default)
+		)
+	)
+	(wire
+		(pts
+			(xy 41.91 68.58) (xy 40.64 68.58)
+		)
+		(stroke
+			(width 0)
+			(type default)
+		)
+	)
+	(wire
+		(pts
+			(xy 41.91 57.15) (xy 45.72 57.15)
+		)
+		(stroke
+			(width 0)
+			(type default)
+		)
 	)
 	(wire
@@
 		)
 	)
+	(wire
+		(pts
+			(xy 38.1 57.15) (xy 41.91 57.15)
+		)
+		(stroke
+			(width 0)
+			(type default)
+		)
+	)
+	(wire
+		(pts
+			(xy 41.91 68.58) (xy 41.91 66.04)
+		)
+		(stroke
+			(width 0)
+			(type default)
+		)
+	)
 	(global_label "MOSI_esp32"
 		(shape input)
@@
 	(global_label "MISO_esp32"
 		(shape input)
-		(at 43.18 74.93 0)
+		(at 71.12 85.09 0)
 		(fields_autoplaced yes)
 		(effects
@@
 		)
 		(property "Intersheetrefs" "${INTERSHEET_REFS}"
-			(at 57.4137 74.93 0)
+			(at 85.3537 85.09 0)
 			(effects
 				(font
@@
 				)
 				(justify left)
+				(hide yes)
+			)
+		)
+	)
+	(global_label "3.3V_teensy"
+		(shape input)
+		(at 40.64 68.58 180)
+		(fields_autoplaced yes)
+		(effects
+			(font
+				(size 1.27 1.27)
+			)
+			(justify right)
+		)
+		(property "Intersheetrefs" "${INTERSHEET_REFS}"
+			(at 26.5272 68.58 0)
+			(effects
+				(font
+					(size 1.27 1.27)
+				)
+				(justify right)
 				(hide yes)
 			)
@@
 	(global_label "MOSI_esp32"
 		(shape input)
-		(at 43.18 85.09 0)
+		(at 71.12 95.25 0)
 		(fields_autoplaced yes)
 		(effects
@@
 		)
 		(property "Intersheetrefs" "${INTERSHEET_REFS}"
-			(at 57.4137 85.09 0)
+			(at 85.3537 95.25 0)
 			(effects
 				(font
@@
 	(global_label "CS_esp32"
 		(shape input)
-		(at 45.72 57.15 180)
+		(at 38.1 57.15 180)
 		(fields_autoplaced yes)
 		(effects
@@
 		)
 		(property "Intersheetrefs" "${INTERSHEET_REFS}"
-			(at 33.603 57.15 0)
+			(at 25.983 57.15 0)
 			(effects
 				(font
@@
 		)
 	)
-	(global_label "JTAG_esp32"
+	(global_label "handshake_esp32"
 		(shape bidirectional)
 		(at 45.72 52.07 180)
@@
 		)
 		(property "Intersheetrefs" "${INTERSHEET_REFS}"
-			(at 30.6774 52.07 0)
+			(at 24.9324 52.07 0)
 			(effects
 				(font
@@
 				(path "/0ba8c130-372e-4349-9fc9-4ef188509568/5fc2e8ea-ad51-4d94-b167-6ce076215cd3"
 					(reference "C31")
+					(unit 1)
+				)
+			)
+		)
+	)
+	(symbol
+		(lib_id "Device:R")
+		(at 41.91 62.23 180)
+		(unit 1)
+		(exclude_from_sim no)
+		(in_bom yes)
+		(on_board yes)
+		(dnp no)
+		(property "Reference" "R21"
+			(at 36.83 60.96 0)
+			(effects
+				(font
+					(size 1.27 1.27)
+				)
+				(justify right)
+			)
+		)
+		(property "Value" "10k"
+			(at 36.83 63.5 0)
+			(effects
+				(font
+					(size 1.27 1.27)
+				)
+				(justify right)
+			)
+		)
+		(property "Footprint" ""
+			(at 43.688 62.23 90)
+			(effects
+				(font
+					(size 1.27 1.27)
+				)
+				(hide yes)
+			)
+		)
+		(property "Datasheet" "~"
+			(at 41.91 62.23 0)
+			(effects
+				(font
+					(size 1.27 1.27)
+				)
+				(hide yes)
+			)
+		)
+		(property "Description" "Resistor"
+			(at 41.91 62.23 0)
+			(effects
+				(font
+					(size 1.27 1.27)
+				)
+				(hide yes)
+			)
+		)
+		(pin "2"
+		)
+		(pin "1"
+		)
+		(instances
+			(project ""
+				(path "/0ba8c130-372e-4349-9fc9-4ef188509568/5fc2e8ea-ad51-4d94-b167-6ce076215cd3"
+					(reference "R21")
 					(unit 1)
 				)
@@
 	(symbol
 		(lib_id "Connector:TestPoint")
-		(at 43.18 74.93 90)
+		(at 71.12 85.09 90)
 		(unit 1)
 		(exclude_from_sim no)
@@
 		(dnp no)
 		(property "Reference" "TP8"
-			(at 39.878 69.85 90)
+			(at 67.818 80.01 90)
 			(effects
 				(font
@@
 		)
 		(property "Value" "MISO_esp32"
-			(at 39.878 72.39 90)
+			(at 67.818 82.55 90)
 			(effects
 				(font
@@
 		)
 		(property "Footprint" ""
-			(at 43.18 69.85 0)
+			(at 71.12 80.01 0)
 			(effects
 				(font
@@
 		)
 		(property "Datasheet" "~"
-			(at 43.18 69.85 0)
+			(at 71.12 80.01 0)
 			(effects
 				(font
@@
 		)
 		(property "Description" "test point"
-			(at 43.18 74.93 0)
+			(at 71.12 85.09 0)
 			(effects
 				(font
@@
 	(symbol
 		(lib_id "Connector:TestPoint")
-		(at 43.18 85.09 90)
+		(at 71.12 95.25 90)
 		(unit 1)
 		(exclude_from_sim no)
@@
 		(dnp no)
 		(property "Reference" "TP9"
-			(at 39.878 80.01 90)
+			(at 67.818 90.17 90)
 			(effects
 				(font
@@
 		)
 		(property "Value" "MOSI_esp32"
-			(at 39.878 82.55 90)
+			(at 67.818 92.71 90)
 			(effects
 				(font
@@
 		)
 		(property "Footprint" ""
-			(at 43.18 80.01 0)
+			(at 71.12 90.17 0)
 			(effects
 				(font
@@
 		)
 		(property "Datasheet" "~"
-			(at 43.18 80.01 0)
+			(at 71.12 90.17 0)
 			(effects
 				(font
@@
 		)
 		(property "Description" "test point"
-			(at 43.18 85.09 0)
-			(effects
-				(font
+			(at 71.12 95.25 0)
+			(effects
+				(font

Commit message: first rev
Parts:
- C31: footprint (none) -> Capacitor_SMD:C_0402_1005Metric
- R21: footprint (none) -> Resistor_SMD:R_0402_1005Metric
- TP10, TP8, TP9: footprint (none) -> TestPoint:TestPoint_Pad_1.0x1.0mm
Changed lines of the file:
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@@
 			)
 		)
-		(property "Footprint" ""
+		(property "Footprint" "Capacitor_SMD:C_0402_1005Metric"
 			(at 100.6348 46.99 0)
 			(effects
@@
 			)
 		)
-		(property "Footprint" ""
+		(property "Footprint" "Resistor_SMD:R_0402_1005Metric"
 			(at 43.688 62.23 90)
 			(effects
@@
 			)
 		)
-		(property "Footprint" ""
+		(property "Footprint" "TestPoint:TestPoint_Pad_1.0x1.0mm"
 			(at 71.12 69.85 0)
 			(effects
@@
 			)
 		)
-		(property "Footprint" ""
+		(property "Footprint" "TestPoint:TestPoint_Pad_1.0x1.0mm"
 			(at 71.12 80.01 0)
 			(effects
@@
 			)
 		)
-		(property "Footprint" ""
+		(property "Footprint" "TestPoint:TestPoint_Pad_1.0x1.0mm"
 			(at 71.12 90.17 0)
 			(effects
