File: 02-main_board[main_board_v1]/02-main_board[main_board_v1].kicad_sch (KiCad schematic)
At the start: 0 parts

Commit message: finished schematic v1
Parts:
- added BT1: Battery_Cell, symbol Device:Battery_Cell
- added C32: 0.1uF, symbol Device:C
- added R19, R20: 47, symbol Device:R
- added U4: Teensy4.1, footprints:Teensy41, symbol symbols:Teensy4.1
Connections:
- new net: BT1.1 (+), U4.50 (VBAT)
- new net: R20.2, U4.26 (34_RX8)
- new net: R19.1, U4.27 (35_TX8)
- new net !CS_adc: U4.29 (37_CS)
- new net !ERROR_adc: U4.33 (41_A17)
- new net 3.3V_teensy: U4.46 (3V3)
- new net 5V: C32.2, U4.48 (VIN)
- new net CS_esp32: U4.28 (36_CS)
- new net GNDD: BT1.2 (-), U4.1 (GND), U4.47 (GND), U4.52 (GND), U4.58 (GND), U4.59 (GND), U4.64 (GND)
- new net GNDPWR: C32.1
- new net GP/Int1: R19.2
- new net GP/Int2: R20.1
- new net HFX_3.3V_3: U4.45 (23_A9_CRX1_MCLK1)
- new net HFX_3.3V_cvt: U4.43 (21_A7_RX5_BCLK1)
- new net HFX_3.3V_eng: U4.44 (22_A8_CTX1)
- new net JTAG_esp32: U4.41 (19_A5_SCL)
- new net LED_CONTROL: U4.39 (17_A3_TX4_SDA1)
- new net MISO_adc: U4.31 (39_MISO1_OUT1A)
- new net MISO_esp32: U4.14 (12_MISO_MQSL)
- new net MOSI_adc: U4.18 (26_A12_MOSI1)
- new net MOSI_esp32: U4.13 (11_MOSI_CTX1)
- new net RD+: U4.60 (R+)
- new net RD-: U4.65 (R-)
- new net RXD: U4.2 (0_RX1_CRX2_CS1)
- new net SCLK_adc: U4.19 (27_A13_SCK1)
- new net SCLK_esp32: U4.35 (13_SCK_LED)
- new net STBY_can: U4.4 (2_OUT2)
- new net TD+: U4.63 (T+)
- new net TD-: U4.62 (T-)
- new net TXD: U4.3 (1_TX1_CTX2_MISO1)
- new net USB_D_N: U4.66 (D-)
- new net USB_D_P: U4.67 (D+)
- new net USB_SEL: U4.38 (16_A2_RX4_SCL1)
- no-connect marks 0 -> 32
Other:
- added sheet analog processing (analog processing.kicad_sch)
- added sheet connectors (connectors.kicad_sch)
- added sheet digital processing (digital processing.kicad_sch)
- added sheet esp32 (esp32.kicad_sch)

Commit message: Updated with changes from PDR
Connections:
- net !OE_lvlshift: now reaches U4.6 (4_BCLK2)
- net JTAG_esp32 renamed handshake_esp32
- no-connect marks 32 -> 31
Changed lines of the file:
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@@
-	)
-	(no_connect
-		(at 186.69 49.53)
 	)
 	(no_connect
@@
 		)
 	)
-	(global_label "JTAG_esp32"
+	(global_label "handshake_esp32"
 		(shape bidirectional)
 		(at 242.57 54.61 0)
@@
 		)
 		(property "Intersheetrefs" "${INTERSHEET_REFS}"
-			(at 257.6126 54.61 0)
+			(at 263.3576 54.61 0)
 			(effects
 				(font
@@
 				(hide yes)
 			)
+		)
+	)
+	(global_label "!OE_lvlshift"
+		(shape output)
+		(at 186.69 49.53 180)
+		(fields_autoplaced yes)
+		(effects
+			(font
+				(size 1.27 1.27)
+			)
+			(justify right)
+		)
+		(property "Intersheetrefs" "${INTERSHEET_REFS}"
+			(at 173.1216 49.53 0)
+			(effects
+				(font
+					(size 1.27 1.27)
+				)
+				(justify right)
+				(hide yes)
+			)

Commit message: first rev
Parts:
- added H3, H4, H5, H6: MountingHole_Pad, MountingHole:MountingHole_2.5mm_Pad, symbol Mechanical:MountingHole_Pad
- added NT1: NetTie_1, NetTie:NetTie-2_THT_Pad0.3mm, symbol Device:NetTie_2
- added NT2: NetTie_2, NetTie:NetTie-2_THT_Pad0.3mm, symbol Device:NetTie_2
- BT1: footprint (none) -> footprints:BAT-HLD-012-SMT_TEC
- C32: footprint (none) -> Capacitor_SMD:C_0402_1005Metric
- R19, R20: footprint (none) -> Resistor_SMD:R_0402_1005Metric
Connections:
- net !ERROR_adc: now also U4.20 (28_RX7); no longer U4.33 (41_A17)
- net !OE_lvlshift: now also U4.36 (14_A0_TX3_SPDIF_OUT); no longer U4.6 (4_BCLK2)
- net GNDD: now also NT2.1; no longer BT1.2 (-)
- net GNDPWR: now also BT1.2 (-), H3.1, H5.1, NT1.2, NT2.2
- net HFX_3.3V_3: now also U4.39 (17_A3_TX4_SDA1); no longer U4.45 (23_A9_CRX1_MCLK1)
- net HFX_3.3V_cvt: now also U4.37 (15_A1_RX3_SPDIF_IN); no longer U4.43 (21_A7_RX5_BCLK1)
- net HFX_3.3V_eng: now also U4.38 (16_A2_RX4_SCL1); no longer U4.44 (22_A8_CTX1)
- net LED_CONTROL: now also U4.9 (7_RX2_OUT1A); no longer U4.39 (17_A3_TX4_SDA1)
- net USB_SEL: now also U4.8 (6_OUT1D); no longer U4.38 (16_A2_RX4_SCL1)
- net handshake_esp32: now also U4.6 (4_BCLK2); no longer U4.41 (19_A5_SCL)
- new net GNDA: H4.1, H6.1, NT1.1
- no-connect marks 31 -> 32

Commit message: first rev ready for design review
Parts:
- removed NT1: NetTie_1, NetTie:NetTie-2_THT_Pad0.3mm, symbol Device:NetTie_2
- removed NT2: NetTie_2, NetTie:NetTie-2_THT_Pad0.3mm, symbol Device:NetTie_2
- BT1: footprint footprints:BAT-HLD-012-SMT_TEC -> footprints:BatteryHolder_LINX_BAT-HLD-012-SMT
Connections:
- net GNDD is gone; now on net GNDA: U4.1 (GND), U4.47 (GND), U4.52 (GND), U4.58 (GND), U4.59 (GND), U4.64 (GND)
- net GNDPWR is gone; now on net GNDA: BT1.2 (-), C32.1, H3.1, H5.1
- no-connect marks 32 -> 31
Changed lines of the file:
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@@
-	)
-	(no_connect
-		(at 55.88 -1.27)
 	)
 	(no_connect
@@
 	(no_connect
 		(at 186.69 87.63)
-	)
-	(bus_entry
-		(at 195.58 165.1)
-		(size 2.54 2.54)
-		(stroke
-			(width 0)
-			(type default)
-		)
-	)
-	(bus_entry
-		(at 208.28 165.1)
-		(size 2.54 2.54)
-		(stroke
-			(width 0)
-			(type default)
-		)
 	)
 	(wire
@@
 			)
 		)
-		(property "Footprint" "footprints:BAT-HLD-012-SMT_TEC"
+		(property "Footprint" "footprints:BatteryHolder_LINX_BAT-HLD-012-SMT"
 			(at 207.01 134.366 90)
 			(effects
@@
 	)
 	(symbol
-		(lib_id "Device:NetTie_2")
-		(at 80.01 156.21 0)
-		(unit 1)
-		(exclude_from_sim no)
-		(in_bom no)
-		(on_board yes)
-		(dnp no)
-		(fields_autoplaced yes)
-		(property "Reference" "NT1"
-			(at 80.01 151.13 0)
-			(effects
-				(font
-					(size 1.27 1.27)
-				)
-			)
-		)
-		(property "Value" "NetTie_1"
-			(at 80.01 153.67 0)
-			(effects
-				(font
-					(size 1.27 1.27)
-				)
-			)
-		)
-		(property "Footprint" "NetTie:NetTie-2_THT_Pad0.3mm"
-			(at 80.01 156.21 0)
-			(effects
-				(font
-					(size 1.27 1.27)
-				)
-				(hide yes)
-			)
-		)
-		(property "Datasheet" "~"
-			(at 80.01 156.21 0)
-			(effects
-				(font
-					(size 1.27 1.27)
-				)
-				(hide yes)
-			)
-		)
-		(property "Description" "Net tie, 2 pins"
-			(at 80.01 156.21 0)
-			(effects
-				(font
-					(size 1.27 1.27)
-				)
-				(hide yes)
-			)
-		)
-		(pin "1"
-		)
-		(pin "2"
-		)
-		(instances
-			(project ""
-				(path "/0ba8c130-372e-4349-9fc9-4ef188509568"
-					(reference "NT1")
-					(unit 1)
-				)
-			)
-		)
-	)
-	(symbol
 		(lib_id "Mechanical:MountingHole_Pad")
 		(at 38.1 166.37 270)
@@
 	)
 	(symbol
-		(lib_id "Device:NetTie_2")
-		(at 80.01 163.83 0)
-		(unit 1)
-		(exclude_from_sim no)
-		(in_bom no)
-		(on_board yes)
-		(dnp no)
-		(fields_autoplaced yes)
-		(property "Reference" "NT2"
-			(at 80.01 158.75 0)
-			(effects
-				(font
-					(size 1.27 1.27)
-				)
-			)
-		)
-		(property "Value" "NetTie_2"
-			(at 80.01 161.29 0)
-			(effects
-				(font
-					(size 1.27 1.27)
-				)
-			)
-		)
-		(property "Footprint" "NetTie:NetTie-2_THT_Pad0.3mm"
-			(at 80.01 163.83 0)
-			(effects
-				(font
-					(size 1.27 1.27)
-				)
-				(hide yes)
-			)
-		)
-		(property "Datasheet" "~"
-			(at 80.01 163.83 0)
-			(effects
-				(font
-					(size 1.27 1.27)
-				)
-				(hide yes)
-			)
-		)
-		(property "Description" "Net tie, 2 pins"
-			(at 80.01 163.83 0)
-			(effects
-				(font
-					(size 1.27 1.27)
-				)
-				(hide yes)
-			)
-		)
-		(pin "1"
-		)
-		(pin "2"
-		)
-		(instances
-			(project "02-main_board[main_board_v1]"
-				(path "/0ba8c130-372e-4349-9fc9-4ef188509568"
-					(reference "NT2")
-					(unit 1)
-				)
-			)
-		)
-	)
-	(symbol
 		(lib_id "power:GNDPWR")
-		(at 82.55 156.21 90)
+		(at 77.47 156.21 90)
 		(unit 1)
 		(exclude_from_sim no)
@@
 		(fields_autoplaced yes)
 		(property "Reference" "#PWR039"
-			(at 87.63 156.21 0)
+			(at 82.55 156.21 0)
 			(effects
 				(font
@@
 		)
 		(property "Value" "GNDPWR"
-			(at 86.36 156.3369 90)
+			(at 81.28 156.3369 90)
 			(effects
 				(font
@@
 		)
 		(property "Footprint" ""
-			(at 83.82 156.21 0)
+			(at 78.74 156.21 0)
 			(effects
 				(font
@@
 		)
 		(property "Datasheet" ""
-			(at 83.82 156.21 0)
+			(at 78.74 156.21 0)
 			(effects
 				(font
@@
 		)
 		(property "Description" "Power symbol creates a global label with name \"GNDPWR\" , global ground"
-			(at 82.55 156.21 0)
+			(at 77.47 156.21 0)
 			(effects
 				(font
@@
 	(symbol
 		(lib_id "power:GNDPWR")
-		(at 82.55 163.83 90)
+		(at 77.47 163.83 90)
 		(unit 1)
 		(exclude_from_sim no)
@@
 		(fields_autoplaced yes)
 		(property "Reference" "#PWR085"
-			(at 87.63 163.83 0)
+			(at 82.55 163.83 0)
 			(effects
 				(font
@@
 		)
 		(property "Value" "GNDPWR"
-			(at 86.36 163.9569 90)
+			(at 81.28 163.9569 90)
 			(effects
 				(font
@@
 		)
 		(property "Footprint" ""
-			(at 83.82 163.83 0)
+			(at 78.74 163.83 0)
 			(effects
 				(font
@@
 		)
 		(property "Datasheet" ""
-			(at 83.82 163.83 0)
+			(at 78.74 163.83 0)
 			(effects
 				(font
@@
 		)
 		(property "Description" "Power symbol creates a global label with name \"GNDPWR\" , global ground"
-			(at 82.55 163.83 0)
-			(effects
-				(font
+			(at 77.47 163.83 0)
+			(effects
+				(font
