File: 02-main_board[main_board_v1]/02-main_board[main_board_v1].kicad_sch (KiCad schematic)
At the start: 9 parts, among them U1 Teensy4.1

Commit message: this is what i ordered
Parts:
- C1: MPN (none) -> CC0603KRX7R9BB104; Manufacturer (none) -> YAGEO
- R1, R2: MPN (none) -> RC0603JR-0747RL; Manufacturer (none) -> YAGEO
Changed lines of the file:
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@@
+			)
+		)
+		(property "MPN" "RC0603JR-0747RL"
+			(at 257.81 90.17 90)
+			(effects
+				(font
+					(size 1.27 1.27)
+				)
+				(hide yes)
+			)
+		)
+		(property "Manufacturer" "YAGEO"
+			(at 257.81 90.17 90)
+			(effects
+				(font
+					(size 1.27 1.27)
+				)
+				(hide yes)
 			)
 		)
@@
 			)
 		)
+		(property "MPN" "CC0603KRX7R9BB104"
+			(at 262.89 40.64 0)
+			(effects
+				(font
+					(size 1.27 1.27)
+				)
+				(hide yes)
+			)
+		)
+		(property "Manufacturer" "YAGEO"
+			(at 262.89 40.64 0)
+			(effects
+				(font
+					(size 1.27 1.27)
+				)
+				(hide yes)
+			)
+		)
 		(pin "1"
 		)
@@
 			(effects
 				(font
+					(size 1.27 1.27)
+				)
+				(hide yes)
+			)
+		)
+		(property "MPN" "RC0603JR-0747RL"
+			(at 257.81 92.71 90)
+			(effects
+				(font
+					(size 1.27 1.27)
+				)
+				(hide yes)
+			)
+		)
+		(property "Manufacturer" "YAGEO"
+			(at 257.81 92.71 90)
+			(effects
+				(font
