File: 02-main_board[main_board_v1]/connectors.kicad_sch (KiCad schematic)
At the start: 3 parts, among them J1 2-84952-0, J2 2-84952-4, J3 FH41-15S-0.5SH_05_

Commit message: Updated with changes from PDR
Connections:
- net 5V_ref is gone; now on net GNDPWR: J2.20
- net 5V: no longer J1.19, J1.20
- new net 5V_stable: J1.19, J1.20
Changed lines of the file:
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@@
+		)
+	)
+	(global_label "5V_stable"
+		(shape output)
+		(at 58.42 82.55 180)
+		(fields_autoplaced yes)
+		(effects
+			(font
+				(size 1.27 1.27)
+			)
+			(justify right)
+		)
+		(property "Intersheetrefs" "${INTERSHEET_REFS}"
+			(at 46.3635 82.55 0)
+			(effects
+				(font
+					(size 1.27 1.27)
+				)
+				(justify right)
+				(hide yes)
+			)
 		)
 	)
@@
 		)
 	)
+	(global_label "5V_stable"
+		(shape output)
+		(at 58.42 80.01 180)
+		(fields_autoplaced yes)
+		(effects
+			(font
+				(size 1.27 1.27)
+			)
+			(justify right)
+		)
+		(property "Intersheetrefs" "${INTERSHEET_REFS}"
+			(at 46.3635 80.01 0)
+			(effects
+				(font
+					(size 1.27 1.27)
+				)
+				(justify right)
+				(hide yes)
+			)
+		)
+	)
 	(global_label "5V"
 		(shape input)
@@
 		)
 	)
-	(global_label "5V"
-		(shape output)
-		(at 58.42 80.01 180)
-		(fields_autoplaced yes)
-		(effects
-			(font
-				(size 1.27 1.27)
-			)
-			(justify right)
-		)
-		(property "Intersheetrefs" "${INTERSHEET_REFS}"
-			(at 53.1367 80.01 0)
-			(effects
-				(font
-					(size 1.27 1.27)
-				)
-				(justify right)
-				(hide yes)
-			)
-		)
-	)
 	(global_label "HFX_5V_eng"
 		(shape output)
@@
 		)
 	)
-	(global_label "5V_ref"
-		(shape input)
-		(at 123.19 82.55 180)
-		(fields_autoplaced yes)
-		(effects
-			(font
-				(size 1.27 1.27)
-			)
-			(justify right)
-		)
-		(property "Intersheetrefs" "${INTERSHEET_REFS}"
-			(at 114.3386 82.55 0)
-			(effects
-				(font
-					(size 1.27 1.27)
-				)
-				(justify right)
-				(hide yes)
-			)
-		)
-	)
 	(global_label "USB_SEL"
 		(shape input)
@@
 				)
 				(justify left)
-				(hide yes)
-			)
-		)
-	)
-	(global_label "5V"
-		(shape output)
-		(at 58.42 82.55 180)
-		(fields_autoplaced yes)
-		(effects
-			(font
-				(size 1.27 1.27)
-			)
-			(justify right)
-		)
-		(property "Intersheetrefs" "${INTERSHEET_REFS}"
-			(at 53.1367 82.55 0)
-			(effects
-				(font
-					(size 1.27 1.27)
-				)
-				(justify right)
 				(hide yes)
 			)
@@
 					(unit 1)
 				)
+			)
+		)
+	)
+	(symbol
+		(lib_id "power:GNDPWR")
+		(at 123.19 82.55 270)
+		(unit 1)
+		(exclude_from_sim no)
+		(in_bom yes)
+		(on_board yes)
+		(dnp no)
+		(fields_autoplaced yes)
+		(property "Reference" "#PWR03"
+			(at 118.11 82.55 0)
+			(effects
+				(font
+					(size 1.27 1.27)
+				)
+				(hide yes)
+			)
+		)
+		(property "Value" "GNDPWR"
+			(at 119.38 82.4229 90)
+			(effects
+				(font
+					(size 1.27 1.27)
+				)
+				(justify right)
+			)
+		)
+		(property "Footprint" ""
+			(at 121.92 82.55 0)
+			(effects
+				(font
+					(size 1.27 1.27)
+				)
+				(hide yes)
+			)
+		)
+		(property "Datasheet" ""
+			(at 121.92 82.55 0)
+			(effects
+				(font
+					(size 1.27 1.27)
+				)
+				(hide yes)
+			)
+		)
+		(property "Description" "Power symbol creates a global label with name \"GNDPWR\" , global ground"
+			(at 123.19 82.55 0)
+			(effects
+				(font
+					(size 1.27 1.27)
+				)
+				(hide yes)
+			)
+		)
+		(pin "1"
+		)
+		(instances
+			(project "02-main_board[main_board_v1]"
+				(path "/0ba8c130-372e-4349-9fc9-4ef188509568/30cd09ab-8475-4f60-a19c-f1ae2b3560f0"
+					(reference "#PWR03")
+					(unit 1)
+				)

Commit message: first rev
Connections:
- net 3.3V_esp32: now also J1.20; no longer J1.17
- net 3.3V_teensy: now also J1.18; no longer J1.15
- net 5V_stable: now also J1.13, J1.14; no longer J1.19, J1.20
- net GNDA: now also J2.11, J2.13, J2.15, J2.21, J2.23, J2.7, J2.9; no longer J2.10, J2.12, J2.14, J2.16, J2.18, J2.2, J2.4
- net GNDD: now also J1.15, J1.17, J1.19, J1.2, J1.4, J1.6; no longer J1.13, J1.14, J1.18, J1.3, J1.5, J1.7
- net GNDPWR: now also J2.3, J2.4, J2.5; no longer J2.20, J2.21, J2.22
- net GP/Int1: now also J1.7; no longer J1.1
- net GP/Int2: now also J1.8; no longer J1.2
- net HFX_5V_3: now also J1.1; no longer J1.8
- net HFX_5V_cvt: now also J1.5; no longer J1.4
- net HFX_5V_eng: now also J1.3; no longer J1.6
- net analog_6: now also J2.20; no longer J2.11
- net analog_7: now also J2.22; no longer J2.13
- net analog_8: now also J2.24; no longer J2.15
- net linpot_BL: now also J2.16; no longer J2.7
- net linpot_BR: now also J2.14; no longer J2.5
- net linpot_FL: now also J2.12; no longer J2.3
- net linpot_FR: now also J2.10; no longer J2.1
- net steering_pot: now also J2.18; no longer J2.9
- removed net 11.1V: J2.23, J2.24
- net CAN_H renamed CAN+
- net CAN_L renamed CAN-
- net RX_N renamed RX-
- net RX_P renamed RX+
- net TX_N renamed TX+
- net TX_P renamed TX-
- new net 11.1V_battery: J2.1, J2.2
