File: 02-main_board[main_board_v1]/connectors.kicad_sch (KiCad schematic)
At the start: 3 parts, among them J1 2-84952-0, J2 2-84952-4, J3 FH41-15S-0.5SH_05_

Commit message: this is what i ordered
Parts:
- J3: Manufacturer (none) -> Hirose; Manufacturer_Name Hirose -> (none)
Changed lines of the file:
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@@
-			)
-		)
-		(property "Manufacturer_Name" "Hirose"
-			(at -503.15 82.55 0)
-			(effects
-				(font
-					(size 1.27 1.27)
-				)
-				(justify left top)
-				(hide yes)
 			)
 		)
@@
 				(hide yes)
 			)
+		)
+		(property "Manufacturer" "Hirose"
+			(at 186.69 35.56 90)
+			(effects
+				(font
+					(size 1.27 1.27)
+				)
+				(hide yes)
+			)
