File: 02-main_board[main_board_v1]/digital processing.kicad_sch (KiCad schematic)
At the start: 19 parts, among them U5 PT61018PEL, U6 RCLAMP3354S_TCT, U7 ATA6561-GAQW-N, U8 74LVC4245APW_118

Commit message: Updated with changes from PDR
Parts:
- added C4: 0.1uF, symbol Device:C
Connections:
- net GNDD: now also C4.1; no longer R11.1, R12.2, U8.22 (~OE)
- net 5V_ref renamed 5V_stable
- new net: C4.2, R11.1, R12.2
- new net !OE_lvlshift: U8.22 (~OE)
Other:
- moved on the sheet: C28, C30

Commit message: first rev
Parts:
- C24, C25, C26, C27, C28, C29, C30, C4: footprint (none) -> Capacitor_SMD:C_0402_1005Metric
- R11, R12, R13, R14, R15, R16, R17, R18: footprint (none) -> Resistor_SMD:R_0402_1005Metric
- U5: footprint SOIC_PT61018PEL -> footprints:SOIC_PT61018PEL
- U6: footprint SOT-23-5L_SEM -> footprints:RCLAMP3354S_TCT
- U7: footprint SOIC8_4P9X3P9MC_MCH -> footprints:ATA6561-GAQW-N
- U8: footprint 74LVC4245APW_118:SOP65P640X110-24N -> footprints:74LVC4245APW_118
Connections:
- net RD+: now also U5.1, U6.5; no longer U5.6, U6.3
- net RD-: now also U5.3, U6.4; no longer U5.8, U6.1
- net RX+: now also U5.16; no longer U5.11
- net RX-: now also U5.14; no longer U5.9
- net TD+: now also U5.8, U6.3; no longer U5.1, U6.5
- net TD-: now also U5.6, U6.1; no longer U5.3, U6.4
- net TX+: now also U5.9; no longer U5.16
- net TX-: now also U5.11; no longer U5.14
- net CAN_H renamed CAN+
- net CAN_L renamed CAN-
