File: 02-main_board[main_board_v1]/digital processing.kicad_sch (KiCad schematic)
At the start: 20 parts, among them U5 PT61018PEL, U6 74LVC4245APW_118, U7 RCLAMP3354S_TCT, U8 ATA6561-GAQW-N

Commit message: this is what i ordered
Parts:
- C25, C26, C27, C28, C29, C30, C31, C32: MPN (none) -> CC0603KRX7R9BB104; Manufacturer (none) -> YAGEO
- R16, R17, R22: MPN (none) -> RT0603BRD071K1L; Manufacturer (none) -> YAGEO
- R18, R19, R23: MPN (none) -> RC0603FR-072KL; Manufacturer (none) -> YAGEO
- R20, R21: MPN (none) -> CRCW060360R4FKEA; Manufacturer (none) -> Vishay Dale
- U6: MPN 74LVC4245APW,118 -> (none)
