File: 02-main_board[main_board_v1]/power.kicad_sch (KiCad schematic)
At the start: 20 parts, among them U1 LT3973EMSE-5-PBF, U2 MAX6105EUR+T, U3 TPS2115ADRBR

Commit message: finished schematic v1
Parts:
- U1: footprint MSOP-10_MSE_LIT -> footprints:LT3973EMSE-5#PBF
- U2: footprint 21-0051H_MXM -> footprints:MAX6105EUR+T
- U3: footprint DRB8_2P4X1P65 -> footprints:TPS2115ADRBR
Connections:
- net PGND renamed GNDPWR
Other:
- note added: "600kHz switching frequency"

Commit message: Updated with changes from PDR
Parts:
- removed C4, C5: 1uF, symbol Device:C
- removed TP4: 5V_ref, symbol Connector:TestPoint
- removed U2: MAX6105EUR+T, footprints:MAX6105EUR+T, symbol symbols:MAX6105EUR+T
- added C33, C34: 1uF, symbol Device:C
- added H1, H2: Jumper Pin, footprints:PinHeader_1x01_P2.54mm_Vertical, symbol Mechanical:MountingHole_Pad
- added R23: 12k, symbol Device:R
- added R24: 10k, symbol Device:R
- added U9: LDL1117S50R_, footprints:LDL1117S50R_, symbol symbols:LDL1117S50R_
- TP2: value 11.1V -> 5V_stable
Connections:
- net 11.1V: now also H2.1; no longer TP2.1
- net 5V: now also C33.1, U9.3 (VIN)
- net GNDPWR: now also C33.2, C34.2, R24.1, U9.1 (GND)
- net at C1.1, D1.1 (K), U1.4 (VIN): now also R23.2; no longer U1.3 (EN/UVLO)
- new net: R23.1, R24.2, U1.3 (EN/UVLO)
- new net 11.1V_battery: H1.1
- new net 5V_stable: C34.1, TP2.1, U9.2 (VOUT), U9.4 (VOUT)
Other:
- note added: "Linear Regulator"
- note added: "Resistor Divider: Vout = Vin*(r2/(r1+r2)) 5V = 11.1V*(10000/(10000+12000))"
- note removed: "5v ref"
- moved on the sheet: TP1, TP3

Commit message: first rev
Parts:
- C1, C2, C3, C33, C34, C6, C7, C8: footprint (none) -> Capacitor_SMD:C_0402_1005Metric
- D1, D2: footprint (none) -> Diode_SMD:Nexperia_CFP3_SOD-123W
- L1: footprint (none) -> footprints:IND_TAIYO_NRS4018_TAY
- R1, R2, R23, R24: footprint (none) -> Resistor_SMD:R_0402_1005Metric
- TP1, TP2, TP3: footprint (none) -> TestPoint:TestPoint_Pad_1.0x1.0mm
Connections:
- net 5V: no longer C33.1, U9.3 (VIN)
- net at C8.1, D2.2 (A), U3.7 (OUT): now also C33.1, U9.3 (VIN)
Other:
- moved on the sheet: C33, C34, D2, TP2, TP3, U9
