File: 02-main_board[main_board_v1]/02-main_board[main_board_v1].kicad_pcb (KiCad board)
At the start: 4 copper layers, 91 parts, among them IC1 AD7175-8BCPZ-RL7, J1 2-84952-0, J2 2-84952-4, J3 FH41-15S-0.5SH_05_, Q1 XIAO_ESP32S3, U1 LT3973EMSE-5-PBF, U3 TPS2115ADRBR, U4 Teensy4.1, U5 PT61018PEL, U6 RCLAMP3354S_TCT, U7 ATA6561-GAQW-N, U8 74LVC4245APW_118, U9 LDL1117S50R_

Commit message: first rev ready for design review
Parts:
- removed NT1: NetTie_1, NetTie:NetTie-2_THT_Pad0.3mm
- removed NT2: NetTie_2, NetTie:NetTie-2_THT_Pad0.3mm
- added G***: BJR_LOGO, footprints:BJR_LOGO, F.Cu at (86.9, 68.9)
- BT1: footprint footprints:BAT-HLD-012-SMT_TEC -> footprints:BatteryHolder_LINX_BAT-HLD-012-SMT
- moved H4 0.10 mm to (128.1, 68.0)
- moved H6 0.10 mm to (128.1, 120.0)
- turned BT1 to 90 degrees
Connections:
- BT1 pad 2: GNDPWR -> GNDA
- C1 pad 2: GNDPWR -> GNDA
- C13 pad 2: GNDD -> GNDA
- C14 pad 2: GNDD -> GNDA
- C16 pad 1: GNDD -> GNDA
- C24 pad 2: GNDPWR -> GNDA
- C26 pad 1: GNDPWR -> GNDA
- C27 pad 1: GNDPWR -> GNDA
- C28 pad 1: GNDPWR -> GNDA
- C29 pad 1: GNDPWR -> GNDA
- C3 pad 2: GNDPWR -> GNDA
- C30 pad 2: GNDD -> GNDA
- C31 pad 1: GNDPWR -> GNDA
- C32 pad 1: GNDPWR -> GNDA
- C33 pad 2: GNDPWR -> GNDA
- C34 pad 2: GNDPWR -> GNDA
- C4 pad 1: GNDD -> GNDA
- C6 pad 2: GNDPWR -> GNDA
- C7 pad 2: GNDPWR -> GNDA
- C8 pad 2: GNDPWR -> GNDA
- C9 pad 2: GNDD -> GNDA
- H3 pad 1: GNDPWR -> GNDA
- H5 pad 1: GNDPWR -> GNDA
- IC1 pad 19: GNDD -> GNDA
- IC1 pad 21: GNDD -> GNDA
- IC1 pad 39: GNDD -> GNDA
- IC1 pad 41: GNDD -> GNDA
- J1 pad 10: GNDD -> GNDA
- J1 pad 11: GNDD -> GNDA
- J1 pad 12: GNDD -> GNDA
- J1 pad 15: GNDD -> GNDA
- J1 pad 16: GNDD -> GNDA
- J1 pad 17: GNDD -> GNDA
- J1 pad 19: GNDD -> GNDA
- J1 pad 2: GNDD -> GNDA
- J1 pad 4: GNDD -> GNDA
- J1 pad 6: GNDD -> GNDA
- J1 pad 9: GNDD -> GNDA
- J2 pad 3: GNDPWR -> GNDA
- J2 pad 4: GNDPWR -> GNDA
- J2 pad 5: GNDPWR -> GNDA
- J3 pad 13: GNDD -> GNDA
- J3 pad 4: GNDD -> GNDA
- J3 pad G1: GNDD -> GNDA
- J3 pad G2: GNDD -> GNDA
- J3 pad G3: GNDD -> GNDA
- J3 pad MP1: GNDD -> GNDA
- J3 pad MP2: GNDD -> GNDA
- Q1 pad 13: GNDD -> GNDA
- R1 pad 2: GNDPWR -> GNDA
- R14 pad 1: GNDD -> GNDA
- R15 pad 1: GNDD -> GNDA
- R17 pad 1: GNDD -> GNDA
- R2 pad 1: GNDPWR -> GNDA
- R24 pad 1: GNDPWR -> GNDA
- U1 pad 5: GNDPWR -> GNDA
- U3 pad 2: GNDPWR -> GNDA
- U3 pad 5: GNDPWR -> GNDA
- U3 pad 9: GNDPWR -> GNDA
- U4 pad 1: GNDD -> GNDA
- U4 pad 47: GNDD -> GNDA
- U4 pad 52: GNDD -> GNDA
- U4 pad 58: GNDD -> GNDA
- U4 pad 59: GNDD -> GNDA
- U4 pad 64: GNDD -> GNDA
- U6 pad 2: GNDPWR -> GNDA
- U7 pad 2: GNDD -> GNDA
- U8 pad 11: GNDD -> GNDA
- U8 pad 12: GNDD -> GNDA
- U8 pad 13: GNDD -> GNDA
- U9 pad 1: GNDPWR -> GNDA
Routing:
- net GNDA: track 46.3 -> 175.0 mm, vias 27 -> 92
- net GNDPWR: track 77.9 -> 0.00 mm, vias 30 -> 0
- net GNDD: track 58.6 -> 0.00 mm, vias 36 -> 0
- net 5V: track 22.1 -> 29.3 mm, vias 5 -> 9
- net 3.3V_teensy: track 28.0 -> 32.1 mm, vias 5 -> 6
- net Net-(BT1-+): track 32.7 -> 33.8 mm
- net GP/Int1: track 6.75 -> 7.35 mm
- net 5V_buck: track 15.3 -> 14.8 mm
- removed copper zone on In1.Cu, net GNDD
- removed copper zone on In1.Cu, net GNDPWR
Other:
- board outline added: 82.9 x 60.6 mm
- board text added: "5V"
- board text added: "5V_B"
- board text added: "5V_S"
- board text added: "BIN"
- board text added: "BOUT"
- board text added: "Blue Jay Racing 23XT_Main Board Rev 1 Stephen Zhou, Gwenyth Tran, Sophie Noureddine"
- board text added: "CLK"
- board text added: "MISO"
- board text added: "MOSI"
- board text added: "MSI"
- board text added: "MSO"
- board text added: "SCLK"
- board text added: "SN:"

Commit message: ready for 2nd review
Parts:
- removed C34: 1uF, Capacitor_SMD:C_0402_1005Metric
- removed TP10: SCLK_esp32, TestPoint:TestPoint_Pad_1.0x1.0mm
- removed U9: LDL1117S50R_, footprints:LDL1117S50R_
- added C5: 0.1uF, Capacitor_SMD:C_0603_1608Metric, B.Cu at (87.9, 101.3)
- added TP4: MISO_adc, TestPoint:TestPoint_Pad_1.0x1.0mm, F.Cu at (124.2, 95.7)
- added U2: LT3973EMSE-5-PBF, footprints:LT3973EMSE-5#PBF, B.Cu at (101.4, 99.9)
- C1: value 4.7uF -> 0.1uF; footprint Capacitor_SMD:C_0402_1005Metric -> Capacitor_SMD:C_0603_1608Metric
- C10, C12, C13, C16, C17, C18, C2, C20, C21, C22, C23, C25, C26, C27, C28, C29, C30, C32, C7, C8: footprint Capacitor_SMD:C_0402_1005Metric -> Capacitor_SMD:C_0603_1608Metric
- C11, C14: value 1uF -> 0.1uF; footprint Capacitor_SMD:C_0402_1005Metric -> Capacitor_SMD:C_0603_1608Metric
- C15, C19, C6: value 0.1uF -> 1uF; footprint Capacitor_SMD:C_0402_1005Metric -> Capacitor_SMD:C_0603_1608Metric
- C24: footprint Capacitor_SMD:C_0402_1005Metric -> Capacitor_SMD:C_0603_1608Metric; moved to F.Cu
- C3: value 22uF -> 4.7uF; footprint Capacitor_SMD:C_0402_1005Metric -> Capacitor_SMD:C_0603_1608Metric
- C31: footprint Capacitor_SMD:C_0402_1005Metric -> Capacitor_SMD:C_0603_1608Metric; moved to B.Cu
- C33: value 1uF -> 0.1uF; footprint Capacitor_SMD:C_0402_1005Metric -> Capacitor_SMD:C_0603_1608Metric; moved to F.Cu
- C4: value 0.1uF -> 22uF; footprint Capacitor_SMD:C_0402_1005Metric -> Capacitor_SMD:C_0603_1608Metric
- C9: value 0.1uF -> 1uF; footprint Capacitor_SMD:C_0402_1005Metric -> Capacitor_SMD:C_0603_1608Metric; moved to B.Cu
- H1, H2: value Jumper Pin -> MountingHole_Pad; footprint footprints:PinHeader_1x01_P2.54mm_Vertical -> MountingHole:MountingHole_2.5mm_Pad
- H5, H6: value MountingHole_Pad -> Jumper Pin; footprint MountingHole:MountingHole_2.5mm_Pad -> footprints:PinHeader_1x01_P2.54mm_Vertical
- R1: value 215k -> 47; footprint Resistor_SMD:R_0402_1005Metric -> Resistor_SMD:R_0603_1608Metric; moved to F.Cu
- R10, R16, R7, R8, R9: footprint Resistor_SMD:R_0402_1005Metric -> Resistor_SMD:R_0603_1608Metric
- R11, R12: value 60 -> 2.2k; footprint Resistor_SMD:R_0402_1005Metric -> Resistor_SMD:R_0603_1608Metric; moved to F.Cu
- R13: value 1.1k -> 2.2k; footprint Resistor_SMD:R_0402_1005Metric -> Resistor_SMD:R_0603_1608Metric; moved to F.Cu
- R14: value 2k -> 2.2k; footprint Resistor_SMD:R_0402_1005Metric -> Resistor_SMD:R_0603_1608Metric; moved to F.Cu
- R15: value 2k -> 10k; footprint Resistor_SMD:R_0402_1005Metric -> Resistor_SMD:R_0603_1608Metric; moved to F.Cu
- R17: value 2k -> 1.1k; footprint Resistor_SMD:R_0402_1005Metric -> Resistor_SMD:R_0603_1608Metric
- R18: value 1.1k -> 2k; footprint Resistor_SMD:R_0402_1005Metric -> Resistor_SMD:R_0603_1608Metric
- R19: value 47 -> 2k; footprint Resistor_SMD:R_0402_1005Metric -> Resistor_SMD:R_0603_1608Metric; moved to B.Cu
- R2: value 400 -> 47; footprint Resistor_SMD:R_0402_1005Metric -> Resistor_SMD:R_0603_1608Metric; moved to F.Cu
- R20: value 47 -> 60; footprint Resistor_SMD:R_0402_1005Metric -> Resistor_SMD:R_0603_1608Metric; moved to B.Cu
- R21: value 10k -> 60; footprint Resistor_SMD:R_0402_1005Metric -> Resistor_SMD:R_0603_1608Metric; moved to B.Cu
- R22: value 10k -> 1.1k; footprint Resistor_SMD:R_0402_1005Metric -> Resistor_SMD:R_0603_1608Metric; moved to B.Cu
- R23: value 12k -> 2k; footprint Resistor_SMD:R_0402_1005Metric -> Resistor_SMD:R_0603_1608Metric
- R24: footprint Resistor_SMD:R_0402_1005Metric -> Resistor_SMD:R_0603_1608Metric; moved to F.Cu
- R3: value 2.2k -> 10k; footprint Resistor_SMD:R_0402_1005Metric -> Resistor_SMD:R_0603_1608Metric; moved to B.Cu
- R4: value 2.2k -> 215k; footprint Resistor_SMD:R_0402_1005Metric -> Resistor_SMD:R_0603_1608Metric; moved to B.Cu
- R5: value 2.2k -> 12k; footprint Resistor_SMD:R_0402_1005Metric -> Resistor_SMD:R_0603_1608Metric; moved to B.Cu
- R6: value 2.2k -> 400; footprint Resistor_SMD:R_0402_1005Metric -> Resistor_SMD:R_0603_1608Metric; moved to B.Cu
- TP2: value 5V_stable -> 5V
- TP3: value 5V -> 5V_stable
- TP5: value MISO_adc -> MOSI_adc
- TP6: value MOSI_adc -> SCLK_adc
- TP7: value SCLK_adc -> SCLK_esp32
- U1: value LT3973EMSE-5-PBF -> Teensy4.1; footprint footprints:LT3973EMSE-5#PBF -> footprints:Teensy41_OG; moved to F.Cu
- U4: value Teensy4.1 -> LDL1117S50R_; footprint footprints:Teensy41 -> footprints:LDL1117S50R_; moved to B.Cu
- U6: value RCLAMP3354S_TCT -> 74LVC4245APW_118; footprint footprints:RCLAMP3354S_TCT -> footprints:74LVC4245APW_118
- U7: value ATA6561-GAQW-N -> RCLAMP3354S_TCT; footprint footprints:ATA6561-GAQW-N -> footprints:RCLAMP3354S_TCT
- U8: value 74LVC4245APW_118 -> ATA6561-GAQW-N; footprint footprints:74LVC4245APW_118 -> footprints:ATA6561-GAQW-N
- moved R14 68.5 mm to (128.6, 112.1), turned to -90 degrees
- moved R12 67.8 mm to (125.4, 109.0), turned to -90 degrees
- moved R15 59.5 mm to (114.9, 95.2)
- moved R22 57.1 mm to (58.8, 97.8), turned to -90 degrees
- moved R11 55.9 mm to (112.6, 109.0)
- moved R13 55.7 mm to (115.8, 112.1), turned to -90 degrees
- moved C24 52.8 mm to (111.7, 97.5), turned to 180 degrees
- moved R23 46.3 mm to (57.2, 97.8), turned to 90 degrees
- moved H5 43.5 mm to (98.0, 112.0)
- moved H1 43.4 mm to (55.2, 120.0)
- moved C4 42.5 mm to (102.0, 94.9)
- moved C1 42.3 mm to (71.7, 73.0), turned to 0 degrees
- moved TP7 41.9 mm to (76.0, 95.5), turned to 0 degrees
- moved C9 40.4 mm to (80.6, 105.2), turned to -90 degrees
- moved C25 39.5 mm to (71.2, 107.0), turned to 0 degrees
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Connections:
- C1 pad 1: Net-(D1-K) -> GNDA
- C1 pad 2: GNDA -> 5V
- C11 pad 2: Net-(IC1-REGCAPA) -> filtered_1
- C12 pad 2: filtered_1 -> filtered_5
- C13 pad 1: 3.3V_teensy -> GNDA
- C13 pad 2: GNDA -> filtered_2
- C14 pad 1: Net-(IC1-REGCAPD) -> GNDA
- C14 pad 2: GNDA -> filtered_6
- C16 pad 2: Net-(IC1-REGCAPD) -> Net-(IC1-REGCAPA)
- C17 pad 2: filtered_2 -> filtered_3
- C18 pad 2: filtered_3 -> filtered_7
- C19 pad 1: GNDA -> Net-(IC1-REGCAPD)
- C19 pad 2: filtered_4 -> GNDA
- C2 pad 1: Net-(U1-BOOST) -> Net-(U2-BOOST)
- C2 pad 2: Net-(U1-SW) -> Net-(U2-SW)
- C20 pad 2: filtered_5 -> Net-(IC1-REGCAPD)
- C21 pad 1: GNDA -> 5V_stable
- C21 pad 2: filtered_6 -> GNDA
- C22 pad 2: filtered_7 -> filtered_4
- C24 pad 1: Net-(C24-Pad1) -> 3.3V_teensy
- C25 pad 1: Net-(C25-Pad1) -> 5V_stable
- C26 pad 1: GNDA -> Net-(C26-Pad1)
- C26 pad 2: 5V -> GNDA
- C27 pad 1: GNDA -> Net-(C27-Pad1)
- C27 pad 2: 3.3V_teensy -> GNDA
- C3 pad 1: 5V_buck -> Net-(D1-K)
- C30 pad 1: 5V_stable -> GNDA
- C30 pad 2: GNDA -> Net-(C30-Pad2)
- C32 pad 2: 5V -> 3.3V_teensy
- C33 pad 1: Net-(D2-A) -> GNDA
- C33 pad 2: GNDA -> 5V
- C4 pad 1: GNDA -> 5V_buck
- C4 pad 2: Net-(C4-Pad2) -> GNDA
- C6 pad 1: 5V_usb -> 5V_stable
- C9 pad 1: 5V_stable -> Net-(D2-A)
- H1 pad 1: 11.1V_battery -> GNDA
- H2 pad 1: 11.1V -> GNDA
- H5 pad 1: GNDA -> 11.1V_battery
- H6 pad 1: GNDA -> 11.1V
- L1 pad 2: Net-(U1-SW) -> Net-(U2-SW)
- R1 pad 1: Net-(U1-RT) -> Net-(U1-35_TX8)
- R1 pad 2: GNDA -> GP/Int1
- R10 pad 1: filtered_8 -> filtered_6
- R10 pad 2: analog_8 -> analog_6
- R11 pad 1: Net-(C4-Pad2) -> filtered_3
- R11 pad 2: CAN+ -> linpot_BR
- R12 pad 1: CAN- -> filtered_7
- R12 pad 2: Net-(C4-Pad2) -> analog_7
- R13 pad 1: HFX_3.3V_cvt -> filtered_4
- R13 pad 2: HFX_5V_cvt -> linpot_BL
- R14 pad 1: GNDA -> filtered_8
- R14 pad 2: HFX_3.3V_cvt -> analog_8
- R15 pad 1: GNDA -> !CS_adc
- R15 pad 2: HFX_3.3V_3 -> 3.3V_teensy
- R16 pad 1: HFX_3.3V_3 -> HFX_3.3V_cvt
- R16 pad 2: HFX_5V_3 -> HFX_5V_cvt
- R17 pad 1: GNDA -> HFX_3.3V_3
- R17 pad 2: HFX_3.3V_eng -> HFX_5V_3
- R18 pad 1: HFX_3.3V_eng -> GNDA
- R18 pad 2: HFX_5V_eng -> HFX_3.3V_cvt
- R19 pad 1: Net-(U4-35_TX8) -> GNDA
- R19 pad 2: GP/Int1 -> HFX_3.3V_3
- R2 pad 1: GNDA -> GP/Int2
- R2 pad 2: Net-(U3-ILIM) -> Net-(U1-34_RX8)
- R20 pad 1: GP/Int2 -> Net-(C30-Pad2)
- R20 pad 2: Net-(U4-34_RX8) -> CAN+
- R21 pad 1: 3.3V_teensy -> CAN-
- R21 pad 2: CS_esp32 -> Net-(C30-Pad2)
- R22 pad 1: !CS_adc -> HFX_3.3V_eng
- R22 pad 2: 3.3V_teensy -> HFX_5V_eng
- R23 pad 1: Net-(U1-EN/UVLO) -> GNDA
- R23 pad 2: Net-(D1-K) -> HFX_3.3V_eng
- R24 pad 1: GNDA -> 3.3V_teensy
- R24 pad 2: Net-(U1-EN/UVLO) -> CS_esp32
- R3 pad 1: filtered_1 -> GNDA
- R3 pad 2: linpot_FR -> Net-(U2-EN/UVLO)
- R4 pad 1: filtered_2 -> Net-(U2-RT)
- R4 pad 2: linpot_FL -> GNDA
- R5 pad 1: filtered_3 -> Net-(U2-EN/UVLO)
- R5 pad 2: linpot_BR -> Net-(D1-K)
- R6 pad 1: filtered_4 -> GNDA
- R6 pad 2: linpot_BL -> Net-(U3-ILIM)
- R7 pad 1: filtered_5 -> filtered_1
- R7 pad 2: steering_pot -> linpot_FR
- R8 pad 1: filtered_6 -> filtered_5
- R8 pad 2: analog_6 -> steering_pot
- R9 pad 1: filtered_7 -> filtered_2
- R9 pad 2: analog_7 -> linpot_FL
- TP2 pad 1: 5V_stable -> 5V
- TP3 pad 1: 5V -> 5V_stable
- TP5 pad 1: MISO_adc -> MOSI_adc
- TP6 pad 1: MOSI_adc -> SCLK_adc
- TP7 pad 1: SCLK_adc -> SCLK_esp32
- U1 pad 1: 5V_buck -> GNDA
- U1 pad 10: Net-(U1-RT) -> unconnected-(U1-8_TX2_IN1-Pad10)
- U1 pad 2: 5V_buck -> RXD
- U1 pad 3: Net-(U1-EN/UVLO) -> TXD
- U1 pad 4: Net-(D1-K) -> STBY_can
- U1 pad 5: GNDA -> unconnected-(U1-3_LRCLK2-Pad5)
- U1 pad 6: Net-(U1-SW) -> handshake_esp32
- U1 pad 7: Net-(U1-BOOST) -> unconnected-(U1-5_IN2-Pad7)
- U1 pad 8: 5V_buck -> USB_SEL
- U1 pad 9: unconnected-(U1-PG-Pad9) -> LED_CONTROL
- U4 pad 2: RXD -> 5V_stable
- U4 pad 3: TXD -> Net-(D2-A)
- U4 pad 4: STBY_can -> 5V_stable
- U5 pad 10: Net-(C24-Pad1) -> Net-(C27-Pad1)
- U5 pad 15: Net-(C24-Pad1) -> Net-(C27-Pad1)
- U5 pad 2: Net-(C25-Pad1) -> Net-(C26-Pad1)
- U5 pad 7: Net-(C25-Pad1) -> Net-(C26-Pad1)
- U6 pad 1: TD- -> 5V
- U6 pad 2: GNDA -> 5V_stable
- U6 pad 3: TD+ -> HFX_5V_cvt
- U6 pad 4: RD- -> unconnected-(U6-A1-Pad4)
- U6 pad 5: RD+ -> HFX_5V_eng
- U7 pad 1: TXD -> TD-
- U7 pad 3: 5V -> TD+
- U7 pad 4: RXD -> RD-
- U7 pad 5: 3.3V_teensy -> RD+
- U8 pad 1: 5V -> TXD
- U8 pad 2: 5V_stable -> GNDA
- U8 pad 3: HFX_5V_cvt -> 5V
- U8 pad 4: unconnected-(U8-A1-Pad4) -> RXD
- U8 pad 5: HFX_5V_eng -> 3.3V_teensy
- U8 pad 6: unconnected-(U8-A3-Pad6) -> CAN-
- U8 pad 7: HFX_5V_3 -> CAN+
- U8 pad 8: unconnected-(U8-A5-Pad8) -> STBY_can
Routing:
- net Net-(U4-35_TX8): track 87.4 -> 0.00 mm, vias 2 -> 0
- net Net-(U1-35_TX8): track 0.00 -> 86.3 mm, vias 0 -> 2
- net Net-(U4-34_RX8): track 79.7 -> 0.00 mm, vias 2 -> 0
- net Net-(U1-34_RX8): track 0.00 -> 78.8 mm, vias 0 -> 2
- net GNDA: track 175.0 -> 159.4 mm, vias 92 -> 113
- net Net-(C27-Pad1): track 0.00 -> 9.63 mm, vias 0 -> 2
- net Net-(C24-Pad1): track 9.63 -> 0.00 mm, vias 2 -> 0
- net Net-(C26-Pad1): track 0.00 -> 9.48 mm, vias 0 -> 2
- net Net-(C25-Pad1): track 9.48 -> 0.00 mm, vias 2 -> 0
- net Net-(U2-SW): track 0.00 -> 7.78 mm
- net Net-(U2-EN/UVLO): track 0.00 -> 6.61 mm
- net Net-(U1-SW): track 6.31 -> 0.00 mm
- net analog_7: track 7.27 -> 13.2 mm
- net Net-(U1-EN/UVLO): track 5.32 -> 0.00 mm
- net filtered_8: track 11.5 -> 16.7 mm
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- added copper zone on B.Cu, net 11.1V
- added copper zone on In2.Cu, net GNDA
- removed copper zone on In2.Cu, net 11.1V
Other:
- outline, holes or cut-outs redrawn
- board text added: "!CSa"
- board text added: "0"
- board text added: "2"
- board text added: "3.3V"
- board text added: "4"
- board text added: "6"
- board text added: "8"
- board text added: "CSe"
- board text added: "GND"
- board text added: "GP1"
- board text added: "GP2"
- board text added: "LED"
- board text added: "OE"
- board text added: "RX"
- board text added: "TX"
- board text added: "cvt"
- board text added: "eng"
- board text added: "err"
- board text added: "hESP"
- board text added: "hfx3"

Commit message: ready to order
Routing:
- net GNDA: track 159.4 -> 151.3 mm, vias 113 -> 103
Changed lines of the file:
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@@
-	)
-	(segment
-		(start 98.45 116.8398)
-		(end 98.45 118.2)
-		(width 0.2)
-		(layer "F.Cu")
-		(net 7)
 	)
 	(segment
@@
 	)
 	(segment
-		(start 104.449998 118.199998)
-		(end 104.75 118.5)
-		(width 0.2)
-		(layer "F.Cu")
-		(net 7)
-	)
-	(segment
 		(start 60.3 81.364)
 		(end 60.3 80.95)
@@
 	)
 	(segment
-		(start 75.250004 118.250004)
-		(end 75.5 118.5)
-		(width 0.2)
-		(layer "F.Cu")
-		(net 7)
-	)
-	(segment
 		(start 81.250005 118.250005)
 		(end 81.5 118.5)
@@
 	)
 	(segment
-		(start 74.250003 116.7648)
-		(end 74.250003 118.250003)
-		(width 0.2)
-		(layer "F.Cu")
-		(net 7)
-	)
-	(segment
 		(start 117.38 112.875)
 		(end 117.9 112.355)
@@
 	)
 	(segment
+		(start 74.250003 116.7648)
+		(end 77.250005 116.7648)
+		(width 0.2)
+		(layer "F.Cu")
+		(net 7)
+	)
+	(segment
 		(start 112.45 118.2)
 		(end 112.75 118.5)
@@
 	)
 	(segment
-		(start 77.250005 118.250005)
-		(end 77.5 118.5)
-		(width 0.2)
-		(layer "F.Cu")
-		(net 7)
-	)
-	(segment
 		(start 69.250006 118.250006)
 		(end 69.5 118.5)
@@
 	)
 	(segment
-		(start 80.250004 116.7648)
-		(end 80.250004 118.250004)
-		(width 0.2)
-		(layer "F.Cu")
-		(net 7)
-	)
-	(segment
 		(start 110.449999 118.199999)
 		(end 110.75 118.5)
@@
 	)
 	(segment
-		(start 74.250003 118.250003)
-		(end 74.5 118.5)
-		(width 0.2)
-		(layer "F.Cu")
-		(net 7)
-	)
-	(segment
 		(start 117.9 112.355)
 		(end 117.9 112.2)
@@
 	)
 	(segment
-		(start 82.250005 116.7648)
-		(end 82.250005 118.250005)
-		(width 0.2)
-		(layer "F.Cu")
-		(net 7)
-	)
-	(segment
 		(start 54.162 78.925)
 		(end 55.375 78.925)
@@
 	)
 	(segment
-		(start 75.250004 116.7648)
-		(end 75.250004 118.250004)
-		(width 0.2)
-		(layer "F.Cu")
-		(net 7)
-	)
-	(segment
 		(start 123.6 104)
 		(end 123.6 103.375)
@@
 	)
 	(segment
-		(start 101.449999 116.8398)
-		(end 101.449999 118.199999)
-		(width 0.2)
-		(layer "F.Cu")
-		(net 7)
-	)
-	(segment
-		(start 104.449998 116.8398)
-		(end 104.449998 118.199998)
-		(width 0.2)
-		(layer "F.Cu")
-		(net 7)
-	)
-	(segment
 		(start 114.449999 118.199999)
 		(end 114.75 118.5)
@@
 	)
 	(segment
-		(start 82.250005 118.250005)
-		(end 82.5 118.5)
-		(width 0.2)
-		(layer "F.Cu")
-		(net 7)
-	)
-	(segment
 		(start 123.8 112.9)
 		(end 122.9 113.8)
@@
 	)
 	(segment
-		(start 102.45 118.2)
-		(end 102.75 118.5)
-		(width 0.2)
-		(layer "F.Cu")
-		(net 7)
-	)
-	(segment
-		(start 77.250005 116.7648)
-		(end 77.250005 118.250005)
-		(width 0.2)
-		(layer "F.Cu")
-		(net 7)
-	)
-	(segment
 		(start 53.737 86.175)
 		(end 55.025 86.175)
@@
 	)
 	(segment
-		(start 100.449999 118.199999)
-		(end 100.75 118.5)
-		(width 0.2)
-		(layer "F.Cu")
-		(net 7)
-	)
-	(segment
-		(start 100.449999 116.8398)
-		(end 100.449999 118.199999)
-		(width 0.2)
-		(layer "F.Cu")
-		(net 7)
-	)
-	(segment
 		(start 130.2 113.5)
 		(end 129.6 114.1)
@@
 	)
 	(segment
+		(start 101.449999 116.8398)
+		(end 98.45 116.8398)
+		(width 0.2)
+		(layer "F.Cu")
+		(net 7)
+	)
+	(segment
 		(start 54.975 83.675)
 		(end 55 83.65)
@@
 	)
 	(segment
-		(start 102.45 116.8398)
-		(end 102.45 118.2)
-		(width 0.2)
-		(layer "F.Cu")
-		(net 7)
-	)
-	(segment
 		(start 122.5 102.7)
 		(end 121.825 102.7)
@@
 	)
 	(segment
-		(start 101.449999 118.199999)
-		(end 101.75 118.5)
-		(width 0.2)
-		(layer "F.Cu")
-		(net 7)
-	)
-	(segment
 		(start 67.250005 118.250005)
 		(end 67.5 118.5)
@@
 	)
 	(segment
-		(start 80.250004 118.250004)
-		(end 80.5 118.5)
-		(width 0.2)
-		(layer "F.Cu")
-		(net 7)
-	)
-	(segment
 		(start 53.737 81.175)
 		(end 54.975 81.175)
@@
 	)
 	(segment
+		(start 82.250005 116.7648)
+		(end 80.250004 116.7648)
+		(width 0.2)
+		(layer "F.Cu")
+		(net 7)
+	)
+	(segment
 		(start 67.250005 116.7648)
 		(end 67.250005 118.250005)
@@
 		(start 108.450001 118.200001)
 		(end 108.75 118.5)
-		(width 0.2)
-		(layer "F.Cu")
-		(net 7)
-	)
-	(segment
-		(start 98.45 118.2)
-		(end 98.75 118.5)
 		(width 0.2)
 		(layer "F.Cu")
@@
 	)
 	(segment
+		(start 102.45 116.8398)
+		(end 104.449998 116.8398)
+		(width 0.2)
+		(layer "F.Cu")
+		(net 7)
+	)
+	(segment
 		(start 113.45 99.34353)
 		(end 113.45 100.1)
@@
 	)
 	(via
-		(at 98.75 118.5)
-		(size 0.6)
-		(drill 0.3)
-		(layers "F.Cu" "B.Cu")
-		(net 7)
-	)
-	(via
 		(at 109.1 103.8)
 		(size 0.6)
@@
 	)
 	(via
-		(at 104.75 118.5)
-		(size 0.6)
-		(drill 0.3)
-		(layers "F.Cu" "B.Cu")
-		(net 7)
-	)
-	(via
 		(at 55 81.15)
 		(size 0.6)
@@
 	)
 	(via
-		(at 82.5 118.5)
-		(size 0.6)
-		(drill 0.3)
-		(layers "F.Cu" "B.Cu")
-		(net 7)
-	)
-	(via
 		(at 100.4 122.8)
 		(size 0.6)
@@
 	)
 	(via
-		(at 77.5 118.5)
-		(size 0.6)
-		(drill 0.3)
-		(layers "F.Cu" "B.Cu")
-		(net 7)
-	)
-	(via
 		(at 72.9 94.7)
 		(size 0.6)
@@
 	)
 	(via
-		(at 100.75 118.5)
-		(size 0.6)
-		(drill 0.3)
-		(layers "F.Cu" "B.Cu")
-		(net 7)
-	)
-	(via
 		(at 66.7 68.2)
 		(size 0.6)
@@
 	)
 	(via
-		(at 80.5 118.5)
-		(size 0.6)
-		(drill 0.3)
-		(layers "F.Cu" "B.Cu")
-		(net 7)
-	)
-	(via
 		(at 131.3 100.2)
 		(size 0.6)
@@
 	)
 	(via
-		(at 74.5 118.5)
-		(size 0.6)
-		(drill 0.3)
-		(layers "F.Cu" "B.Cu")
-		(net 7)
-	)
-	(via
 		(at 81.5 118.5)
 		(size 0.6)
@@
 	)
 	(via
-		(at 75.5 118.5)
-		(size 0.6)
-		(drill 0.3)
-		(layers "F.Cu" "B.Cu")
-		(net 7)
-	)
-	(via
 		(at 126.240894 110.438047)
 		(size 0.6)
@@
 	)
 	(via
-		(at 102.75 118.5)
-		(size 0.6)
-		(drill 0.3)
-		(layers "F.Cu" "B.Cu")
-		(net 7)
-	)
-	(via
 		(at 131.5 65.6)
 		(size 0.6)
@@
 		(size 0.6)
 		(drill 0.3)
-		(layers "F.Cu" "B.Cu")
-		(net 7)
-	)
-	(via
-		(at 101.75 118.5)
-		(size 0.6)
-		(drill 0.3)
