File: 06-main-peripheral/06-main-peripheral.kicad_sch (KiCad schematic)
At the start: 16 parts, among them J1 T4040014041000, J2 FH41-20S-0.5SH-05_, J3 T4040014041000, J4 T4040014041000, Q1 SSF2302, SW1 100SP1K1B25M1QEH-ND, U1 LM74700-Q1

Commit message: PDR Changes
Parts:
- removed C2: 100pF, symbol Device:C_Small
- removed D1: DDZ9691-7, Diode_THT:D_DO-35_SOD27_P7.62mm_Horizontal, symbol Diode:1N914
- added C2: 47uF, symbol Device:C_Small_US
- added C5: 100nF, symbol Device:C_Small
- added D1: SMBJ6.0CA, symbol Device:D_TVS
- C1: value 100pF -> 22nF
- C3: value 2.2uF -> 0.1uF
- J2: value FH41-20S-0.5SH-05_ -> FH-41-15S-0.5SH-05_
- Q1: value SSF2302 -> DMT6007LFG
Connections:
- net 3.3V: now also J2.14; no longer J2.8
- net 5V: now also J2.15, C5.1; no longer J2.18
- net CAN_H: now also J2.10; no longer J2.19
- net CAN_L: now also J2.11; no longer J2.20
- net GND: now also J1.SH, J3.SH, J4.SH, C2.2, C5.2, D1.1 (A1); no longer J2.13, J2.17, J2.7, J2.9
- net LED_CONTROL: now also J2.9; no longer J2.5
- net RX_N: now also J2.5; no longer J2.11
- net RX_P: now also J2.4; no longer J2.10
- net TX_N: now also J2.7; no longer J2.15
- net TX_P: now also J2.6; no longer J2.14
- net USB_5V: now also J2.13, C2.1; no longer J2.6
- net USB_SEL: now also C4.2, J2.8; no longer J2.4
- net at C1.1, C3.1, F1.1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: now also D1.2 (A2)
- net at R2.2, SW1.2 (B): no longer C4.2
- no-connect marks 4 -> 1
Other:
- moved on the sheet: C4, R1, R2

Commit message: layout revision before 1 on 1
Parts:
- C1, C3, C4, C5: footprint (none) -> Capacitor_SMD:C_0402_1005Metric_Pad0.74x0.62mm_HandSolder
- C2: footprint (none) -> Main_Peripheral:WCAP-ASLI_5X5.5_DXL_
- D1: footprint (none) -> Main_Peripheral:DIOM4336X265N
- D2: footprint (none) -> Main_Peripheral:LED 5050
- F1: footprint (none) -> Main_Peripheral:0ZCH0050FF2G
- J1, J3, J4: footprint (none) -> Main_Peripheral:T4040014041000
- J2: footprint (none) -> Main_Peripheral:FH4115S05SH05
- Q1: value DMT6007LFG -> DMN3018SSD-13; footprint Package_TO_SOT_SMD:SOT-23 -> Main_Peripheral:SOIC127P600X170-8N
- R1, R2: footprint (none) -> Resistor_SMD:R_0402_1005Metric_Pad0.72x0.64mm_HandSolder
- SW1: footprint (none) -> Main_Peripheral:SW_EG1218
- U1: footprint Package_TO_SOT_SMD:SOT-23-6 -> Main_Peripheral:LM74610QDGKRQ1
Connections:
- net TX_N: now also J2.6; no longer J2.7
- net TX_P: now also J2.7; no longer J2.6
- net CAN_H renamed CAN_P
- net CAN_L renamed CAN_N
Other:
- note added: "EG1218"
Changed lines of the file:
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@@
 		)
 	)
+	(text "EG1218"
+		(exclude_from_sim no)
+		(at 141.224 140.716 0)
+		(effects
+			(font
+				(size 1.27 1.27)
+			)
+		)
+	)
 	(text "Ethernet"
 		(exclude_from_sim no)
@@
 	(global_label "TX_P"
 		(shape bidirectional)
-		(at 78.74 132.08 0)
+		(at 78.74 134.62 0)
 		(fields_autoplaced yes)
 		(effects
@@
 		)
 		(property "Intersheetrefs" "${INTERSHEET_REFS}"
-			(at 87.2512 132.08 0)
+			(at 87.2512 134.62 0)
 			(hide yes)
 			(show_name no)
@@
 	(global_label "TX_N"
 		(shape bidirectional)
-		(at 78.74 134.62 0)
+		(at 78.74 132.08 0)
 		(fields_autoplaced yes)
 		(effects
@@
 		)
 		(property "Intersheetrefs" "${INTERSHEET_REFS}"
-			(at 87.3117 134.62 0)
+			(at 87.3117 132.08 0)
 			(hide yes)
 			(show_name no)
@@
 		)
 	)
-	(global_label "CAN_L"
+	(global_label "CAN_N"
 		(shape bidirectional)
 		(at 78.74 144.78 0)
@@
 		)
 		(property "Intersheetrefs" "${INTERSHEET_REFS}"
-			(at 88.5213 144.78 0)
+			(at 88.8237 144.78 0)
 			(hide yes)
 			(show_name no)
@@
 		)
 	)
-	(global_label "CAN_L"
+	(global_label "CAN_N"
 		(shape input)
 		(at 190.5 119.38 180)
@@
 		)
 		(property "Intersheetrefs" "${INTERSHEET_REFS}"
-			(at 181.83 119.38 0)
+			(at 181.5276 119.38 0)
 			(hide yes)
 			(show_name no)
@@
 		)
 	)
-	(global_label "CAN_H"
+	(global_label "CAN_P"
 		(shape bidirectional)
 		(at 78.74 142.24 0)
@@
 		)
 		(property "Intersheetrefs" "${INTERSHEET_REFS}"
-			(at 88.8237 142.24 0)
+			(at 88.7632 142.24 0)
 			(hide yes)
 			(show_name no)
@@
 		)
 	)
-	(global_label "CAN_H"
+	(global_label "CAN_P"
 		(shape input)
 		(at 190.5 116.84 180)
@@
 		)
 		(property "Intersheetrefs" "${INTERSHEET_REFS}"
-			(at 181.5276 116.84 0)
+			(at 181.5881 116.84 0)
 			(hide yes)
 			(show_name no)
@@
 			)
 		)
-		(property "Footprint" ""
+		(property "Footprint" "Capacitor_SMD:C_0402_1005Metric_Pad0.74x0.62mm_HandSolder"
 			(at 257.81 55.88 0)
 			(hide yes)
@@
 			)
 		)
-		(property "Footprint" ""
+		(property "Footprint" "Resistor_SMD:R_0402_1005Metric_Pad0.72x0.64mm_HandSolder"
 			(at 227.33 55.88 0)
 			(hide yes)
@@
 			)
 		)
-		(property "Footprint" ""
+		(property "Footprint" "Main_Peripheral:T4040014041000"
 			(at 246.888 119.38 0)
 			(hide yes)
@@
 		(in_pos_files yes)
 		(dnp no)
-		(fields_autoplaced yes)
 		(property "Reference" "Q1"
 			(at 111.76 69.85 90)
@@
 			)
 		)
-		(property "Value" "DMT6007LFG"
+		(property "Value" "DMN3018SSD-13"
 			(at 111.76 72.39 90)
 			(show_name no)
@@
 			)
 		)
-		(property "Footprint" "Package_TO_SOT_SMD:SOT-23"
+		(property "Footprint" "Main_Peripheral:SOIC127P600X170-8N"
 			(at 109.855 68.58 0)
 			(hide yes)
@@
 			)
 		)
-		(property "Footprint" ""
+		(property "Footprint" "Main_Peripheral:DIOM4336X265N"
 			(at 91.44 54.61 0)
 			(hide yes)
@@
 			)
 		)
-		(property "Footprint" ""
+		(property "Footprint" "Capacitor_SMD:C_0402_1005Metric_Pad0.74x0.62mm_HandSolder"
 			(at 130.81 44.45 0)
 			(hide yes)
@@
 			)
 		)
-		(property "Footprint" ""
+		(property "Footprint" "Main_Peripheral:LED 5050"
 			(at 242.57 55.88 0)
 			(hide yes)
@@
 			)
 		)
-		(property "Footprint" ""
+		(property "Footprint" "Main_Peripheral:T4040014041000"
 			(at 57.912 53.34 0)
 			(hide yes)
@@
 			)
 		)
-		(property "Footprint" ""
+		(property "Footprint" "Capacitor_SMD:C_0402_1005Metric_Pad0.74x0.62mm_HandSolder"
 			(at 125.73 138.43 0)
 			(hide yes)
@@
 			)
 		)
-		(property "Footprint" ""
+		(property "Footprint" "Capacitor_SMD:C_0402_1005Metric_Pad0.74x0.62mm_HandSolder"
 			(at 101.6 53.34 0)
 			(hide yes)
@@
 			)
 		)
-		(property "Footprint" ""
+		(property "Footprint" "Main_Peripheral:0ZCH0050FF2G"
 			(at 76.2 52.07 0)
 			(hide yes)
@@
 			)
 		)
-		(property "Footprint" ""
+		(property "Footprint" "Main_Peripheral:T4040014041000"
 			(at 199.898 119.38 0)
 			(hide yes)
@@
 			)
 		)
-		(property "Footprint" ""
+		(property "Footprint" "Main_Peripheral:SW_EG1218"
 			(at 143.51 144.78 0)
 			(hide yes)
@@
 			)
 		)
-		(property "Footprint" ""
+		(property "Footprint" "Main_Peripheral:WCAP-ASLI_5X5.5_DXL_"
 			(at 120.65 78.74 0)
 			(hide yes)
@@
 			)
 		)
-		(property "Footprint" "Package_TO_SOT_SMD:SOT-23-6"
+		(property "Footprint" "Main_Peripheral:LM74610QDGKRQ1"
 			(at 144.78 48.895 0)
 			(hide yes)
@@
 			)
 		)
-		(property "Footprint" ""
+		(property "Footprint" "Main_Peripheral:FH4115S05SH05"
 			(at 66.04 135.89 0)
 			(hide yes)
@@
 			)
 		)
-		(property "Footprint" ""
+		(property "Footprint" "Resistor_SMD:R_0402_1005Metric_Pad0.72x0.64mm_HandSolder"
 			(at 132.08 134.62 0)
 			(hide yes)

Commit message: before revision from overlords
Parts:
- C1, C3, C4, C5: footprint Capacitor_SMD:C_0402_1005Metric_Pad0.74x0.62mm_HandSolder -> Capacitor_SMD:C_0603_1608Metric_Pad1.08x0.95mm_HandSolder
- R1, R2: footprint Resistor_SMD:R_0402_1005Metric_Pad0.72x0.64mm_HandSolder -> Resistor_SMD:R_0603_1608Metric_Pad0.98x0.95mm_HandSolder
Changed lines of the file:
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@@
 			)
 		)
-		(property "Footprint" "Capacitor_SMD:C_0402_1005Metric_Pad0.74x0.62mm_HandSolder"
+		(property "Footprint" "Capacitor_SMD:C_0603_1608Metric_Pad1.08x0.95mm_HandSolder"
 			(at 257.81 55.88 0)
 			(hide yes)
@@
 			)
 		)
-		(property "Footprint" "Resistor_SMD:R_0402_1005Metric_Pad0.72x0.64mm_HandSolder"
+		(property "Footprint" "Resistor_SMD:R_0603_1608Metric_Pad0.98x0.95mm_HandSolder"
 			(at 227.33 55.88 0)
 			(hide yes)
@@
 			)
 		)
-		(property "Footprint" "Capacitor_SMD:C_0402_1005Metric_Pad0.74x0.62mm_HandSolder"
+		(property "Footprint" "Capacitor_SMD:C_0603_1608Metric_Pad1.08x0.95mm_HandSolder"
 			(at 130.81 44.45 0)
 			(hide yes)
@@
 			)
 		)
-		(property "Footprint" "Capacitor_SMD:C_0402_1005Metric_Pad0.74x0.62mm_HandSolder"
+		(property "Footprint" "Capacitor_SMD:C_0603_1608Metric_Pad1.08x0.95mm_HandSolder"
 			(at 125.73 138.43 0)
 			(hide yes)
@@
 			)
 		)
-		(property "Footprint" "Capacitor_SMD:C_0402_1005Metric_Pad0.74x0.62mm_HandSolder"
+		(property "Footprint" "Capacitor_SMD:C_0603_1608Metric_Pad1.08x0.95mm_HandSolder"
 			(at 101.6 53.34 0)
 			(hide yes)
@@
 			)
 		)
-		(property "Footprint" "Resistor_SMD:R_0402_1005Metric_Pad0.72x0.64mm_HandSolder"
+		(property "Footprint" "Resistor_SMD:R_0603_1608Metric_Pad0.98x0.95mm_HandSolder"
 			(at 132.08 134.62 0)
 			(hide yes)

Commit message: Fixed mosfet routing
Connections:
- net USB_5V: now also Q1.7 (D); no longer Q1.3 (D)
- net at Q1.1 (S): now also C1.1, C3.1, D1.2 (A2), F1.1, U1.3 (EN), U1.6 (ANODE); no longer U1.5 (GATE)
- new net: Q1.2 (G), U1.5 (GATE)
Changed lines of the file:
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@@
 		(pin "2"
 		)
-		(pin "3"
+		(pin "7"
 		)
 		(instances
