File: 07-crashtest-v1/crashtest-v1/untitled.kicad_sch (KiCad schematic)
At the start: 7 parts, among them U5 INA827AIDGKR

Commit message: stuff
Connections:
- net AIN+ renamed AIN
- net AIN- renamed AGND

Commit message: stuff
Connections:
- net AGND is gone; now on net VREF_1V65: C39.2
Changed lines of the file:
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@@
 		)
 	)
-	(global_label "AGND"
+	(global_label "VREF_1V65"
 		(shape input)
 		(at 170.18 87.63 0)
@@
 		)
 		(property "Intersheetrefs" "${INTERSHEET_REFS}"
-			(at 177.4701 87.63 0)
+			(at 183.4461 87.63 0)
 			(hide yes)
 			(show_name no)
