File: 07-crashtest-v1/crashtest-v1/ADC.kicad_sch (KiCad schematic)
At the start: 0 parts

Commit message: stuff
Parts:
- added C20, C25: 1uF, Capacitor_SMD:C_0603_1608Metric, symbol Device:C
- added C21, C22, C23, C24, C27, C29, C32, C33, C34, C35, C36, C37, C38: 0.1uF, Capacitor_SMD:C_0603_1608Metric, symbol Device:C
- added IC1: AD7175-8BCPZ-RL7, footprints:AD7175-8BCPZ-RL7, symbol symbols:AD7175-8BCPZ-RL7
- added R44: 10k, Resistor_SMD:R_0603_1608Metric, symbol Device:R
- added R45, R58, R59, R60, R61, R62, R63, R64: 2.2k, Resistor_SMD:R_0603_1608Metric, symbol Device:R
- added TP4: MISO_adc, TestPoint:TestPoint_Pad_1.0x1.0mm, symbol Connector:TestPoint
- added TP5: MOSI_adc, TestPoint:TestPoint_Pad_1.0x1.0mm, symbol Connector:TestPoint
- added TP6: SCLK_adc, TestPoint:TestPoint_Pad_1.0x1.0mm, symbol Connector:TestPoint
Connections:
- new net: C25.1, C27.2, IC1.22 (REGCAPD)
- new net: C20.2, C21.2, IC1.7 (REGCAPA)
- new net !CS_adc: IC1.17 (~{CS}), R44.1
- new net !ERROR_adc: IC1.18 (~{ERROR})
- new net 3.3V_teensy: C24.1, IC1.20 (IOVDD), R44.2
- new net 5V_stable: C22.1, C23.1, IC1.10 (AVDD2), IC1.40 (REF+), IC1.9 (AVDD1)
- new net GNDA: C20.1, C21.1, C22.2, C29.1, C32.1, C33.1, C34.1, C35.1, C36.1, C37.1, C38.1, IC1.11 (PDSW), IC1.8 (AVSS)
- new net GNDD: C23.2, C24.2, C25.2, C27.1, IC1.19 (~{SYNC}), IC1.21 (DGND), IC1.39 (REF-), IC1.41 (EP)
- new net MISO_adc: IC1.14 (DOUT/~{RDY}), TP4.1
- new net MOSI_adc: IC1.15 (DIN), TP5.1
- new net SCLK_adc: IC1.16 (SCLK), TP6.1
- new net analog_6: R62.2
- new net analog_7: R63.2
- new net analog_8: R64.2
- new net filtered_1: C29.2, IC1.31 (AIN9), R45.1
- new net filtered_2: C32.2, IC1.32 (AIN10), R58.1
- new net filtered_3: C33.2, IC1.33 (AIN11), R59.1
- new net filtered_4: C34.2, IC1.34 (AIN12), R60.1
- new net filtered_5: C35.2, IC1.35 (AIN13), R61.1
- new net filtered_6: C36.2, IC1.36 (AIN14), R62.1
- new net filtered_7: C37.2, IC1.37 (AIN15), R63.1
- new net filtered_8: C38.2, IC1.38 (GPO3), R64.1
- new net linpot_BL: R60.2
- new net linpot_BR: R59.2
- new net linpot_FL: R58.2
- new net linpot_FR: R45.2
- new net steering_pot: R61.2
- no-connect marks 0 -> 16
Other:
- note added: "ADC"
- note added: "Nyquist Filters"
- note added: "sampling rate: 2kHz Nyquist rate = 2kHz/2 = 1kHz cutoff frequency = 1/(2piRC) = 1/(2*pi*2.2k*0.1uF) = 723Hz"

Commit message: mcu pinout started
Connections:
- net !CS_adc renamed CS_adc
- net 3.3V_teensy renamed 3V3
