File: 07-crashtest-v1/crashtest-v1/MCU.kicad_sch (KiCad schematic)
At the start: 0 parts

Commit message: mcu pinout started
Parts:
- added U4: DEV-16771, DEV-16771:MODULE_DEV-16771, symbol Crashtest Symbols:DEV-16771
Connections:
- new net !ERROR_adc: U4.15 (A1)
- new net 2V5_EN: U4.14 (A0)
- new net 3.3V: U4.3.3V_1 (3.3V), U4.3.3V_2 (3.3V), U4.3.3V_3 (3.3V)
- new net CS_DAC: U4.36 (CS2)
- new net CS_adc: U4.10 (CS1)
- new net GND: U4.GND1 (GND), U4.GND2 (GND), U4.GND3 (GND), U4.GND4 (GND), U4.GND5 (GND), U4.USB_GND1 (USB_GND), U4.USB_GND2 (USB_GND)
- new net MISO_adc: U4.12 (MISO)
- new net MOSI_DAC: U4.26 (A12)
- new net MOSI_adc: U4.11 (MOSI)
- new net SCLK_adc: U4.13 (SCK)
Other:
- note added: "figure 5V out"
